File: _saved_demoBoard_v1.sch (KiCad schematic (older format))
At the start: 47 parts, among them P1 SPI_Header, P10 RTC_Serial, P11 WD_Header, P12 WD_1.2V_NC, P13 RTC_Aux, P14 Flash_3v3_NC, P15 WD_SENSE_3.3V_NC, P2 3x_CS_Header, P3 Power_Header, P4 LOAD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

Commit message: Beginning board layout
Parts:
- C4: footprint (none) -> SFUSat:Supercap_v2
- P1, P13, P2, P6, P7: footprint (none) -> SFUSat:3x_01In_Header
- P10: footprint (none) -> SFUSat:4x01In_Header
- P11, P12, P14, P15, P3, P4, P5, P8, P9: footprint (none) -> SFUSat:2x01In_Header
- Q1, Q2, Q3, Q4: footprint (none) -> SFUSat:SOT23_DMN2075U
- SW1: footprint (none) -> SFUSat:Tact_SW_SMD
- U1, U2, U3: footprint (none) -> SFUSat:SOT-8_208mil_medium
- U4: footprint (none) -> SFUSat:RTC_AB-RTCMC_EA09_S3
- U5: footprint (none) -> SFUSat:SOT_23_6
- U6: footprint (none) -> SFUSat:SOT25
- U7: footprint (none) -> SFUSat:VSSOP_8
Changed lines of the file:
@@
 F 0 "U1" H 2550 1700 60  0000 C CNN
 F 1 "S25FL164K0XMFV010" H 2550 1850 60  0000 C CNN
-F 2 "" H 2550 1700 60  0001 C CNN
+F 2 "SFUSat:SOT-8_208mil_medium" H 2550 1700 60  0001 C CNN
 F 3 "" H 2550 1700 60  0001 C CNN
 	1    2550 1400
@@
 F 0 "U2" H 5450 1700 60  0000 C CNN
 F 1 "S25FL164K0XMFV010" H 5450 1850 60  0000 C CNN
-F 2 "" H 5450 1700 60  0001 C CNN
+F 2 "SFUSat:SOT-8_208mil_medium" H 5450 1700 60  0001 C CNN
 F 3 "" H 5450 1700 60  0001 C CNN
 	1    5450 1400
@@
 F 0 "U3" H 8450 1700 60  0000 C CNN
 F 1 "S25FL164K0XMFV010" H 8450 1850 60  0000 C CNN
-F 2 "" H 8450 1700 60  0001 C CNN
+F 2 "SFUSat:SOT-8_208mil_medium" H 8450 1700 60  0001 C CNN
 F 3 "" H 8450 1700 60  0001 C CNN
 	1    8450 1400
@@
 F 0 "P1" H 1750 2600 50  0000 C CNN
 F 1 "SPI_Header" V 1850 2400 50  0000 C CNN
-F 2 "" H 1750 2400 50  0001 C CNN
+F 2 "SFUSat:3x_01In_Header" H 1750 2400 50  0001 C CNN
 F 3 "" H 1750 2400 50  0000 C CNN
 	1    1750 2400
@@
 F 0 "P2" H 2950 2650 50  0000 C CNN
 F 1 "3x_CS_Header" V 3050 2450 50  0000 C CNN
-F 2 "" H 2950 2450 50  0001 C CNN
+F 2 "SFUSat:3x_01In_Header" H 2950 2450 50  0001 C CNN
 F 3 "" H 2950 2450 50  0000 C CNN
 	1    2950 2450
@@
 F 0 "P3" H 5000 6900 50  0000 C CNN
 F 1 "Power_Header" V 5100 6750 50  0000 C CNN
-F 2 "" H 5000 6750 50  0001 C CNN
+F 2 "SFUSat:2x01In_Header" H 5000 6750 50  0001 C CNN
 F 3 "" H 5000 6750 50  0000 C CNN
 	1    5000 6750
@@
 F 0 "U5" H 9450 3050 60  0000 C CNN
 F 1 "TPS3110" H 9450 3400 60  0000 C CNN
-F 2 "" H 9450 3050 60  0001 C CNN
+F 2 "SFUSat:SOT_23_6" H 9450 3050 60  0001 C CNN
 F 3 "" H 9450 3050 60  0001 C CNN
 	1    9450 3050
@@
 F 0 "U6" H 6800 2700 60  0000 C CNN
 F 1 "AP7331" H 6800 3050 60  0000 C CNN
-F 2 "" H 6800 2700 60  0001 C CNN
+F 2 "SFUSat:SOT25" H 6800 2700 60  0001 C CNN
 F 3 "" H 6800 2700 60  0001 C CNN
 	1    6800 2800
@@
 F 0 "U4" H 9400 4750 60  0000 C CNN
 F 1 "AB-RTCMC-EOA9-S3" H 9450 5300 60  0000 C CNN
-F 2 "" H 9400 4900 60  0001 C CNN
+F 2 "SFUSat:RTC_AB-RTCMC_EA09_S3" H 9400 4900 60  0001 C CNN
 F 3 "" H 9400 4900 60  0001 C CNN
 	1    9400 4900
@@
 F 0 "C4" H 10875 5000 50  0000 L CNN
 F 1 "470µF" H 10875 4800 50  0000 L CNN
-F 2 "" H 10850 4900 50  0001 C CNN
+F 2 "SFUSat:Supercap_v2" H 10850 4900 50  0001 C CNN
 F 3 "" H 10850 4900 50  0000 C CNN
 	1    10850 4900
@@
 F 0 "P10" H 8100 6400 50  0000 C CNN
 F 1 "RTC_Serial" V 8200 6150 50  0000 C CNN
-F 2 "" H 8100 6150 50  0001 C CNN
+F 2 "SFUSat:4x01In_Header" H 8100 6150 50  0001 C CNN
 F 3 "" H 8100 6150 50  0000 C CNN
 	1    8100 6150
@@
 F 0 "P13" H 10050 6350 50  0000 C CNN
 F 1 "RTC_Aux" V 10150 6150 50  0000 C CNN
-F 2 "" H 10050 6150 50  0001 C CNN
+F 2 "SFUSat:3x_01In_Header" H 10050 6150 50  0001 C CNN
 F 3 "" H 10050 6150 50  0000 C CNN
 	1    10050 6150
@@
 F 0 "U7" H 3050 4950 60  0000 C CNN
 F 1 "INA301" H 3050 5150 60  0000 C CNN
-F 2 "" H 3050 4800 60  0001 C CNN
+F 2 "SFUSat:VSSOP_8" H 3050 4800 60  0001 C CNN
 F 3 "" H 3050 4800 60  0001 C CNN
 	1    3050 4800
@@
 F 0 "P7" H 3950 4150 50  0000 C CNN
 F 1 "INA_Power" V 4050 3950 50  0000 C CNN
-F 2 "" H 3950 3950 50  0001 C CNN
+F 2 "SFUSat:3x_01In_Header" H 3950 3950 50  0001 C CNN
 F 3 "" H 3950 3950 50  0000 C CNN
 	1    3950 3950
@@
 F 0 "P6" H 2350 3400 50  0000 C CNN
 F 1 "INA_GND" V 2450 3200 50  0000 C CNN
-F 2 "" H 2350 3200 50  0001 C CNN
+F 2 "SFUSat:3x_01In_Header" H 2350 3200 50  0001 C CNN
 F 3 "" H 2350 3200 50  0000 C CNN
 	1    2350 3200
@@
 F 0 "P5" H 1650 3350 50  0000 C CNN
 F 1 "INA_Signal" V 1750 3200 50  0000 C CNN
-F 2 "" H 1650 3200 50  0001 C CNN
+F 2 "SFUSat:2x01In_Header" H 1650 3200 50  0001 C CNN
 F 3 "" H 1650 3200 50  0000 C CNN
 	1    1650 3200
@@
 F 0 "P11" H 9650 3900 50  0000 C CNN
 F 1 "WD_Header" V 9750 3750 50  0000 C CNN
-F 2 "" H 9650 3750 50  0001 C CNN
+F 2 "SFUSat:2x01In_Header" H 9650 3750 50  0001 C CNN
 F 3 "" H 9650 3750 50  0000 C CNN
 	1    9650 3750
@@
 F 0 "P4" H 1000 3350 50  0000 C CNN
 F 1 "LOAD" V 1100 3200 50  0000 C CNN
-F 2 "" H 1000 3200 50  0001 C CNN
+F 2 "SFUSat:2x01In_Header" H 1000 3200 50  0001 C CNN
 F 3 "" H 1000 3200 50  0000 C CNN
 	1    1000 3200
@@
 F 0 "P14" H 10450 1200 50  0000 C CNN
 F 1 "Flash_3v3_NC" V 10550 1050 50  0000 C CNN
-F 2 "" H 10450 1050 50  0001 C CNN
+F 2 "SFUSat:2x01In_Header" H 10450 1050 50  0001 C CNN
 F 3 "" H 10450 1050 50  0000 C CNN
 	1    10450 1050
@@
 F 0 "P8" H 6000 2450 50  0000 C CNN
 F 1 "1.2V_3.3V_NC" V 6100 2300 50  0000 C CNN
-F 2 "" H 6000 2300 50  0001 C CNN
+F 2 "SFUSat:2x01In_Header" H 6000 2300 50  0001 C CNN
 F 3 "" H 6000 2300 50  0000 C CNN
 	1    6000 2300
@@
 F 0 "P12" H 10050 2500 50  0000 C CNN
 F 1 "WD_1.2V_NC" V 10150 2350 50  0000 C CNN
-F 2 "" H 10050 2350 50  0001 C CNN
+F 2 "SFUSat:2x01In_Header" H 10050 2350 50  0001 C CNN
 F 3 "" H 10050 2350 50  0000 C CNN
 	1    10050 2350
@@
 F 0 "P9" H 7950 4550 50  0000 C CNN
 F 1 "RTC_3.3_NC" V 8050 4400 50  0000 C CNN
-F 2 "" H 7950 4400 50  0001 C CNN
+F 2 "SFUSat:2x01In_Header" H 7950 4400 50  0001 C CNN
 F 3 "" H 7950 4400 50  0000 C CNN
 	1    7950 4400
@@
 F 0 "P15" H 10650 2650 50  0000 C CNN
 F 1 "WD_SENSE_3.3V_NC" V 10750 2500 50  0000 C CNN
-F 2 "" H 10650 2500 50  0001 C CNN
+F 2 "SFUSat:2x01In_Header" H 10650 2500 50  0001 C CNN
 F 3 "" H 10650 2500 50  0000 C CNN
 	1    10650 2500
@@
 F 0 "Q1" H 1100 6800 60  0000 C CNN
 F 1 "DMN2075U" H 1450 7050 60  0000 C CNN
-F 2 "" H 1100 6800 60  0001 C CNN
+F 2 "SFUSat:SOT23_DMN2075U" H 1100 6800 60  0001 C CNN
 F 3 "" H 1100 6800 60  0001 C CNN
 	1    1150 6900
@@
 F 0 "Q2" H 2700 6800 60  0000 C CNN
 F 1 "DMN2075U" H 3050 7050 60  0000 C CNN
-F 2 "" H 2700 6800 60  0001 C CNN
+F 2 "SFUSat:SOT23_DMN2075U" H 2700 6800 60  0001 C CNN
 F 3 "" H 2700 6800 60  0001 C CNN
 	1    2750 6900
@@
 F 0 "Q3" H 6700 4200 60  0000 C CNN
 F 1 "DMN2075U" H 7050 4450 60  0000 C CNN
-F 2 "" H 6700 4200 60  0001 C CNN
+F 2 "SFUSat:SOT23_DMN2075U" H 6700 4200 60  0001 C CNN
 F 3 "" H 6700 4200 60  0001 C CNN
 	1    6750 4300
@@
 F 0 "Q4" H 6150 5650 60  0000 C CNN
 F 1 "DMN2075U" H 6500 5900 60  0000 C CNN
-F 2 "" H 6150 5650 60  0001 C CNN
+F 2 "SFUSat:SOT23_DMN2075U" H 6150 5650 60  0001 C CNN
 F 3 "" H 6150 5650 60  0001 C CNN
 	1    6200 5750
@@
 F 0 "SW1" H 8400 3600 60  0000 C CNN
 F 1 "Tact_Switch_NO" H 8400 3800 60  0000 C CNN
-F 2 "" H 8400 3650 60  0001 C CNN
+F 2 "SFUSat:Tact_SW_SMD" H 8400 3650 60  0001 C CNN
 F 3 "" H 8400 3650 60  0001 C CNN
 	1    8400 3650
