File: OBC_prototypeA/SPI.sch (KiCad schematic (older format))
At the start: 2 parts, among them U1 TMS570LS0714

Commit message: Fixing issues raised by board review.
Orient silkscreen in single direction - done as much as possible.
Decrease thickness of large font - done.
Fixed global mask clearance and updated clearence for problematic parts.
1v2 power net width - 0.25mm can handle 460mA @ 10ºC raise. Max expected is around 360mA (for very brief periods of self test), normal ops are ~150mA.
Ground island pin 44 of TMS570 - this was always connected, but traces have been re routed to maximize ground plane area.
Island net U5 - cleaned up the area.
add gitignore for -bak. Done.
Todo: add pot for INA301, add FTDI.
Parts:
- renumbered SPI5_EN1 to W15
Changed lines of the file:
@@
 	6400 3100 6200 3100
 $Comp
-L TEST_1P SPI5_EN1
+L TEST_1P W15
 U 1 1 59741C61
 P 6100 4000
-F 0 "SPI5_EN1" H 6100 4270 50  0000 C CNN
+F 0 "W15" H 6100 4270 50  0000 C CNN
 F 1 "TEST_1P" H 6100 4200 50  0000 C CNN
 F 2 "SFUSat:Test_Point" H 6300 4000 50  0001 C CNN
