File: OBC_prototypeA/GPIO.sch (KiCad schematic (older format))
At the start: 7 parts, among them Q5 DMN2075U, U1 TMS570LS0714

Commit message: Added FTDI FT230 and beefed up main 1v2 bus lines
Parts:
- R9: value 100 -> 270
Changed lines of the file:
@@
 P 3950 2400
 F 0 "R9" V 4030 2400 50  0000 C CNN
-F 1 "100" V 3950 2400 50  0000 C CNN
+F 1 "270" V 3950 2400 50  0000 C CNN
 F 2 "SFUSat:R_0402" V 3880 2400 50  0001 C CNN
 F 3 "" H 3950 2400 50  0000 C CNN
@@
 GIOA6
 $Comp
-L +3V3 #PWR59
+L +3V3 #PWR058
 U 1 1 5965EBB1
 P 3950 2100
-F 0 "#PWR59" H 3950 1950 50  0001 C CNN
+F 0 "#PWR058" H 3950 1950 50  0001 C CNN
 F 1 "+3V3" H 3950 2240 50  0000 C CNN
 F 2 "" H 3950 2100 50  0000 C CNN
@@
 $EndComp
 $Comp
-L GND #PWR58
+L GND #PWR059
 U 1 1 5965EBE8
 P 3750 3900
-F 0 "#PWR58" H 3750 3650 50  0001 C CNN
+F 0 "#PWR059" H 3750 3650 50  0001 C CNN
 F 1 "GND" H 3750 3750 50  0000 C CNN
 F 2 "" H 3750 3900 50  0000 C CNN
@@
 3v3
 $Comp
-L +3V3 #PWR61
+L +3V3 #PWR060
 U 1 1 5967FAD1
 P 8800 1100
-F 0 "#PWR61" H 8800 950 50  0001 C CNN
+F 0 "#PWR060" H 8800 950 50  0001 C CNN
 F 1 "+3V3" H 8800 1240 50  0000 C CNN
 F 2 "" H 8800 1100 50  0000 C CNN
@@
 $EndComp
 $Comp
-L GND #PWR60
+L GND #PWR061
 U 1 1 59711F64
 P 5750 3700
-F 0 "#PWR60" H 5750 3450 50  0001 C CNN
+F 0 "#PWR061" H 5750 3450 50  0001 C CNN
 F 1 "GND" H 5750 3550 50  0000 C CNN
 F 2 "" H 5750 3700 50  0000 C CNN
