File: OBC_prototypeA/PC104_Connector.sch (KiCad schematic (older format))
At the start: 4 parts, among them J1 PC104-8BIT, P6 USB_PORT, Q4 DMN2075U

Commit message: Added FTDI FT230 and beefed up main 1v2 bus lines
Parts:
- added C1, C3: 47pF, SFUSat:C_0402, symbol C_Small
- added C33: 10nF, SFUSat:C_0402, symbol C_Small
- added C8: 100nF, SFUSat:C_0402, symbol C_Small
- added D4: TX, SFUSat:LED_0603, symbol LED
- added D5: RX, SFUSat:LED_0603, symbol LED
- added P11: USB_5V, SFUSat:2x01In_Header_v2, symbol CONN_01X02
- added R2, R31: 27, SFUSat:R_0402, symbol R
- added R32, R33, R34, R35: 10k, SFUSat:R_0402, symbol R
- added R36, R37: 270, SFUSat:R_0402, symbol R
- added U10: FT230XQ-R, SFUSat:QFN-16_650P, symbol FT230XQ-R
Connections:
- net labels added: FTDI_VCCIO, USB_2, USB_3, USB_5V
- wire segments 132 -> 184

Commit message: Added gerbers, redid USB section (just need to add differential pair), fixed USB connector paste
Parts:
- removed C1, C3: 47pF, SFUSat:C_0402, symbol C_Small
Connections:
- net labels added: RUSB_N, RUSB_P, USB_N, USB_P
- net labels removed: USB_2, USB_3
- wire segments 184 -> 178
Changed lines of the file:
@@
 104_In_GND
 Text GLabel 7500 5300 0    60   Input ~ 0
-USB_2
+USB_N
 Text GLabel 7500 5450 0    60   Input ~ 0
-USB_3
+USB_P
 $Comp
 L USB_PORT P6
@@
 USB_5V
 Text GLabel 950  6150 0    60   Input ~ 0
-USB_2
+USB_N
 Text GLabel 950  6300 0    60   Input ~ 0
-USB_3
+USB_P
 $Comp
 L R R2
@@
 Wire Wire Line
 	1850 6250 1900 6250
-$Comp
-L C_Small C1
-U 1 1 597E74BC
-P 1050 6500
-F 0 "C1" H 1060 6570 50  0000 L CNN
-F 1 "47pF" H 700 6400 50  0000 L CNN
-F 2 "SFUSat:C_0402" H 1050 6500 50  0001 C CNN
-F 3 "" H 1050 6500 50  0000 C CNN
-	1    1050 6500
-	1    0    0    -1
-$EndComp
-$Comp
-L C_Small C3
-U 1 1 597E74F8
-P 1250 6500
-F 0 "C3" H 1260 6570 50  0000 L CNN
-F 1 "47pF" H 1260 6420 50  0000 L CNN
-F 2 "SFUSat:C_0402" H 1250 6500 50  0001 C CNN
-F 3 "" H 1250 6500 50  0000 C CNN
-	1    1250 6500
-	1    0    0    -1
-$EndComp
-Wire Wire Line
-	1050 6400 1050 6150
-Connection ~ 1050 6150
-Wire Wire Line
-	1250 6400 1250 6300
-Connection ~ 1250 6300
-Wire Wire Line
-	1050 6600 1050 6650
-Wire Wire Line
-	1050 6650 1250 6650
-Wire Wire Line
-	1250 6650 1250 6600
-Text GLabel 1150 6850 3    60   Input ~ 0
-104_In_GND
-Wire Wire Line
-	1150 6650 1150 6850
-Connection ~ 1150 6650
 Wire Wire Line
 	8200 5700 7450 5700
@@
 Wire Wire Line
 	4050 6100 4050 5700
+Text GLabel 4300 5800 2    60   Input ~ 0
+UART_RX
 Text GLabel 4300 5950 2    60   Input ~ 0
-UART_RX
-Text GLabel 4300 5800 2    60   Input ~ 0
 UART_TX
 Connection ~ 3450 5800
@@
 Connection ~ 3450 5150
 Connection ~ 5150 5400
+Text Label 1800 6150 0    60   ~ 0
+RUSB_N
+Text Label 1800 6300 0    60   ~ 0
+RUSB_P
 $EndSCHEMATC
