File: OBC_prototypeA/MCU_Support_Reset.sch (KiCad schematic (older format))
At the start: 22 parts, among them P12 JTAG_20PIN, P7 OSC_FUALT_INJECT, SW1 SPST, SW2 SPST, U1 TMS570LS0714, U9 TPS3110, Y1 XTAL

Commit message: Watchdog enable jumper
Parts:
- added P13: WD_EN, SFUSat:2x01In_Header_v2, symbol CONN_01X02
Connections:
- wire segments 90 -> 91
Changed lines of the file:
@@
 L +3V3 #PWR039
 U 1 1 597111CE
-P 6750 1700
-F 0 "#PWR039" H 6750 1550 50  0001 C CNN
-F 1 "+3V3" H 6750 1840 50  0000 C CNN
-F 2 "" H 6750 1700 50  0000 C CNN
-F 3 "" H 6750 1700 50  0000 C CNN
-	1    6750 1700
+P 7100 1700
+F 0 "#PWR039" H 7100 1550 50  0001 C CNN
+F 1 "+3V3" H 7100 1840 50  0000 C CNN
+F 2 "" H 7100 1700 50  0000 C CNN
+F 3 "" H 7100 1700 50  0000 C CNN
+	1    7100 1700
 	1    0    0    -1
 $EndComp
@@
 Wire Wire Line
 	4550 6250 4700 6250
+$Comp
+L CONN_01X02 P13
+U 1 1 59780157
+P 6800 1500
+F 0 "P13" H 6800 1650 50  0000 C CNN
+F 1 "WD_EN" V 6900 1500 50  0000 C CNN
+F 2 "SFUSat:2x01In_Header_v2" H 6800 1500 50  0001 C CNN
+F 3 "" H 6800 1500 50  0000 C CNN
+	1    6800 1500
+	0    -1   -1   0
+$EndComp
+Wire Wire Line
+	6850 1700 7100 1700
 $EndSCHEMATC

Commit message: Fixing issues raised by board review.
Orient silkscreen in single direction - done as much as possible.
Decrease thickness of large font - done.
Fixed global mask clearance and updated clearence for problematic parts.
1v2 power net width - 0.25mm can handle 460mA @ 10ºC raise. Max expected is around 360mA (for very brief periods of self test), normal ops are ~150mA.
Ground island pin 44 of TMS570 - this was always connected, but traces have been re routed to maximize ground plane area.
Island net U5 - cleaned up the area.
add gitignore for -bak. Done.
Todo: add pot for INA301, add FTDI.
Parts:
- JTAG_5V_SRC1: value JTAG_5V_SRC -> JTAG5V_IN
Changed lines of the file:
@@
 P 4500 6550
 F 0 "JTAG_5V_SRC1" H 4500 6700 50  0000 C CNN
-F 1 "JTAG_5V_SRC" V 4600 6550 50  0000 C CNN
+F 1 "JTAG5V_IN" V 4600 6550 50  0000 C CNN
 F 2 "SFUSat:2x01In_Header_v2" H 4500 6550 50  0001 C CNN
 F 3 "" H 4500 6550 50  0000 C CNN

Commit message: Added FTDI FT230 and beefed up main 1v2 bus lines
Parts:
- renumbered JTAG_5V_SRC1 to JTAG5V_IN1
Changed lines of the file:
@@
 $EndComp
 $Comp
-L +3V3 #PWR37
+L +3V3 #PWR034
 U 1 1 5956048B
 P 1200 700
-F 0 "#PWR37" H 1200 550 50  0001 C CNN
+F 0 "#PWR034" H 1200 550 50  0001 C CNN
 F 1 "+3V3" H 1200 840 50  0000 C CNN
 F 2 "" H 1200 700 50  0000 C CNN
@@
 Connection ~ 1550 1700
 $Comp
-L GND #PWR35
+L GND #PWR035
 U 1 1 59682837
 P 1050 1650
-F 0 "#PWR35" H 1050 1400 50  0001 C CNN
+F 0 "#PWR035" H 1050 1400 50  0001 C CNN
 F 1 "GND" H 1050 1500 50  0000 C CNN
 F 2 "" H 1050 1650 50  0000 C CNN
@@
 	8800 3300 8800 2500
 $Comp
-L GND #PWR51
+L GND #PWR036
 U 1 1 5968A38D
 P 8700 3350
-F 0 "#PWR51" H 8700 3100 50  0001 C CNN
+F 0 "#PWR036" H 8700 3100 50  0001 C CNN
 F 1 "GND" H 8700 3200 50  0000 C CNN
 F 2 "" H 8700 3350 50  0000 C CNN
@@
 $EndComp
 $Comp
-L +3V3 #PWR53
+L +3V3 #PWR037
 U 1 1 5968A3C2
 P 9600 2100
-F 0 "#PWR53" H 9600 1950 50  0001 C CNN
+F 0 "#PWR037" H 9600 1950 50  0001 C CNN
 F 1 "+3V3" H 9600 2240 50  0000 C CNN
 F 2 "" H 9600 2100 50  0000 C CNN
@@
 1v2
 $Comp
-L +1V2 #PWR38
+L +1V2 #PWR038
 U 1 1 5968AD45
 P 1500 700
-F 0 "#PWR38" H 1500 550 50  0001 C CNN
+F 0 "#PWR038" H 1500 550 50  0001 C CNN
 F 1 "+1V2" H 1500 840 50  0000 C CNN
 F 2 "" H 1500 700 50  0000 C CNN
@@
 	8550 1400 9150 1400
 $Comp
-L +3V3 #PWR48
+L +3V3 #PWR039
 U 1 1 597111CE
 P 7100 1700
-F 0 "#PWR48" H 7100 1550 50  0001 C CNN
+F 0 "#PWR039" H 7100 1550 50  0001 C CNN
 F 1 "+3V3" H 7100 1840 50  0000 C CNN
 F 2 "" H 7100 1700 50  0000 C CNN
@@
 $EndComp
 $Comp
-L GND #PWR44
+L GND #PWR040
 U 1 1 59711206
 P 5200 2050
-F 0 "#PWR44" H 5200 1800 50  0001 C CNN
+F 0 "#PWR040" H 5200 1800 50  0001 C CNN
 F 1 "GND" H 5200 1900 50  0000 C CNN
 F 2 "" H 5200 2050 50  0000 C CNN
@@
 $EndComp
 $Comp
-L GND #PWR47
+L GND #PWR041
 U 1 1 59711388
 P 6750 2600
-F 0 "#PWR47" H 6750 2350 50  0001 C CNN
+F 0 "#PWR041" H 6750 2350 50  0001 C CNN
 F 1 "GND" H 6750 2450 50  0000 C CNN
 F 2 "" H 6750 2600 50  0000 C CNN
@@
 	5500 2200 5600 2200
 $Comp
-L GND #PWR45
+L GND #PWR042
 U 1 1 5971283C
 P 5500 3250
-F 0 "#PWR45" H 5500 3000 50  0001 C CNN
+F 0 "#PWR042" H 5500 3000 50  0001 C CNN
 F 1 "GND" H 5500 3100 50  0000 C CNN
 F 2 "" H 5500 3250 50  0000 C CNN
@@
 $EndComp
 $Comp
-L +1V2 #PWR49
+L +1V2 #PWR043
 U 1 1 59712E3B
 P 7700 1650
-F 0 "#PWR49" H 7700 1500 50  0001 C CNN
+F 0 "#PWR043" H 7700 1500 50  0001 C CNN
 F 1 "+1V2" H 7700 1790 50  0000 C CNN
 F 2 "" H 7700 1650 50  0000 C CNN
@@
 	7700 1800 7700 1650
 $Comp
-L GND #PWR50
+L GND #PWR044
 U 1 1 59713064
 P 7700 2750
-F 0 "#PWR50" H 7700 2500 50  0001 C CNN
+F 0 "#PWR044" H 7700 2500 50  0001 C CNN
 F 1 "GND" H 7700 2600 50  0000 C CNN
 F 2 "" H 7700 2750 50  0000 C CNN
@@
 	7700 2650 7700 2750
 $Comp
-L +3V3 #PWR52
+L +3V3 #PWR045
 U 1 1 597134C1
 P 8900 950
-F 0 "#PWR52" H 8900 800 50  0001 C CNN
+F 0 "#PWR045" H 8900 800 50  0001 C CNN
 F 1 "+3V3" H 8900 1090 50  0000 C CNN
 F 2 "" H 8900 950 50  0000 C CNN
@@
 	1050 5250 1050 5450
 $Comp
-L +3V3 #PWR41
+L +3V3 #PWR046
 U 1 1 59719A03
 P 3300 5050
-F 0 "#PWR41" H 3300 4900 50  0001 C CNN
+F 0 "#PWR046" H 3300 4900 50  0001 C CNN
 F 1 "+3V3" H 3300 5190 50  0000 C CNN
 F 2 "" H 3300 5050 50  0000 C CNN
@@
 $EndComp
 $Comp
-L +3V3 #PWR40
+L +3V3 #PWR047
 U 1 1 59719A6D
 P 3000 4750
-F 0 "#PWR40" H 3000 4600 50  0001 C CNN
+F 0 "#PWR047" H 3000 4600 50  0001 C CNN
 F 1 "+3V3" H 3000 4890 50  0000 C CNN
 F 2 "" H 3000 4750 50  0000 C CNN
@@
 $EndComp
 $Comp
-L +3V3 #PWR36
+L +3V3 #PWR048
 U 1 1 59719ABA
 P 1050 4850
-F 0 "#PWR36" H 1050 4700 50  0001 C CNN
+F 0 "#PWR048" H 1050 4700 50  0001 C CNN
 F 1 "+3V3" H 1050 4990 50  0000 C CNN
 F 2 "" H 1050 4850 50  0000 C CNN
@@
 $EndComp
 $Comp
-L +3V3 #PWR34
+L +3V3 #PWR049
 U 1 1 59719B8B
 P 850 5100
-F 0 "#PWR34" H 850 4950 50  0001 C CNN
+F 0 "#PWR049" H 850 4950 50  0001 C CNN
 F 1 "+3V3" H 850 5240 50  0000 C CNN
 F 2 "" H 850 5100 50  0000 C CNN
@@
 	1400 5300 1400 4850
 $Comp
-L GND #PWR39
+L GND #PWR050
 U 1 1 59740380
 P 1500 5900
-F 0 "#PWR39" H 1500 5650 50  0001 C CNN
+F 0 "#PWR050" H 1500 5650 50  0001 C CNN
 F 1 "GND" H 1500 5750 50  0000 C CNN
 F 2 "" H 1500 5900 50  0000 C CNN
@@
 	1500 5150 1500 5900
 $Comp
-L +3V3 #PWR43
+L +3V3 #PWR051
 U 1 1 597406F6
 P 4650 5250
-F 0 "#PWR43" H 4650 5100 50  0001 C CNN
+F 0 "#PWR051" H 4650 5100 50  0001 C CNN
 F 1 "+3V3" H 4650 5390 50  0000 C CNN
 F 2 "" H 4650 5250 50  0000 C CNN
@@
 	4650 5350 4650 5250
 $Comp
-L GND #PWR46
+L GND #PWR052
 U 1 1 59740B82
 P 5950 6350
-F 0 "#PWR46" H 5950 6100 50  0001 C CNN
+F 0 "#PWR052" H 5950 6100 50  0001 C CNN
 F 1 "GND" H 5950 6200 50  0000 C CNN
 F 2 "" H 5950 6350 50  0000 C CNN
@@
 Connection ~ 5950 6250
 $Comp
-L CONN_01X02 JTAG_5V_SRC1
+L CONN_01X02 JTAG5V_IN1
 U 1 1 59741105
 P 4500 6550
-F 0 "JTAG_5V_SRC1" H 4500 6700 50  0000 C CNN
+F 0 "JTAG5V_IN1" V 4600 6550 50  0000 C CNN
 F 1 "JTAG5V_IN" V 4600 6550 50  0000 C CNN
 F 2 "SFUSat:2x01In_Header_v2" H 4500 6550 50  0001 C CNN
@@
 $EndComp
 $Comp
-L +5V #PWR42
+L +5V #PWR053
 U 1 1 597411F2
 P 4250 6350
-F 0 "#PWR42" H 4250 6200 50  0001 C CNN
+F 0 "#PWR053" H 4250 6200 50  0001 C CNN
 F 1 "+5V" H 4250 6490 50  0000 C CNN
 F 2 "" H 4250 6350 50  0000 C CNN

Commit message: Fixed oscillator circuit.
Parts:
- added R38: 1k, SFUSat:R_0402, symbol R
Connections:
- wire segments 91 -> 92
Changed lines of the file:
@@
 $EndComp
 $Comp
-L +3V3 #PWR034
+L +3V3 #PWR37
 U 1 1 5956048B
 P 1200 700
-F 0 "#PWR034" H 1200 550 50  0001 C CNN
+F 0 "#PWR37" H 1200 550 50  0001 C CNN
 F 1 "+3V3" H 1200 840 50  0000 C CNN
 F 2 "" H 1200 700 50  0000 C CNN
@@
 L C_Small C27
 U 1 1 596825F7
-P 1900 1850
-F 0 "C27" H 1910 1920 50  0000 L CNN
-F 1 "33pF" H 1910 1770 50  0000 L CNN
-F 2 "SFUSat:C_0402" H 1900 1850 50  0001 C CNN
-F 3 "" H 1900 1850 50  0000 C CNN
-	1    1900 1850
-	0    -1   -1   0
+P 1800 1800
+F 0 "C27" H 1810 1870 50  0000 L CNN
+F 1 "33pF" H 1810 1720 50  0000 L CNN
+F 2 "SFUSat:C_0402" H 1800 1800 50  0001 C CNN
+F 3 "" H 1800 1800 50  0000 C CNN
+	1    1800 1800
+	1    0    0    -1
 $EndComp
 $Comp
 L C_Small C28
 U 1 1 59682616
-P 1900 2150
-F 0 "C28" H 1910 2220 50  0000 L CNN
-F 1 "33pF" H 1500 2100 50  0000 L CNN
-F 2 "SFUSat:C_0402" H 1900 2150 50  0001 C CNN
-F 3 "" H 1900 2150 50  0000 C CNN
-	1    1900 2150
-	0    -1   -1   0
-$EndComp
-Wire Wire Line
-	2000 1850 2250 1850
-Wire Wire Line
-	1800 1700 1800 2250
-Wire Wire Line
-	1800 2000 2250 2000
-Connection ~ 1800 2000
-Wire Wire Line
-	2250 2150 2000 2150
-Wire Wire Line
-	1300 1700 1800 1700
-Connection ~ 1800 1850
-Wire Wire Line
-	1800 2250 1300 2250
-Connection ~ 1800 2150
+P 1800 2150
+F 0 "C28" H 1810 2220 50  0000 L CNN
+F 1 "33pF" H 1400 2100 50  0000 L CNN
+F 2 "SFUSat:C_0402" H 1800 2150 50  0001 C CNN
+F 3 "" H 1800 2150 50  0000 C CNN
+	1    1800 2150
+	1    0    0    -1
+$EndComp
+Wire Wire Line
+	1300 1700 2250 1700
+Wire Wire Line
+	1300 2250 2250 2250
 $Comp
 L CONN_01X02 P7
 U 1 1 596827B1
-P 1100 1400
-F 0 "P7" H 1100 1550 50  0000 C CNN
-F 1 "OSC_FUALT_INJECT" V 1200 1400 50  0000 C CNN
-F 2 "SFUSat:2x01In_Header_v2" H 1100 1400 50  0001 C CNN
-F 3 "" H 1100 1400 50  0000 C CNN
-	1    1100 1400
+P 850 1300
+F 0 "P7" H 850 1450 50  0000 C CNN
+F 1 "OSC_FUALT_INJECT" V 950 1300 50  0000 C CNN
+F 2 "SFUSat:2x01In_Header_v2" H 850 1300 50  0001 C CNN
+F 3 "" H 850 1300 50  0000 C CNN
+	1    850  1300
 	0    -1   -1   0
 $EndComp
 Wire Wire Line
-	1150 1600 1550 1600
-Wire Wire Line
-	1550 1600 1550 1700
+	1550 1500 1550 1700
 Connection ~ 1550 1700
 $Comp
-L GND #PWR035
+L GND #PWR34
 U 1 1 59682837
-P 1050 1650
-F 0 "#PWR035" H 1050 1400 50  0001 C CNN
-F 1 "GND" H 1050 1500 50  0000 C CNN
-F 2 "" H 1050 1650 50  0000 C CNN
-F 3 "" H 1050 1650 50  0000 C CNN
-	1    1050 1650
-	1    0    0    -1
-$EndComp
-Wire Wire Line
-	1050 1600 1050 1650
+P 800 1550
+F 0 "#PWR34" H 800 1300 50  0001 C CNN
+F 1 "GND" H 800 1400 50  0000 C CNN
+F 2 "" H 800 1550 50  0000 C CNN
+F 3 "" H 800 1550 50  0000 C CNN
+	1    800  1550
+	1    0    0    -1
+$EndComp
+Wire Wire Line
+	800  1500 800  1550
 Text GLabel 5350 1800 0    60   Input ~ 0
 MASTER_RESET
@@
 	8800 3300 8800 2500
 $Comp
-L GND #PWR036
+L GND #PWR51
 U 1 1 5968A38D
 P 8700 3350
-F 0 "#PWR036" H 8700 3100 50  0001 C CNN
+F 0 "#PWR51" H 8700 3100 50  0001 C CNN
 F 1 "GND" H 8700 3200 50  0000 C CNN
 F 2 "" H 8700 3350 50  0000 C CNN
@@
 $EndComp
 $Comp
-L +3V3 #PWR037
+L +3V3 #PWR53
 U 1 1 5968A3C2
 P 9600 2100
-F 0 "#PWR037" H 9600 1950 50  0001 C CNN
+F 0 "#PWR53" H 9600 1950 50  0001 C CNN
 F 1 "+3V3" H 9600 2240 50  0000 C CNN
 F 2 "" H 9600 2100 50  0000 C CNN
@@
 1v2
 $Comp
-L +1V2 #PWR038
+L +1V2 #PWR38
 U 1 1 5968AD45
 P 1500 700
-F 0 "#PWR038" H 1500 550 50  0001 C CNN
+F 0 "#PWR38" H 1500 550 50  0001 C CNN
 F 1 "+1V2" H 1500 840 50  0000 C CNN
 F 2 "" H 1500 700 50  0000 C CNN
@@
 	8550 1400 9150 1400
 $Comp
-L +3V3 #PWR039
+L +3V3 #PWR48
 U 1 1 597111CE
 P 7100 1700
-F 0 "#PWR039" H 7100 1550 50  0001 C CNN
+F 0 "#PWR48" H 7100 1550 50  0001 C CNN
 F 1 "+3V3" H 7100 1840 50  0000 C CNN
 F 2 "" H 7100 1700 50  0000 C CNN
@@
 $EndComp
 $Comp
-L GND #PWR040
+L GND #PWR44
 U 1 1 59711206
 P 5200 2050
-F 0 "#PWR040" H 5200 1800 50  0001 C CNN
+F 0 "#PWR44" H 5200 1800 50  0001 C CNN
 F 1 "GND" H 5200 1900 50  0000 C CNN
 F 2 "" H 5200 2050 50  0000 C CNN
@@
 $EndComp
 $Comp
-L GND #PWR041
+L GND #PWR47
 U 1 1 59711388
 P 6750 2600
-F 0 "#PWR041" H 6750 2350 50  0001 C CNN
+F 0 "#PWR47" H 6750 2350 50  0001 C CNN
 F 1 "GND" H 6750 2450 50  0000 C CNN
 F 2 "" H 6750 2600 50  0000 C CNN
@@
 	5500 2200 5600 2200
 $Comp
-L GND #PWR042
+L GND #PWR45
 U 1 1 5971283C
 P 5500 3250
-F 0 "#PWR042" H 5500 3000 50  0001 C CNN
+F 0 "#PWR45" H 5500 3000 50  0001 C CNN
 F 1 "GND" H 5500 3100 50  0000 C CNN
 F 2 "" H 5500 3250 50  0000 C CNN
@@
 $EndComp
 $Comp
-L +1V2 #PWR043
+L +1V2 #PWR49
 U 1 1 59712E3B
 P 7700 1650
-F 0 "#PWR043" H 7700 1500 50  0001 C CNN
+F 0 "#PWR49" H 7700 1500 50  0001 C CNN
 F 1 "+1V2" H 7700 1790 50  0000 C CNN
 F 2 "" H 7700 1650 50  0000 C CNN
@@
 	7700 1800 7700 1650
 $Comp
-L GND #PWR044
+L GND #PWR50
 U 1 1 59713064
 P 7700 2750
-F 0 "#PWR044" H 7700 2500 50  0001 C CNN
+F 0 "#PWR50" H 7700 2500 50  0001 C CNN
 F 1 "GND" H 7700 2600 50  0000 C CNN
 F 2 "" H 7700 2750 50  0000 C CNN
@@
 	7700 2650 7700 2750
 $Comp
-L +3V3 #PWR045
+L +3V3 #PWR52
 U 1 1 597134C1
 P 8900 950
-F 0 "#PWR045" H 8900 800 50  0001 C CNN
+F 0 "#PWR52" H 8900 800 50  0001 C CNN
 F 1 "+3V3" H 8900 1090 50  0000 C CNN
 F 2 "" H 8900 950 50  0000 C CNN
@@
 	1050 5250 1050 5450
 $Comp
-L +3V3 #PWR046
+L +3V3 #PWR41
 U 1 1 59719A03
 P 3300 5050
-F 0 "#PWR046" H 3300 4900 50  0001 C CNN
+F 0 "#PWR41" H 3300 4900 50  0001 C CNN
 F 1 "+3V3" H 3300 5190 50  0000 C CNN
 F 2 "" H 3300 5050 50  0000 C CNN
@@
 $EndComp
 $Comp
-L +3V3 #PWR047
+L +3V3 #PWR40
 U 1 1 59719A6D
 P 3000 4750
-F 0 "#PWR047" H 3000 4600 50  0001 C CNN
+F 0 "#PWR40" H 3000 4600 50  0001 C CNN
 F 1 "+3V3" H 3000 4890 50  0000 C CNN
 F 2 "" H 3000 4750 50  0000 C CNN
@@
 $EndComp
 $Comp
-L +3V3 #PWR048
+L +3V3 #PWR36
 U 1 1 59719ABA
 P 1050 4850
-F 0 "#PWR048" H 1050 4700 50  0001 C CNN
+F 0 "#PWR36" H 1050 4700 50  0001 C CNN
 F 1 "+3V3" H 1050 4990 50  0000 C CNN
 F 2 "" H 1050 4850 50  0000 C CNN
@@
 $EndComp
 $Comp
-L +3V3 #PWR049
+L +3V3 #PWR35
 U 1 1 59719B8B
 P 850 5100
-F 0 "#PWR049" H 850 4950 50  0001 C CNN
+F 0 "#PWR35" H 850 4950 50  0001 C CNN
 F 1 "+3V3" H 850 5240 50  0000 C CNN
 F 2 "" H 850 5100 50  0000 C CNN
@@
 	1400 5300 1400 4850
 $Comp
-L GND #PWR050
+L GND #PWR39
 U 1 1 59740380
 P 1500 5900
-F 0 "#PWR050" H 1500 5650 50  0001 C CNN
+F 0 "#PWR39" H 1500 5650 50  0001 C CNN
 F 1 "GND" H 1500 5750 50  0000 C CNN
 F 2 "" H 1500 5900 50  0000 C CNN
@@
 	1500 5150 1500 5900
 $Comp
-L +3V3 #PWR051
+L +3V3 #PWR43
 U 1 1 597406F6
 P 4650 5250
-F 0 "#PWR051" H 4650 5100 50  0001 C CNN
+F 0 "#PWR43" H 4650 5100 50  0001 C CNN
 F 1 "+3V3" H 4650 5390 50  0000 C CNN
 F 2 "" H 4650 5250 50  0000 C CNN
@@
 	4650 5350 4650 5250
 $Comp
-L GND #PWR052
+L GND #PWR46
 U 1 1 59740B82
 P 5950 6350
-F 0 "#PWR052" H 5950 6100 50  0001 C CNN
+F 0 "#PWR46" H 5950 6100 50  0001 C CNN
 F 1 "GND" H 5950 6200 50  0000 C CNN
 F 2 "" H 5950 6350 50  0000 C CNN
@@
 $EndComp
 $Comp
-L +5V #PWR053
+L +5V #PWR42
 U 1 1 597411F2
 P 4250 6350
-F 0 "#PWR053" H 4250 6200 50  0001 C CNN
+F 0 "#PWR42" H 4250 6200 50  0001 C CNN
 F 1 "+5V" H 4250 6490 50  0000 C CNN
 F 2 "" H 4250 6350 50  0000 C CNN
@@
 Wire Wire Line
 	6850 1700 7100 1700
+Wire Wire Line
+	1800 1900 1800 2050
+Wire Wire Line
+	1800 2000 2250 2000
+Connection ~ 1800 2000
+Wire Wire Line
+	2250 2250 2250 2150
+Connection ~ 1800 2250
+Wire Wire Line
+	2250 1700 2250 1850
+Connection ~ 1800 1700
+$Comp
+L R R38
+U 1 1 597F6613
+P 1200 1500
+F 0 "R38" V 1280 1500 50  0000 C CNN
+F 1 "1k" V 1200 1500 50  0000 C CNN
+F 2 "SFUSat:R_0402" V 1130 1500 50  0001 C CNN
+F 3 "" H 1200 1500 50  0000 C CNN
+	1    1200 1500
+	0    1    1    0
+$EndComp
+Wire Wire Line
+	1350 1500 1550 1500
+Wire Wire Line
+	1050 1500 900  1500
 $EndSCHEMATC

Commit message: Removed gnd plane from under oscillator, added differential oscillator signal. Generated gerbers
Connections:
- net labels added: OSC_N, OSC_P
Changed lines of the file:
@@
 Wire Wire Line
 	1050 1500 900  1500
+Text Label 1950 1700 0    60   ~ 0
+OSC_P
+Text Label 2000 2250 0    60   ~ 0
+OSC_N
 $EndSCHEMATC
