File: OBC_prototypeA/bulk_power.sch (KiCad schematic (older format))
At the start: 39 parts, among them P1 3v3_IN_CONNECTOR, P2 INA_INPUT, P3 INA_GND, P4 INA_EN, P5 INA_OUTPUT, Q1 DMN2075U, Q2 DMN2075U, Q3 1v2_GOOD, U1 TMS570LS0714, U2 AP7331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

Commit message: Added 10k pot and removed R2 to allow current limit to be adjusted
Parts:
- removed R2: 10k, SFUSat:R_0402, symbol R
- added VR1: Trimpot, SFUSat:Trimpot_Bourns_TC33, symbol Trimpot
- R1: value 2k -> 7.5k

Commit message: Added FTDI FT230 and beefed up main 1v2 bus lines
Parts:
- R6: value 100 -> 270
Changed lines of the file:
@@
 	7800 4900 7800 5100
 $Comp
-L GND #PWR21
+L GND #PWR01
 U 1 1 595695D8
 P 7800 5450
-F 0 "#PWR21" H 7800 5200 50  0001 C CNN
+F 0 "#PWR01" H 7800 5200 50  0001 C CNN
 F 1 "GND" H 7800 5300 50  0000 C CNN
 F 2 "" H 7800 5450 50  0000 C CNN
@@
 $EndComp
 $Comp
-L +3V3 #PWR4
+L +3V3 #PWR02
 U 1 1 59569610
 P 1000 800
-F 0 "#PWR4" H 1000 650 50  0001 C CNN
+F 0 "#PWR02" H 1000 650 50  0001 C CNN
 F 1 "+3V3" H 1000 940 50  0000 C CNN
 F 2 "" H 1000 800 50  0000 C CNN
@@
 	1000 800  1000 900
 $Comp
-L +3V3 #PWR3
+L +3V3 #PWR03
 U 1 1 595697BF
 P 800 2250
-F 0 "#PWR3" H 800 2100 50  0001 C CNN
+F 0 "#PWR03" H 800 2100 50  0001 C CNN
 F 1 "+3V3" H 800 2390 50  0000 C CNN
 F 2 "" H 800 2250 50  0000 C CNN
@@
 $EndComp
 $Comp
-L GND #PWR6
+L GND #PWR04
 U 1 1 59569803
 P 1450 2800
-F 0 "#PWR6" H 1450 2550 50  0001 C CNN
+F 0 "#PWR04" H 1450 2550 50  0001 C CNN
 F 1 "GND" H 1450 2650 50  0000 C CNN
 F 2 "" H 1450 2800 50  0000 C CNN
@@
 	950  2250 800  2250
 $Comp
-L +1V2 #PWR23
+L +1V2 #PWR05
 U 1 1 595698EB
 P 8750 750
-F 0 "#PWR23" H 8750 600 50  0001 C CNN
+F 0 "#PWR05" H 8750 600 50  0001 C CNN
 F 1 "+1V2" H 8750 890 50  0000 C CNN
 F 2 "" H 8750 750 50  0000 C CNN
@@
 $EndComp
 $Comp
-L GND #PWR15
+L GND #PWR06
 U 1 1 595699CF
 P 6850 1500
-F 0 "#PWR15" H 6850 1250 50  0001 C CNN
+F 0 "#PWR06" H 6850 1250 50  0001 C CNN
 F 1 "GND" H 6850 1350 50  0000 C CNN
 F 2 "" H 6850 1500 50  0000 C CNN
@@
 Connection ~ 8500 850
 $Comp
-L +3V3 #PWR17
+L +3V3 #PWR07
 U 1 1 59569C16
 P 7100 800
-F 0 "#PWR17" H 7100 650 50  0001 C CNN
+F 0 "#PWR07" H 7100 650 50  0001 C CNN
 F 1 "+3V3" H 7100 940 50  0000 C CNN
 F 2 "" H 7100 800 50  0000 C CNN
@@
 $EndComp
 $Comp
-L GND #PWR2
+L GND #PWR08
 U 1 1 59569D86
 P 750 6650
-F 0 "#PWR2" H 750 6400 50  0001 C CNN
+F 0 "#PWR08" H 750 6400 50  0001 C CNN
 F 1 "GND" H 750 6500 50  0000 C CNN
 F 2 "" H 750 6650 50  0000 C CNN
@@
 $EndComp
 $Comp
-L GND #PWR7
+L GND #PWR09
 U 1 1 59569E21
 P 1950 6650
-F 0 "#PWR7" H 1950 6400 50  0001 C CNN
+F 0 "#PWR09" H 1950 6400 50  0001 C CNN
 F 1 "GND" H 1950 6500 50  0000 C CNN
 F 2 "" H 1950 6650 50  0000 C CNN
@@
 $EndComp
 $Comp
-L +1V2 #PWR11
+L +1V2 #PWR010
 U 1 1 59569E8C
 P 3250 6050
-F 0 "#PWR11" H 3250 5900 50  0001 C CNN
+F 0 "#PWR010" H 3250 5900 50  0001 C CNN
 F 1 "+1V2" H 3250 6190 50  0000 C CNN
 F 2 "" H 3250 6050 50  0000 C CNN
@@
 	3450 6050 3250 6050
 $Comp
-L +1V2 #PWR12
+L +1V2 #PWR011
 U 1 1 59569FC3
 P 4750 6050
-F 0 "#PWR12" H 4750 5900 50  0001 C CNN
+F 0 "#PWR011" H 4750 5900 50  0001 C CNN
 F 1 "+1V2" H 4750 6190 50  0000 C CNN
 F 2 "" H 4750 6050 50  0000 C CNN
@@
 	4600 6050 4750 6050
 $Comp
-L +3V3 #PWR13
+L +3V3 #PWR012
 U 1 1 5956A06D
 P 5300 5250
-F 0 "#PWR13" H 5300 5100 50  0001 C CNN
+F 0 "#PWR012" H 5300 5100 50  0001 C CNN
 F 1 "+3V3" H 5300 5390 50  0000 C CNN
 F 2 "" H 5300 5250 50  0000 C CNN
@@
 $EndComp
 $Comp
-L +3V3 #PWR16
+L +3V3 #PWR013
 U 1 1 5956A12A
 P 7050 5250
-F 0 "#PWR16" H 7050 5100 50  0001 C CNN
+F 0 "#PWR013" H 7050 5100 50  0001 C CNN
 F 1 "+3V3" H 7050 5390 50  0000 C CNN
 F 2 "" H 7050 5250 50  0000 C CNN
@@
 $EndComp
 $Comp
-L +3V3 #PWR20
+L +3V3 #PWR014
 U 1 1 5956A1DB
 P 7800 4900
-F 0 "#PWR20" H 7800 4750 50  0001 C CNN
+F 0 "#PWR014" H 7800 4750 50  0001 C CNN
 F 1 "+3V3" H 7800 5040 50  0000 C CNN
 F 2 "" H 7800 4900 50  0000 C CNN
@@
 	7350 5600 7350 5800
 $Comp
-L GND #PWR19
+L GND #PWR015
 U 1 1 5956A394
 P 7350 6150
-F 0 "#PWR19" H 7350 5900 50  0001 C CNN
+F 0 "#PWR015" H 7350 5900 50  0001 C CNN
 F 1 "GND" H 7350 6000 50  0000 C CNN
 F 2 "" H 7350 6150 50  0000 C CNN
@@
 $EndComp
 $Comp
-L +3V3 #PWR18
+L +3V3 #PWR016
 U 1 1 5956A39A
 P 7350 5600
-F 0 "#PWR18" H 7350 5450 50  0001 C CNN
+F 0 "#PWR016" H 7350 5450 50  0001 C CNN
 F 1 "+3V3" H 7350 5740 50  0000 C CNN
 F 2 "" H 7350 5600 50  0000 C CNN
@@
 	2750 6150 2750 6350
 $Comp
-L GND #PWR10
+L GND #PWR017
 U 1 1 5956A940
 P 2750 6700
-F 0 "#PWR10" H 2750 6450 50  0001 C CNN
+F 0 "#PWR017" H 2750 6450 50  0001 C CNN
 F 1 "GND" H 2750 6550 50  0000 C CNN
 F 2 "" H 2750 6700 50  0000 C CNN
@@
 5v0
 $Comp
-L +5V #PWR1
+L +5V #PWR018
 U 1 1 595699C9
 P 750 800
-F 0 "#PWR1" H 750 650 50  0001 C CNN
+F 0 "#PWR018" H 750 650 50  0001 C CNN
 F 1 "+5V" H 750 940 50  0000 C CNN
 F 2 "" H 750 800 50  0000 C CNN
@@
 $EndComp
 $Comp
-L GND #PWR22
+L GND #PWR019
 U 1 1 5956AAB6
 P 8500 1750
-F 0 "#PWR22" H 8500 1500 50  0001 C CNN
+F 0 "#PWR019" H 8500 1500 50  0001 C CNN
 F 1 "GND" H 8500 1600 50  0000 C CNN
 F 2 "" H 8500 1750 50  0000 C CNN
@@
 $EndComp
 $Comp
-L +5V #PWR8
+L +5V #PWR020
 U 1 1 5956AE0D
 P 2450 750
-F 0 "#PWR8" H 2450 600 50  0001 C CNN
+F 0 "#PWR020" H 2450 600 50  0001 C CNN
 F 1 "+5V" H 2450 890 50  0000 C CNN
 F 2 "" H 2450 750 50  0000 C CNN
@@
 	5300 2650 5750 2650
 $Comp
-L +3V3 #PWR14
+L +3V3 #PWR021
 U 1 1 595A8DFE
 P 5750 2650
-F 0 "#PWR14" H 5750 2500 50  0001 C CNN
+F 0 "#PWR021" H 5750 2500 50  0001 C CNN
 F 1 "+3V3" H 5750 2790 50  0000 C CNN
 F 2 "" H 5750 2650 50  0000 C CNN
@@
 3v3_OUTPUT
 $Comp
-L +3V3 #PWR5
+L +3V3 #PWR022
 U 1 1 595A95DC
 P 1150 3850
-F 0 "#PWR5" H 1150 3700 50  0001 C CNN
+F 0 "#PWR022" H 1150 3700 50  0001 C CNN
 F 1 "+3V3" H 1150 3990 50  0000 C CNN
 F 2 "" H 1150 3850 50  0000 C CNN
@@
 104_GND
 $Comp
-L GND #PWR25
+L GND #PWR023
 U 1 1 595B0A44
 P 10000 4050
-F 0 "#PWR25" H 10000 3800 50  0001 C CNN
+F 0 "#PWR023" H 10000 3800 50  0001 C CNN
 F 1 "GND" H 10000 3900 50  0000 C CNN
 F 2 "" H 10000 4050 50  0000 C CNN
@@
 P 10450 1550
 F 0 "R6" V 10530 1550 50  0000 C CNN
-F 1 "100" V 10450 1550 50  0000 C CNN
+F 1 "270" V 10450 1550 50  0000 C CNN
 F 2 "SFUSat:R_0402" V 10380 1550 50  0001 C CNN
 F 3 "" H 10450 1550 50  0000 C CNN
@@
 	10450 1700 10450 1800
 $Comp
-L +1V2 #PWR24
+L +1V2 #PWR024
 U 1 1 5965C95D
 P 9900 2550
-F 0 "#PWR24" H 9900 2400 50  0001 C CNN
+F 0 "#PWR024" H 9900 2400 50  0001 C CNN
 F 1 "+1V2" H 9900 2690 50  0000 C CNN
 F 2 "" H 9900 2550 50  0000 C CNN
@@
 $EndComp
 $Comp
-L GND #PWR26
+L GND #PWR025
 U 1 1 5965C9F5
 P 10250 3100
-F 0 "#PWR26" H 10250 2850 50  0001 C CNN
+F 0 "#PWR025" H 10250 2850 50  0001 C CNN
 F 1 "GND" H 10250 2950 50  0000 C CNN
 F 2 "" H 10250 3100 50  0000 C CNN
@@
 $EndComp
 $Comp
-L +3V3 #PWR27
+L +3V3 #PWR026
 U 1 1 5965CA8D
 P 10450 1250
-F 0 "#PWR27" H 10450 1100 50  0001 C CNN
+F 0 "#PWR026" H 10450 1100 50  0001 C CNN
 F 1 "+3V3" H 10450 1390 50  0000 C CNN
 F 2 "" H 10450 1250 50  0000 C CNN
@@
 Connection ~ 9900 2600
 $Comp
-L +1V2 #PWR9
+L +1V2 #PWR027
 U 1 1 59725D84
 P 2750 6150
-F 0 "#PWR9" H 2750 6000 50  0001 C CNN
+F 0 "#PWR027" H 2750 6000 50  0001 C CNN
 F 1 "+1V2" H 2750 6290 50  0000 C CNN
 F 2 "" H 2750 6150 50  0000 C CNN

Commit message: Changed 1.2V regulator from AP7331 to XC6222B121MR-G because the 7331 current limit is too low. Also changed C2 from 1µF to 10µF to meet requirements for new regulator
Parts:
- C2: value 1uF -> 10µF
- U2: value AP7331 -> XC6222B121MR-G
Changed lines of the file:
@@
 P 7700 1200
 F 0 "U2" H 7700 1100 60  0000 C CNN
-F 1 "AP7331" H 7700 1450 60  0000 C CNN
+F 1 "XC6222B121MR-G" H 7700 1450 60  0000 C CNN
 F 2 "SFUSat:SOT25" H 7700 1100 60  0001 C CNN
 F 3 "" H 7700 1100 60  0001 C CNN
@@
 P 8500 1350
 F 0 "C2" H 8525 1450 50  0000 L CNN
-F 1 "1uF" H 8525 1250 50  0000 L CNN
+F 1 "10µF" H 8525 1250 50  0000 L CNN
 F 2 "SFUSat:C_0402" H 8538 1200 50  0001 C CNN
 F 3 "" H 8500 1350 50  0000 C CNN
