File: OBC_prototypeB_04/PC104_Connector.sch (KiCad schematic (older format))
At the start: 18 parts, among them J1 PC104-8BIT, P11 USB_5V, P6 USB_PORT, Q4 DMN2075U, U10 FT230XQ-R

Commit message: Connected A7 to ANTENNA_DEPLOY
placed DIP switch
added labels in 104 connector describing GPIO functtionality
Other:
- note added: "GIOA7"
- note added: "RF_Deploy"
- note added: "RF_Deploy\n"
Changed lines of the file:
@@
 Text Label 1800 6300 0    60   ~ 0
 RUSB_P
+Text Notes 9600 2000 0    60   ~ 0
+RF_Deploy
+Text Notes 9600 2150 0    60   ~ 0
+RF_Deploy\n
+Text Notes 4100 1950 0    60   ~ 0
+GIOA7
 $EndSCHEMATC

Commit message: Made GPIO reroutes
	B1: is now RTC alert, also on 104 connector
	A0, A2: labelled as RF_deploy on 104 connector (no routing change)
	A5: RF_IRQ
	A7: ANTENNA_DEPLOY
Other:
- note added: "GIOA5 - Support Reset, CLK Section"
- note added: "RTC_INT\n"
Changed lines of the file:
@@
 Text Notes 9600 2000 0    60   ~ 0
 RF_Deploy
-Text Notes 9600 2150 0    60   ~ 0
+Text Notes 9600 2300 0    60   ~ 0
 RF_Deploy\n
 Text Notes 4100 1950 0    60   ~ 0
 GIOA7
+Text Notes 4800 1550 2    60   ~ 0
+GIOA5 - Support Reset, CLK Section
+Text Notes 9950 2450 2    60   ~ 0
+RTC_INT\n
 $EndSCHEMATC

Commit message: Added labels to all GPIO on 104/chip
Also added sun sensor ADC to 104 connector
Connections:
- net labels added: AD1_17, AD1_18, AD1_19, AD1_20
- wire segments 178 -> 194
Other:
- note added: "ANTENNA_ADC"
- note added: "HEAT_ADC"
- note added: "RF.ADC3"
- note added: "RF.ADC4\n"
- note added: "RF.ADC5\n"
- note added: "SENS_ADC"
- note added: "Sun Sensors"

Commit message: Added DC in jack for charging
Also added labels to ADC and GPIO
Parts:
- added P15: 3pin-DC-power, SFUSat:PJ-028-SMT-TR-3pin-DC-jack PJ-028-SMT-TR, symbol 3pin-DC-power
Connections:
- wire segments 194 -> 206

Commit message: Added USB B connector
Parts:
- P6: footprint SFUSat:USB_MINIB_SMD -> SFUSat:USB_B_through
Changed lines of the file:
@@
 F 0 "P6" H 8700 5850 60  0000 C CNN
 F 1 "USB_PORT" H 8250 6050 60  0000 C CNN
-F 2 "SFUSat:USB_MINIB_SMD" H 8250 5750 60  0001 C CNN
+F 2 "SFUSat:USB_B_through" H 8250 5750 60  0001 C CNN
 F 3 "" H 8250 5750 60  0001 C CNN
 	1    8250 5750

Commit message: Removed trimpot
Parts:
- P6: footprint SFUSat:USB_B_through -> SFUSat:USB_MINIB_SMD
Changed lines of the file:
@@
 LIBS:valves
 LIBS:SFUSat
-LIBS:OBC_04-cache
 EELAYER 25 0
 EELAYER END
@@
 F 0 "P6" H 8700 5850 60  0000 C CNN
 F 1 "USB_PORT" H 8250 6050 60  0000 C CNN
-F 2 "SFUSat:USB_B_through" H 8250 5750 60  0001 C CNN
+F 2 "SFUSat:USB_MINIB_SMD" H 8250 5750 60  0001 C CNN
 F 3 "" H 8250 5750 60  0001 C CNN
 	1    8250 5750
