File: OBC_prototypeB_04/RTC.sch (KiCad schematic (older format))
At the start: 7 parts, among them P8 RTC_SPI, U8 AB-RTCMC-EOA9-S3

Commit message: Made GPIO reroutes
	B1: is now RTC alert, also on 104 connector
	A0, A2: labelled as RF_deploy on 104 connector (no routing change)
	A5: RF_IRQ
	A7: ANTENNA_DEPLOY
Connections:
- net labels added: GIOB1
- wire segments 21 -> 24
Changed lines of the file:
@@
 Wire Wire Line
 	1400 2650 1400 2800
+Text GLabel 4800 2800 3    60   Input ~ 0
+GIOB1
+Wire Wire Line
+	4450 2300 4450 2400
+Wire Wire Line
+	4450 2400 4800 2400
+Wire Wire Line
+	4800 2400 4800 2800
 $EndSCHEMATC
