File: OBC_prototypeB_04/GPIO.sch (KiCad schematic (older format))
At the start: 7 parts, among them Q5 DMN2075U, U1 TMS570LS0714

Commit message: Connected A7 to ANTENNA_DEPLOY
placed DIP switch
added labels in 104 connector describing GPIO functtionality
Parts:
- added SW3: DIPSW_218-4LPST, symbol DIPSW_218-4LPST
Connections:
- net labels added: ANTENNA_DEPLOY
- net labels removed: GIOA7
Changed lines of the file:
@@
 L TMS570LS0714 U1
 U 1 1 5965E8A7
-P 7900 2850
-F 0 "U1" H 8300 3400 60  0000 C CNN
-F 1 "TMS570LS0714" H 7850 3400 60  0000 C CNN
-F 2 "Housings_QFP:LQFP-144_20x20mm_Pitch0.5mm" H 5500 1600 60  0001 C CNN
-F 3 "" H 5500 1600 60  0001 C CNN
-	1    7900 2850
+P 6550 2200
+F 0 "U1" H 6950 2750 60  0000 C CNN
+F 1 "TMS570LS0714" H 6500 2750 60  0000 C CNN
+F 2 "Housings_QFP:LQFP-144_20x20mm_Pitch0.5mm" H 4150 950 60  0001 C CNN
+F 3 "" H 4150 950 60  0001 C CNN
+	1    6550 2200
 	1    0    0    -1
 $EndComp
@@
 L DMN2075U Q5
 U 1 1 5965E8EF
-P 3950 3450
-F 0 "Q5" V 3650 3350 60  0000 C CNN
-F 1 "DMN2075U" H 4250 3600 60  0000 C CNN
-F 2 "SFUSat:SOT23_DMN2075U" V 3650 3350 60  0001 C CNN
-F 3 "" V 3650 3350 60  0001 C CNN
-	1    3950 3450
+P 2600 2800
+F 0 "Q5" V 2300 2700 60  0000 C CNN
+F 1 "DMN2075U" H 2900 2950 60  0000 C CNN
+F 2 "SFUSat:SOT23_DMN2075U" V 2300 2700 60  0001 C CNN
+F 3 "" V 2300 2700 60  0001 C CNN
+	1    2600 2800
 	1    0    0    -1
 $EndComp
@@
 L LED D3
 U 1 1 5965E90A
-P 3950 2850
-F 0 "D3" H 3950 2950 50  0000 C CNN
-F 1 "LED" H 3950 2750 50  0000 C CNN
-F 2 "SFUSat:LED_0603" H 3950 2850 50  0001 C CNN
-F 3 "" H 3950 2850 50  0000 C CNN
-	1    3950 2850
+P 2600 2200
+F 0 "D3" H 2600 2300 50  0000 C CNN
+F 1 "LED" H 2600 2100 50  0000 C CNN
+F 2 "SFUSat:LED_0603" H 2600 2200 50  0001 C CNN
+F 3 "" H 2600 2200 50  0000 C CNN
+	1    2600 2200
 	0    -1   -1   0
 $EndComp
@@
 L R R9
 U 1 1 5965E94A
-P 3950 2400
-F 0 "R9" V 4030 2400 50  0000 C CNN
-F 1 "270" V 3950 2400 50  0000 C CNN
-F 2 "SFUSat:R_0402" V 3880 2400 50  0001 C CNN
-F 3 "" H 3950 2400 50  0000 C CNN
-	1    3950 2400
+P 2600 1750
+F 0 "R9" V 2680 1750 50  0000 C CNN
+F 1 "270" V 2600 1750 50  0000 C CNN
+F 2 "SFUSat:R_0402" V 2530 1750 50  0001 C CNN
+F 3 "" H 2600 1750 50  0000 C CNN
+	1    2600 1750
 	1    0    0    -1
 $EndComp
@@
 L R R8
 U 1 1 5965EB3A
-P 3450 3750
-F 0 "R8" V 3550 3750 50  0000 C CNN
-F 1 "10k" V 3450 3750 50  0000 C CNN
-F 2 "SFUSat:R_0402" V 3380 3750 50  0001 C CNN
-F 3 "" H 3450 3750 50  0000 C CNN
-	1    3450 3750
-	1    0    0    -1
-$EndComp
-Text GLabel 6950 2950 0    60   Input ~ 0
+P 2100 3100
+F 0 "R8" V 2200 3100 50  0000 C CNN
+F 1 "10k" V 2100 3100 50  0000 C CNN
+F 2 "SFUSat:R_0402" V 2030 3100 50  0001 C CNN
+F 3 "" H 2100 3100 50  0000 C CNN
+	1    2100 3100
+	1    0    0    -1
+$EndComp
+Text GLabel 5600 2300 0    60   Input ~ 0
 GIOA6
-Text GLabel 3300 3450 0    60   Input ~ 0
+Text GLabel 1950 2800 0    60   Input ~ 0
 GIOA6
 $Comp
-L +3V3 #PWR59
+L +3V3 #PWR61
 U 1 1 5965EBB1
-P 3950 2100
-F 0 "#PWR59" H 3950 1950 50  0001 C CNN
-F 1 "+3V3" H 3950 2240 50  0000 C CNN
-F 2 "" H 3950 2100 50  0000 C CNN
-F 3 "" H 3950 2100 50  0000 C CNN
-	1    3950 2100
-	1    0    0    -1
-$EndComp
-$Comp
-L GND #PWR58
+P 2600 1450
+F 0 "#PWR61" H 2600 1300 50  0001 C CNN
+F 1 "+3V3" H 2600 1590 50  0000 C CNN
+F 2 "" H 2600 1450 50  0000 C CNN
+F 3 "" H 2600 1450 50  0000 C CNN
+	1    2600 1450
+	1    0    0    -1
+$EndComp
+$Comp
+L GND #PWR60
 U 1 1 5965EBE8
-P 3750 3900
-F 0 "#PWR58" H 3750 3650 50  0001 C CNN
-F 1 "GND" H 3750 3750 50  0000 C CNN
-F 2 "" H 3750 3900 50  0000 C CNN
-F 3 "" H 3750 3900 50  0000 C CNN
-	1    3750 3900
-	1    0    0    -1
-$EndComp
-Wire Wire Line
-	3950 2550 3950 2650
-Wire Wire Line
-	3950 3050 3950 3150
-Wire Wire Line
-	3300 3450 3550 3450
-Wire Wire Line
-	3450 3600 3450 3450
-Connection ~ 3450 3450
-Wire Wire Line
-	3450 3900 3950 3900
-Wire Wire Line
-	3950 3900 3950 3750
-Connection ~ 3750 3900
-Wire Wire Line
-	3950 2100 3950 2250
-Text Notes 2950 1800 0    60   ~ 0
+P 2400 3250
+F 0 "#PWR60" H 2400 3000 50  0001 C CNN
+F 1 "GND" H 2400 3100 50  0000 C CNN
+F 2 "" H 2400 3250 50  0000 C CNN
+F 3 "" H 2400 3250 50  0000 C CNN
+	1    2400 3250
+	1    0    0    -1
+$EndComp
+Wire Wire Line
+	2600 1900 2600 2000
+Wire Wire Line
+	2600 2400 2600 2500
+Wire Wire Line
+	1950 2800 2200 2800
+Wire Wire Line
+	2100 2950 2100 2800
+Connection ~ 2100 2800
+Wire Wire Line
+	2100 3250 2600 3250
+Wire Wire Line
+	2600 3250 2600 3100
+Connection ~ 2400 3250
+Wire Wire Line
+	2600 1450 2600 1600
+Text Notes 1600 1150 0    60   ~ 0
 "Pin 16 LED" - for blinky debug\n
 Wire Wire Line
-	7100 2950 6950 2950
+	5750 2300 5600 2300
 Text GLabel 8500 1100 0    60   Input ~ 0
 3v3
 $Comp
-L +3V3 #PWR61
+L +3V3 #PWR63
 U 1 1 5967FAD1
 P 8800 1100
-F 0 "#PWR61" H 8800 950 50  0001 C CNN
+F 0 "#PWR63" H 8800 950 50  0001 C CNN
 F 1 "+3V3" H 8800 1240 50  0000 C CNN
 F 2 "" H 8800 1100 50  0000 C CNN
@@
 Wire Wire Line
 	8500 1100 8800 1100
-Text GLabel 5600 3250 0    60   Input ~ 0
+Text GLabel 4250 2600 0    60   Input ~ 0
 WATCHDOG
 Wire Wire Line
-	5600 3250 7100 3250
+	4250 2600 5750 2600
 $Comp
 L R R26
 U 1 1 59711F3A
-P 5750 3450
-F 0 "R26" V 5830 3450 50  0000 C CNN
-F 1 "10k" V 5750 3450 50  0000 C CNN
-F 2 "SFUSat:R_0402" V 5680 3450 50  0001 C CNN
-F 3 "" H 5750 3450 50  0000 C CNN
-	1    5750 3450
-	1    0    0    -1
-$EndComp
-$Comp
-L GND #PWR60
+P 4400 2800
+F 0 "R26" V 4480 2800 50  0000 C CNN
+F 1 "10k" V 4400 2800 50  0000 C CNN
+F 2 "SFUSat:R_0402" V 4330 2800 50  0001 C CNN
+F 3 "" H 4400 2800 50  0000 C CNN
+	1    4400 2800
+	1    0    0    -1
+$EndComp
+$Comp
+L GND #PWR62
 U 1 1 59711F64
-P 5750 3700
-F 0 "#PWR60" H 5750 3450 50  0001 C CNN
-F 1 "GND" H 5750 3550 50  0000 C CNN
-F 2 "" H 5750 3700 50  0000 C CNN
-F 3 "" H 5750 3700 50  0000 C CNN
-	1    5750 3700
-	1    0    0    -1
-$EndComp
-Wire Wire Line
-	5750 3300 5750 3250
-Connection ~ 5750 3250
-Wire Wire Line
-	5750 3600 5750 3700
+P 4400 3050
+F 0 "#PWR62" H 4400 2800 50  0001 C CNN
+F 1 "GND" H 4400 2900 50  0000 C CNN
+F 2 "" H 4400 3050 50  0000 C CNN
+F 3 "" H 4400 3050 50  0000 C CNN
+	1    4400 3050
+	1    0    0    -1
+$EndComp
+Wire Wire Line
+	4400 2650 4400 2600
+Connection ~ 4400 2600
+Wire Wire Line
+	4400 2950 4400 3050
 $Comp
 L TEST_1P W13
 U 1 1 59714601
-P 6050 3300
-F 0 "W13" H 6050 3570 50  0000 C CNN
-F 1 "WD_TEST" H 6050 3500 50  0000 C CNN
-F 2 "SFUSat:Test_Point" H 6250 3300 50  0001 C CNN
-F 3 "" H 6250 3300 50  0000 C CNN
-	1    6050 3300
+P 4700 2650
+F 0 "W13" H 4700 2920 50  0000 C CNN
+F 1 "WD_TEST" H 4700 2850 50  0000 C CNN
+F 2 "SFUSat:Test_Point" H 4900 2650 50  0001 C CNN
+F 3 "" H 4900 2650 50  0000 C CNN
+	1    4700 2650
 	-1   0    0    1
 $EndComp
 Wire Wire Line
-	6050 3300 6050 3250
-Connection ~ 6050 3250
-Text GLabel 6950 2500 0    60   Input ~ 0
+	4700 2650 4700 2600
+Connection ~ 4700 2600
+Text GLabel 5600 1850 0    60   Input ~ 0
 GIOA0
-Text GLabel 6950 2650 0    60   Input ~ 0
+Text GLabel 5600 2000 0    60   Input ~ 0
 GIOA1
-Text GLabel 6950 2800 0    60   Input ~ 0
+Text GLabel 5600 2150 0    60   Input ~ 0
 GIOA2
 Wire Wire Line
-	6950 2500 7100 2500
-Wire Wire Line
-	6950 2650 7100 2650
-Wire Wire Line
-	6950 2800 7100 2800
-Text GLabel 6950 3100 0    60   Input ~ 0
-GIOA7
-Wire Wire Line
-	6950 3100 7100 3100
-Text GLabel 6900 3400 0    60   Input ~ 0
+	5600 1850 5750 1850
+Wire Wire Line
+	5600 2000 5750 2000
+Wire Wire Line
+	5600 2150 5750 2150
+Text GLabel 5600 2450 0    60   Input ~ 0
+ANTENNA_DEPLOY
+Wire Wire Line
+	5600 2450 5750 2450
+Text GLabel 5550 2750 0    60   Input ~ 0
 GIOB1
-Text GLabel 6900 3550 0    60   Input ~ 0
+Text GLabel 5550 2900 0    60   Input ~ 0
 GIOB2
-Text GLabel 6900 3700 0    60   Input ~ 0
+Text GLabel 5550 3050 0    60   Input ~ 0
 GIOB3
 Wire Wire Line
-	7100 3400 6900 3400
-Wire Wire Line
-	6900 3550 7100 3550
-Wire Wire Line
-	6900 3700 7100 3700
+	5750 2750 5550 2750
+Wire Wire Line
+	5550 2900 5750 2900
+Wire Wire Line
+	5550 3050 5750 3050
+$Comp
+L DIPSW_218-4LPST SW3
+U 1 1 5A52C1FE
+P 3700 4650
+F 0 "SW3" H 3550 4250 60  0000 C CNN
+F 1 "DIPSW_218-4LPST" H 3600 5050 60  0000 C CNN
+F 2 "" H 3700 4650 60  0001 C CNN
+F 3 "" H 3700 4650 60  0001 C CNN
+	1    3700 4650
+	1    0    0    -1
+$EndComp
 $EndSCHEMATC

Commit message: Made GPIO reroutes
	B1: is now RTC alert, also on 104 connector
	A0, A2: labelled as RF_deploy on 104 connector (no routing change)
	A5: RF_IRQ
	A7: ANTENNA_DEPLOY
Other:
- note added: "RTC_INT"
Changed lines of the file:
@@
 	1    0    0    -1
 $EndComp
+Text Notes 5150 2800 2    60   ~ 0
+RTC_INT
 $EndSCHEMATC

Commit message: Changed RESET circuitry
Added jumper to disconnect WD from MASTER_RESET
Changed SW1 name to "Hard reset via WD"
Added SW4 - direct connect (not via WD) to MCU. Enables manual hard reset with WD disabled.
Parts:
- SW3: footprint (none) -> SFUSat:LPST218-4
Changed lines of the file:
@@
 GIOA6
 $Comp
-L +3V3 #PWR61
+L +3V3 #PWR63
 U 1 1 5965EBB1
 P 2600 1450
-F 0 "#PWR61" H 2600 1300 50  0001 C CNN
+F 0 "#PWR63" H 2600 1300 50  0001 C CNN
 F 1 "+3V3" H 2600 1590 50  0000 C CNN
 F 2 "" H 2600 1450 50  0000 C CNN
@@
 $EndComp
 $Comp
-L GND #PWR60
+L GND #PWR62
 U 1 1 5965EBE8
 P 2400 3250
-F 0 "#PWR60" H 2400 3000 50  0001 C CNN
+F 0 "#PWR62" H 2400 3000 50  0001 C CNN
 F 1 "GND" H 2400 3100 50  0000 C CNN
 F 2 "" H 2400 3250 50  0000 C CNN
@@
 3v3
 $Comp
-L +3V3 #PWR63
+L +3V3 #PWR65
 U 1 1 5967FAD1
 P 8800 1100
-F 0 "#PWR63" H 8800 950 50  0001 C CNN
+F 0 "#PWR65" H 8800 950 50  0001 C CNN
 F 1 "+3V3" H 8800 1240 50  0000 C CNN
 F 2 "" H 8800 1100 50  0000 C CNN
@@
 $EndComp
 $Comp
-L GND #PWR62
+L GND #PWR64
 U 1 1 59711F64
 P 4400 3050
-F 0 "#PWR62" H 4400 2800 50  0001 C CNN
+F 0 "#PWR64" H 4400 2800 50  0001 C CNN
 F 1 "GND" H 4400 2900 50  0000 C CNN
 F 2 "" H 4400 3050 50  0000 C CNN
@@
 F 0 "SW3" H 3550 4250 60  0000 C CNN
 F 1 "DIPSW_218-4LPST" H 3600 5050 60  0000 C CNN
-F 2 "" H 3700 4650 60  0001 C CNN
+F 2 "SFUSat:LPST218-4" H 3700 4650 60  0001 C CNN
 F 3 "" H 3700 4650 60  0001 C CNN
 	1    3700 4650

Commit message: WIP initial placement
Parts:
- removed SW3: DIPSW_218-4LPST, SFUSat:LPST218-4, symbol DIPSW_218-4LPST
Changed lines of the file:
@@
 GIOA6
 $Comp
-L +3V3 #PWR63
+L +3V3 #PWR064
 U 1 1 5965EBB1
 P 2600 1450
-F 0 "#PWR63" H 2600 1300 50  0001 C CNN
+F 0 "#PWR064" H 2600 1300 50  0001 C CNN
 F 1 "+3V3" H 2600 1590 50  0000 C CNN
 F 2 "" H 2600 1450 50  0000 C CNN
@@
 $EndComp
 $Comp
-L GND #PWR62
+L GND #PWR065
 U 1 1 5965EBE8
 P 2400 3250
-F 0 "#PWR62" H 2400 3000 50  0001 C CNN
+F 0 "#PWR065" H 2400 3000 50  0001 C CNN
 F 1 "GND" H 2400 3100 50  0000 C CNN
 F 2 "" H 2400 3250 50  0000 C CNN
@@
 3v3
 $Comp
-L +3V3 #PWR65
+L +3V3 #PWR066
 U 1 1 5967FAD1
 P 8800 1100
-F 0 "#PWR65" H 8800 950 50  0001 C CNN
+F 0 "#PWR066" H 8800 950 50  0001 C CNN
 F 1 "+3V3" H 8800 1240 50  0000 C CNN
 F 2 "" H 8800 1100 50  0000 C CNN
@@
 $EndComp
 $Comp
-L GND #PWR64
+L GND #PWR067
 U 1 1 59711F64
 P 4400 3050
-F 0 "#PWR64" H 4400 2800 50  0001 C CNN
+F 0 "#PWR067" H 4400 2800 50  0001 C CNN
 F 1 "GND" H 4400 2900 50  0000 C CNN
 F 2 "" H 4400 3050 50  0000 C CNN
@@
 Wire Wire Line
 	5550 3050 5750 3050
-$Comp
-L DIPSW_218-4LPST SW3
-U 1 1 5A52C1FE
-P 3700 4650
-F 0 "SW3" H 3550 4250 60  0000 C CNN
-F 1 "DIPSW_218-4LPST" H 3600 5050 60  0000 C CNN
-F 2 "SFUSat:LPST218-4" H 3700 4650 60  0001 C CNN
-F 3 "" H 3700 4650 60  0001 C CNN
-	1    3700 4650
-	1    0    0    -1
-$EndComp
 Text Notes 5150 2800 2    60   ~ 0
 RTC_INT

Commit message: Added labels to all GPIO on 104/chip
Also added sun sensor ADC to 104 connector
Other:
- note added: "BLINKY"
- note added: "RF.DEPLOY"
Changed lines of the file:
@@
 Text Notes 5150 2800 2    60   ~ 0
 RTC_INT
+Text Notes 4750 1900 0    60   ~ 0
+RF.DEPLOY
+Text Notes 4750 2200 0    60   ~ 0
+RF.DEPLOY
+Text Notes 4900 2350 0    60   ~ 0
+BLINKY
 $EndSCHEMATC

Commit message: Removed GIOA6 pulldown
Parts:
- removed R8: 10k, SFUSat:R_0402, symbol R
Connections:
- wire segments 20 -> 19
Changed lines of the file:
@@
-	1    0    0    -1
-$EndComp
-$Comp
-L R R8
-U 1 1 5965EB3A
-P 2100 3100
-F 0 "R8" V 2200 3100 50  0000 C CNN
-F 1 "10k" V 2100 3100 50  0000 C CNN
-F 2 "SFUSat:R_0402" V 2030 3100 50  0001 C CNN
-F 3 "" H 2100 3100 50  0000 C CNN
-	1    2100 3100
 	1    0    0    -1
 $EndComp
@@
 	1950 2800 2200 2800
 Wire Wire Line
-	2100 2950 2100 2800
-Connection ~ 2100 2800
-Wire Wire Line
-	2100 3250 2600 3250
-Wire Wire Line
 	2600 3250 2600 3100
-Connection ~ 2400 3250
 Wire Wire Line
 	2600 1450 2600 1600
@@
 Text Notes 4900 2350 0    60   ~ 0
 BLINKY
+Wire Wire Line
+	2400 3250 2600 3250
 $EndSCHEMATC
