File: OBC_prototypeB_04/ADC.sch (KiCad schematic (older format))
At the start: 4 parts, among them U1 TMS570LS0714

Commit message: Added DC in jack for charging
Also added labels to ADC and GPIO
Connections:
- net labels added: AD1_11, AD1_12, AD1_13, AD1_14, AD1_15, AD1_16, AD1_17, AD1_18, AD1_19, AD1_20, AD1_21, AD1_22, AD1_23
- wire segments 39 -> 78
Changed lines of the file:
@@
 L R R7
 U 1 1 595F3B4E
-P 1850 2900
-F 0 "R7" V 1930 2900 50  0000 C CNN
-F 1 "10k" V 1850 2900 50  0000 C CNN
-F 2 "SFUSat:R_0402" V 1780 2900 50  0001 C CNN
-F 3 "" H 1850 2900 50  0000 C CNN
-	1    1850 2900
-	1    0    0    -1
-$EndComp
-Text GLabel 1850 3150 3    60   Input ~ 0
+P 1200 2900
+F 0 "R7" V 1280 2900 50  0000 C CNN
+F 1 "10k" V 1200 2900 50  0000 C CNN
+F 2 "SFUSat:R_0402" V 1130 2900 50  0001 C CNN
+F 3 "" H 1200 2900 50  0000 C CNN
+	1    1200 2900
+	1    0    0    -1
+$EndComp
+Text GLabel 1200 3150 3    60   Input ~ 0
 104_GND
-Text GLabel 1650 2700 0    60   Input ~ 0
+Text GLabel 1000 2700 0    60   Input ~ 0
 INA_OUT
 Wire Wire Line
-	1650 2700 3450 2700
-Wire Wire Line
-	1850 2700 1850 2750
-Connection ~ 1850 2700
-Wire Wire Line
-	1850 3050 1850 3150
+	1000 2700 3450 2700
+Wire Wire Line
+	1200 2700 1200 2750
+Connection ~ 1200 2700
+Wire Wire Line
+	1200 3050 1200 3150
 Text GLabel 4500 1050 0    60   Input ~ 0
 3v3
 $Comp
-L +3V3 #PWR060
+L +3V3 #PWR058
 U 1 1 59681373
 P 4650 1050
-F 0 "#PWR060" H 4650 900 50  0001 C CNN
+F 0 "#PWR058" H 4650 900 50  0001 C CNN
 F 1 "+3V3" H 4650 1190 50  0000 C CNN
 F 2 "" H 4650 1050 50  0000 C CNN
@@
 	4500 1050 4650 1050
 $Comp
-L +3V3 #PWR061
+L +3V3 #PWR059
 U 1 1 596815A0
 P 3300 1750
-F 0 "#PWR061" H 3300 1600 50  0001 C CNN
+F 0 "#PWR059" H 3300 1600 50  0001 C CNN
 F 1 "+3V3" H 3300 1890 50  0000 C CNN
 F 2 "" H 3300 1750 50  0000 C CNN
@@
 $EndComp
 $Comp
-L +3V3 #PWR062
+L +3V3 #PWR060
 U 1 1 596815BA
 P 2550 2100
-F 0 "#PWR062" H 2550 1950 50  0001 C CNN
+F 0 "#PWR060" H 2550 1950 50  0001 C CNN
 F 1 "+3V3" H 2550 2240 50  0000 C CNN
 F 2 "" H 2550 2100 50  0000 C CNN
@@
 $EndComp
 $Comp
-L GND #PWR063
+L GND #PWR061
 U 1 1 596815EE
 P 2900 2000
-F 0 "#PWR063" H 2900 1750 50  0001 C CNN
+F 0 "#PWR061" H 2900 1750 50  0001 C CNN
 F 1 "GND" H 2900 2100 50  0000 C CNN
 F 2 "" H 2900 2000 50  0000 C CNN
@@
 Wire Wire Line
 	2350 2300 3450 2300
-Text GLabel 2500 2800 0    60   Input ~ 0
+Text GLabel 2050 2800 0    60   Input ~ 0
 AD1_3
 Wire Wire Line
-	3450 2800 2500 2800
-Text GLabel 2500 2950 0    60   Input ~ 0
+	2050 2800 3450 2800
+Text GLabel 2050 2950 0    60   Input ~ 0
 AD1_4
-Text GLabel 2500 3100 0    60   Input ~ 0
+Text GLabel 2050 3100 0    60   Input ~ 0
 AD1_5
-Text GLabel 2500 3250 0    60   Input ~ 0
+Text GLabel 2050 3250 0    60   Input ~ 0
 AD1_6
-Text GLabel 2500 3400 0    60   Input ~ 0
+Text GLabel 2050 3400 0    60   Input ~ 0
 AD1_7
-Text GLabel 2500 3550 0    60   Input ~ 0
+Text GLabel 2050 3550 0    60   Input ~ 0
 AD1_8
-Text GLabel 2500 3700 0    60   Input ~ 0
+Text GLabel 2050 3700 0    60   Input ~ 0
 AD1_9
-Text GLabel 2500 3850 0    60   Input ~ 0
+Text GLabel 2050 3850 0    60   Input ~ 0
 AD1_10
 Wire Wire Line
-	2500 2950 2550 2950
-Wire Wire Line
-	2550 2950 2550 2900
-Wire Wire Line
-	2550 2900 3450 2900
-Wire Wire Line
-	3450 3000 2550 3000
-Wire Wire Line
-	2550 3000 2550 3100
-Wire Wire Line
-	2550 3100 2500 3100
-Wire Wire Line
-	2500 3250 2600 3250
-Wire Wire Line
-	2600 3250 2600 3100
-Wire Wire Line
-	2600 3100 3450 3100
-Wire Wire Line
-	2500 3400 2650 3400
-Wire Wire Line
-	2650 3400 2650 3200
-Wire Wire Line
-	2650 3200 3450 3200
-Wire Wire Line
-	2500 3550 2700 3550
-Wire Wire Line
-	2700 3550 2700 3300
-Wire Wire Line
-	2700 3300 3450 3300
-Wire Wire Line
-	2500 3700 2750 3700
-Wire Wire Line
-	2750 3700 2750 3400
-Wire Wire Line
-	2750 3400 3450 3400
-Wire Wire Line
-	2500 3850 2800 3850
-Wire Wire Line
-	2800 3850 2800 3500
-Wire Wire Line
-	2800 3500 3450 3500
+	2050 2950 2100 2950
+Wire Wire Line
+	2100 2950 2100 2900
+Wire Wire Line
+	2100 2900 3450 2900
+Wire Wire Line
+	2100 3000 3450 3000
+Wire Wire Line
+	2100 3000 2100 3100
+Wire Wire Line
+	2100 3100 2050 3100
+Wire Wire Line
+	2050 3250 2150 3250
+Wire Wire Line
+	2150 3250 2150 3100
+Wire Wire Line
+	2150 3100 3450 3100
+Wire Wire Line
+	2050 3400 2200 3400
+Wire Wire Line
+	2200 3400 2200 3200
+Wire Wire Line
+	2200 3200 3450 3200
+Wire Wire Line
+	2050 3550 2250 3550
+Wire Wire Line
+	2250 3550 2250 3300
+Wire Wire Line
+	2250 3300 3450 3300
+Wire Wire Line
+	2050 3700 2300 3700
+Wire Wire Line
+	2300 3700 2300 3400
+Wire Wire Line
+	2300 3400 3450 3400
+Wire Wire Line
+	2050 3850 2350 3850
+Wire Wire Line
+	2350 3850 2350 3500
+Wire Wire Line
+	2350 3500 3450 3500
+Text GLabel 2050 4000 0    60   Input ~ 0
+AD1_11
+Text GLabel 2050 4150 0    60   Input ~ 0
+AD1_12
+Text GLabel 2050 4300 0    60   Input ~ 0
+AD1_13
+Text GLabel 2050 4450 0    60   Input ~ 0
+AD1_14
+Text GLabel 2050 4600 0    60   Input ~ 0
+AD1_15
+Text GLabel 2050 4750 0    60   Input ~ 0
+AD1_16
+Text GLabel 2050 4900 0    60   Input ~ 0
+AD1_17
+Text GLabel 2050 5050 0    60   Input ~ 0
+AD1_18
+Text GLabel 2050 5200 0    60   Input ~ 0
+AD1_19
+Text GLabel 2050 5350 0    60   Input ~ 0
+AD1_20
+Text GLabel 2050 5500 0    60   Input ~ 0
+AD1_21
+Text GLabel 2050 5650 0    60   Input ~ 0
+AD1_22
+Text GLabel 2050 5800 0    60   Input ~ 0
+AD1_23
+Wire Wire Line
+	2050 4000 2400 4000
+Wire Wire Line
+	2400 4000 2400 3600
+Wire Wire Line
+	2400 3600 3450 3600
+Wire Wire Line
+	2050 4150 2450 4150
+Wire Wire Line
+	2450 4150 2450 3700
+Wire Wire Line
+	2450 3700 3450 3700
+Wire Wire Line
+	2500 3800 3450 3800
+Wire Wire Line
+	2500 3800 2500 4300
+Wire Wire Line
+	2500 4300 2050 4300
+Wire Wire Line
+	2050 4450 2550 4450
+Wire Wire Line
+	2550 4450 2550 3900
+Wire Wire Line
+	2550 3900 3450 3900
+Wire Wire Line
+	2050 4600 2600 4600
+Wire Wire Line
+	2600 4600 2600 4000
+Wire Wire Line
+	2600 4000 3450 4000
+Wire Wire Line
+	2650 4100 3450 4100
+Wire Wire Line
+	2650 4100 2650 4750
+Wire Wire Line
+	2650 4750 2050 4750
+Wire Wire Line
+	2050 4900 2700 4900
+Wire Wire Line
+	2700 4900 2700 4200
+Wire Wire Line
+	2700 4200 3450 4200
+Wire Wire Line
+	2750 4300 3450 4300
+Wire Wire Line
+	2750 4300 2750 5050
+Wire Wire Line
+	2750 5050 2050 5050
+Wire Wire Line
+	2050 5200 2800 5200
+Wire Wire Line
+	2800 5200 2800 4400
+Wire Wire Line
+	2800 4400 3450 4400
+Wire Wire Line
+	2050 5350 2850 5350
+Wire Wire Line
+	2850 5350 2850 4500
+Wire Wire Line
+	2850 4500 3450 4500
+Wire Wire Line
+	2050 5500 2900 5500
+Wire Wire Line
+	2900 5500 2900 4600
+Wire Wire Line
+	2900 4600 3450 4600
+Wire Wire Line
+	2050 5650 2950 5650
+Wire Wire Line
+	2950 5650 2950 4700
+Wire Wire Line
+	2950 4700 3450 4700
+Wire Wire Line
+	2050 5800 3000 5800
+Wire Wire Line
+	3000 5800 3000 4800
+Wire Wire Line
+	3000 4800 3450 4800
 $EndSCHEMATC
