File: OBC_prototypeB_04/Flash.sch (KiCad schematic (older format))
At the start: 26 parts, among them P10 FLASH_CS, P9 FLASH_SPI, U5 FLASH_IS25LP016D, U6 FLASH_IS25LP016D, U7 FLASH_IS25LP016D

Commit message: Tied up flash WP, removed flash CS pullup
Parts:
- removed R10, R11, R14, R15, R18, R19: 10k, SFUSat:R_0402, symbol R
Connections:
- wire segments 80 -> 76
Changed lines of the file:
@@
 	1    0    0    -1
 $EndComp
-$Comp
-L R R11
-U 1 1 59660092
-P 1550 1650
-F 0 "R11" V 1630 1650 50  0000 C CNN
-F 1 "10k" V 1550 1650 50  0000 C CNN
-F 2 "SFUSat:R_0402" V 1480 1650 50  0001 C CNN
-F 3 "" H 1550 1650 50  0000 C CNN
-	1    1550 1650
-	1    0    0    -1
-$EndComp
-Wire Wire Line
-	1550 1800 1550 1850
 Wire Wire Line
 	1350 1850 1800 1850
-$Comp
-L +3V3 #PWR69
-U 1 1 596601ED
-P 1550 1450
-F 0 "#PWR69" H 1550 1300 50  0001 C CNN
-F 1 "+3V3" H 1550 1590 50  0000 C CNN
-F 2 "" H 1550 1450 50  0000 C CNN
-F 3 "" H 1550 1450 50  0000 C CNN
-	1    1550 1450
-	1    0    0    -1
-$EndComp
-Wire Wire Line
-	1550 1450 1550 1500
 Text GLabel 1350 1850 0    60   Input ~ 0
 FLASH0_CS
-Connection ~ 1550 1850
 Text GLabel 1350 2000 0    60   Input ~ 0
 FLASH_MISO
@@
 Wire Wire Line
 	3400 1600 3400 1650
-$Comp
-L R R10
-U 1 1 5967C83E
-P 1450 2550
-F 0 "R10" V 1530 2550 50  0000 C CNN
-F 1 "10k" V 1450 2550 50  0000 C CNN
-F 2 "SFUSat:R_0402" V 1380 2550 50  0001 C CNN
-F 3 "" H 1450 2550 50  0000 C CNN
-	1    1450 2550
-	1    0    0    -1
-$EndComp
-$Comp
-L GND #PWR67
-U 1 1 5967C87C
-P 1450 2800
-F 0 "#PWR67" H 1450 2550 50  0001 C CNN
-F 1 "GND" H 1450 2650 50  0000 C CNN
-F 2 "" H 1450 2800 50  0000 C CNN
-F 3 "" H 1450 2800 50  0000 C CNN
-	1    1450 2800
-	1    0    0    -1
-$EndComp
-Wire Wire Line
-	1450 2050 1450 2400
+Wire Wire Line
+	1450 2050 1450 2600
 Wire Wire Line
 	1450 2050 1800 2050
-Wire Wire Line
-	1450 2700 1450 2800
 $Comp
 L TEST_1P W1
@@
 	1    0    0    -1
 $EndComp
-$Comp
-L R R15
-U 1 1 5967D2E8
-P 1450 3950
-F 0 "R15" V 1530 3950 50  0000 C CNN
-F 1 "10k" V 1450 3950 50  0000 C CNN
-F 2 "SFUSat:R_0402" V 1380 3950 50  0001 C CNN
-F 3 "" H 1450 3950 50  0000 C CNN
-	1    1450 3950
-	1    0    0    -1
-$EndComp
-Wire Wire Line
-	1450 4100 1450 4150
 Wire Wire Line
 	1250 4150 1700 4150
-$Comp
-L +3V3 #PWR68
-U 1 1 5967D2F0
-P 1450 3750
-F 0 "#PWR68" H 1450 3600 50  0001 C CNN
-F 1 "+3V3" H 1450 3890 50  0000 C CNN
-F 2 "" H 1450 3750 50  0000 C CNN
-F 3 "" H 1450 3750 50  0000 C CNN
-	1    1450 3750
-	1    0    0    -1
-$EndComp
-Wire Wire Line
-	1450 3750 1450 3800
 Text GLabel 1250 4150 0    60   Input ~ 0
 FLASH1_CS
-Connection ~ 1450 4150
 Text GLabel 1250 4300 0    60   Input ~ 0
 FLASH_MISO
@@
 Wire Wire Line
 	3300 3900 3300 3950
-$Comp
-L R R14
-U 1 1 5967D31E
-P 1350 4850
-F 0 "R14" V 1430 4850 50  0000 C CNN
-F 1 "10k" V 1350 4850 50  0000 C CNN
-F 2 "SFUSat:R_0402" V 1280 4850 50  0001 C CNN
-F 3 "" H 1350 4850 50  0000 C CNN
-	1    1350 4850
-	1    0    0    -1
-$EndComp
-$Comp
-L GND #PWR66
-U 1 1 5967D324
-P 1350 5100
-F 0 "#PWR66" H 1350 4850 50  0001 C CNN
-F 1 "GND" H 1350 4950 50  0000 C CNN
-F 2 "" H 1350 5100 50  0000 C CNN
-F 3 "" H 1350 5100 50  0000 C CNN
-	1    1350 5100
-	1    0    0    -1
-$EndComp
-Wire Wire Line
-	1350 4350 1350 4700
+Wire Wire Line
+	1350 4350 1350 4900
 Wire Wire Line
 	1350 4350 1700 4350
-Wire Wire Line
-	1350 5000 1350 5100
 $Comp
 L TEST_1P W3
@@
 	1    0    0    -1
 $EndComp
-$Comp
-L R R19
-U 1 1 5967D6B6
-P 6300 4850
-F 0 "R19" V 6380 4850 50  0000 C CNN
-F 1 "10k" V 6300 4850 50  0000 C CNN
-F 2 "SFUSat:R_0402" V 6230 4850 50  0001 C CNN
-F 3 "" H 6300 4850 50  0000 C CNN
-	1    6300 4850
-	1    0    0    -1
-$EndComp
-Wire Wire Line
-	6300 5000 6300 5050
 Wire Wire Line
 	6100 5050 6550 5050
-$Comp
-L +3V3 #PWR79
-U 1 1 5967D6BE
-P 6300 4650
-F 0 "#PWR79" H 6300 4500 50  0001 C CNN
-F 1 "+3V3" H 6300 4790 50  0000 C CNN
-F 2 "" H 6300 4650 50  0000 C CNN
-F 3 "" H 6300 4650 50  0000 C CNN
-	1    6300 4650
-	1    0    0    -1
-$EndComp
-Wire Wire Line
-	6300 4650 6300 4700
 Text GLabel 6100 5050 0    60   Input ~ 0
 FLASH2_CS
-Connection ~ 6300 5050
 Text GLabel 6100 5200 0    60   Input ~ 0
 FLASH_MISO
@@
 Wire Wire Line
 	8150 4800 8150 4850
-$Comp
-L R R18
-U 1 1 5967D6EC
-P 6200 5750
-F 0 "R18" V 6280 5750 50  0000 C CNN
-F 1 "10k" V 6200 5750 50  0000 C CNN
-F 2 "SFUSat:R_0402" V 6130 5750 50  0001 C CNN
-F 3 "" H 6200 5750 50  0000 C CNN
-	1    6200 5750
-	1    0    0    -1
-$EndComp
-$Comp
-L GND #PWR78
-U 1 1 5967D6F2
-P 6200 6000
-F 0 "#PWR78" H 6200 5750 50  0001 C CNN
-F 1 "GND" H 6200 5850 50  0000 C CNN
-F 2 "" H 6200 6000 50  0000 C CNN
-F 3 "" H 6200 6000 50  0000 C CNN
-	1    6200 6000
-	1    0    0    -1
-$EndComp
 Wire Wire Line
 	6200 5250 6200 5600
 Wire Wire Line
 	6200 5250 6550 5250
-Wire Wire Line
-	6200 5900 6200 6000
 $Comp
 L TEST_1P W5
@@
 Wire Wire Line
 	2900 6100 2850 6100
+$Comp
+L +3V3 #PWR?
+U 1 1 5A54954F
+P 1250 2600
+F 0 "#PWR?" H 1250 2450 50  0001 C CNN
+F 1 "+3V3" H 1250 2740 50  0000 C CNN
+F 2 "" H 1250 2600 50  0000 C CNN
+F 3 "" H 1250 2600 50  0000 C CNN
+	1    1250 2600
+	1    0    0    -1
+$EndComp
+Wire Wire Line
+	1450 2600 1250 2600
+$Comp
+L +3V3 #PWR?
+U 1 1 5A549794
+P 1150 4900
+F 0 "#PWR?" H 1150 4750 50  0001 C CNN
+F 1 "+3V3" H 1150 5040 50  0000 C CNN
+F 2 "" H 1150 4900 50  0000 C CNN
+F 3 "" H 1150 4900 50  0000 C CNN
+	1    1150 4900
+	1    0    0    -1
+$EndComp
+Wire Wire Line
+	1350 4900 1150 4900
+$Comp
+L +3V3 #PWR?
+U 1 1 5A5499B9
+P 6050 5900
+F 0 "#PWR?" H 6050 5750 50  0001 C CNN
+F 1 "+3V3" H 6050 6040 50  0000 C CNN
+F 2 "" H 6050 5900 50  0000 C CNN
+F 3 "" H 6050 5900 50  0000 C CNN
+	1    6050 5900
+	1    0    0    -1
+$EndComp
+Wire Wire Line
+	6150 5600 6150 5900
+Wire Wire Line
+	6150 5900 6050 5900
+Wire Wire Line
+	6200 5600 6150 5600
 $EndSCHEMATC

Commit message: Removed option to connect flash WP/RESET to MASTER_RESET
Parts:
- removed R12, R16, R20: 0, SFUSat:R_0402, symbol R
Connections:
- net labels removed: MASTER_RESET
- wire segments 76 -> 70
Changed lines of the file:
@@
 Wire Wire Line
 	3300 2050 3050 2050
-Text GLabel 3950 1500 1    60   Input ~ 0
-MASTER_RESET
-$Comp
-L R R12
-U 1 1 5967CA2E
-P 3950 1700
-F 0 "R12" V 4030 1700 50  0000 C CNN
-F 1 "0" V 3950 1700 50  0000 C CNN
-F 2 "SFUSat:R_0402" V 3880 1700 50  0001 C CNN
-F 3 "" H 3950 1700 50  0000 C CNN
-	1    3950 1700
-	1    0    0    -1
-$EndComp
 $Comp
 L R R13
@@
 $EndComp
 Wire Wire Line
-	3950 1500 3950 1550
-Wire Wire Line
 	3050 1950 4300 1950
 Wire Wire Line
-	3950 1950 3950 1850
-Wire Wire Line
 	4200 1950 4200 1850
-Connection ~ 3950 1950
 $Comp
 L +3V3 #PWR77
@@
 Wire Wire Line
 	3200 4350 2950 4350
-Text GLabel 3850 3800 1    60   Input ~ 0
-MASTER_RESET
-$Comp
-L R R16
-U 1 1 5967D338
-P 3850 4000
-F 0 "R16" V 3930 4000 50  0000 C CNN
-F 1 "0" V 3850 4000 50  0000 C CNN
-F 2 "SFUSat:R_0402" V 3780 4000 50  0001 C CNN
-F 3 "" H 3850 4000 50  0000 C CNN
-	1    3850 4000
-	1    0    0    -1
-$EndComp
 $Comp
 L R R17
@@
 $EndComp
 Wire Wire Line
-	3850 3800 3850 3850
-Wire Wire Line
-	2950 4250 4200 4250
-Wire Wire Line
-	3850 4250 3850 4150
-Wire Wire Line
 	4100 4250 4100 4150
-Connection ~ 3850 4250
 $Comp
 L +3V3 #PWR76
@@
 Wire Wire Line
 	8050 5250 7800 5250
-Text GLabel 8700 4700 1    60   Input ~ 0
-MASTER_RESET
-$Comp
-L R R20
-U 1 1 5967D706
-P 8700 4900
-F 0 "R20" V 8780 4900 50  0000 C CNN
-F 1 "0" V 8700 4900 50  0000 C CNN
-F 2 "SFUSat:R_0402" V 8630 4900 50  0001 C CNN
-F 3 "" H 8700 4900 50  0000 C CNN
-	1    8700 4900
-	1    0    0    -1
-$EndComp
 $Comp
 L R R21
@@
 $EndComp
 Wire Wire Line
-	8700 4700 8700 4750
-Wire Wire Line
 	7800 5150 9050 5150
 Wire Wire Line
-	8700 5150 8700 5050
-Wire Wire Line
 	8950 5150 8950 5050
-Connection ~ 8700 5150
 $Comp
 L +3V3 #PWR83
@@
 Wire Wire Line
 	6200 5600 6150 5600
+Wire Wire Line
+	2950 4250 4200 4250
 $EndSCHEMATC

Commit message: WIP initial placement
Parts:
- removed W1, W2, W3, W4, W5, W6: TEST_1P, SFUSat:Test_Point, symbol TEST_1P
Connections:
- wire segments 70 -> 67
Changed lines of the file:
@@
 	3050 2150 3300 2150
 $Comp
-L +3V3 #PWR73
+L +3V3 #PWR068
 U 1 1 59660272
 P 3050 1300
-F 0 "#PWR73" H 3050 1150 50  0001 C CNN
+F 0 "#PWR068" H 3050 1150 50  0001 C CNN
 F 1 "+3V3" H 3050 1440 50  0000 C CNN
 F 2 "" H 3050 1300 50  0000 C CNN
@@
 $EndComp
 $Comp
-L GND #PWR71
+L GND #PWR069
 U 1 1 5966028C
 P 1650 2200
-F 0 "#PWR71" H 1650 1950 50  0001 C CNN
+F 0 "#PWR069" H 1650 1950 50  0001 C CNN
 F 1 "GND" H 1650 2050 50  0000 C CNN
 F 2 "" H 1650 2200 50  0000 C CNN
@@
 $EndComp
 $Comp
-L GND #PWR75
+L GND #PWR070
 U 1 1 596602A6
 P 3400 1650
-F 0 "#PWR75" H 3400 1400 50  0001 C CNN
+F 0 "#PWR070" H 3400 1400 50  0001 C CNN
 F 1 "GND" H 3400 1500 50  0000 C CNN
 F 2 "" H 3400 1650 50  0000 C CNN
@@
 	3400 1600 3400 1650
 Wire Wire Line
-	1450 2050 1450 2600
-Wire Wire Line
 	1450 2050 1800 2050
-$Comp
-L TEST_1P W1
-U 1 1 5967C8EC
-P 1250 2300
-F 0 "W1" H 1250 2570 50  0000 C CNN
-F 1 "TEST_1P" H 1250 2500 50  0000 C CNN
-F 2 "SFUSat:Test_Point" H 1450 2300 50  0001 C CNN
-F 3 "" H 1450 2300 50  0000 C CNN
-	1    1250 2300
-	0    -1   -1   0
-$EndComp
-Wire Wire Line
-	1450 2300 1250 2300
-Connection ~ 1450 2300
 Wire Wire Line
 	3300 2150 3300 2250
@@
 $EndComp
 Wire Wire Line
-	3050 1950 4300 1950
-Wire Wire Line
 	4200 1950 4200 1850
 $Comp
-L +3V3 #PWR77
+L +3V3 #PWR071
 U 1 1 5967CBA8
 P 4200 1500
-F 0 "#PWR77" H 4200 1350 50  0001 C CNN
+F 0 "#PWR071" H 4200 1350 50  0001 C CNN
 F 1 "+3V3" H 4200 1640 50  0000 C CNN
 F 2 "" H 4200 1500 50  0000 C CNN
@@
 Text Notes 4150 1150 0    60   ~ 0
 Note: Only connect one of these at once. \nMASTER_RESET enables simultaneous memory\nand processor reset, with appropriate bits set.
-$Comp
-L TEST_1P W2
-U 1 1 5967CCB2
-P 4300 1950
-F 0 "W2" H 4300 2220 50  0000 C CNN
-F 1 "TEST_1P" H 4300 2150 50  0000 C CNN
-F 2 "SFUSat:Test_Point" H 4500 1950 50  0001 C CNN
-F 3 "" H 4500 1950 50  0000 C CNN
-	1    4300 1950
-	0    1    1    0
-$EndComp
-Connection ~ 4200 1950
 $Comp
 L FLASH_IS25LP016D U6
@@
 	2950 4450 3200 4450
 $Comp
-L +3V3 #PWR72
+L +3V3 #PWR072
 U 1 1 5967D300
 P 2950 3600
-F 0 "#PWR72" H 2950 3450 50  0001 C CNN
+F 0 "#PWR072" H 2950 3450 50  0001 C CNN
 F 1 "+3V3" H 2950 3740 50  0000 C CNN
 F 2 "" H 2950 3600 50  0000 C CNN
@@
 $EndComp
 $Comp
-L GND #PWR70
+L GND #PWR073
 U 1 1 5967D306
 P 1550 4500
-F 0 "#PWR70" H 1550 4250 50  0001 C CNN
+F 0 "#PWR073" H 1550 4250 50  0001 C CNN
 F 1 "GND" H 1550 4350 50  0000 C CNN
 F 2 "" H 1550 4500 50  0000 C CNN
@@
 $EndComp
 $Comp
-L GND #PWR74
+L GND #PWR074
 U 1 1 5967D30C
 P 3300 3950
-F 0 "#PWR74" H 3300 3700 50  0001 C CNN
+F 0 "#PWR074" H 3300 3700 50  0001 C CNN
 F 1 "GND" H 3300 3800 50  0000 C CNN
 F 2 "" H 3300 3950 50  0000 C CNN
@@
 Wire Wire Line
 	1350 4350 1700 4350
-$Comp
-L TEST_1P W3
-U 1 1 5967D32D
-P 1150 4600
-F 0 "W3" H 1150 4870 50  0000 C CNN
-F 1 "TEST_1P" H 1150 4800 50  0000 C CNN
-F 2 "SFUSat:Test_Point" H 1350 4600 50  0001 C CNN
-F 3 "" H 1350 4600 50  0000 C CNN
-	1    1150 4600
-	0    -1   -1   0
-$EndComp
-Wire Wire Line
-	1350 4600 1150 4600
-Connection ~ 1350 4600
 Wire Wire Line
 	3200 4450 3200 4550
@@
 	1    0    0    -1
 $EndComp
-Wire Wire Line
-	4100 4250 4100 4150
-$Comp
-L +3V3 #PWR76
+$Comp
+L +3V3 #PWR075
 U 1 1 5967D349
 P 4100 3800
-F 0 "#PWR76" H 4100 3650 50  0001 C CNN
+F 0 "#PWR075" H 4100 3650 50  0001 C CNN
 F 1 "+3V3" H 4100 3940 50  0000 C CNN
 F 2 "" H 4100 3800 50  0000 C CNN
@@
 Text Notes 4050 3450 0    60   ~ 0
 Note: Only connect one of these at once. \nMASTER_RESET enables simultaneous memory\nand processor reset, with appropriate bits set.
-$Comp
-L TEST_1P W4
-U 1 1 5967D351
-P 4200 4250
-F 0 "W4" H 4200 4520 50  0000 C CNN
-F 1 "TEST_1P" H 4200 4450 50  0000 C CNN
-F 2 "SFUSat:Test_Point" H 4400 4250 50  0001 C CNN
-F 3 "" H 4400 4250 50  0000 C CNN
-	1    4200 4250
-	0    1    1    0
-$EndComp
-Connection ~ 4100 4250
 $Comp
 L FLASH_IS25LP016D U7
@@
 	7800 5350 8050 5350
 $Comp
-L +3V3 #PWR81
+L +3V3 #PWR076
 U 1 1 5967D6CE
 P 7800 4500
-F 0 "#PWR81" H 7800 4350 50  0001 C CNN
+F 0 "#PWR076" H 7800 4350 50  0001 C CNN
 F 1 "+3V3" H 7800 4640 50  0000 C CNN
 F 2 "" H 7800 4500 50  0000 C CNN
@@
 $EndComp
 $Comp
-L GND #PWR80
+L GND #PWR077
 U 1 1 5967D6D4
 P 6400 5400
-F 0 "#PWR80" H 6400 5150 50  0001 C CNN
+F 0 "#PWR077" H 6400 5150 50  0001 C CNN
 F 1 "GND" H 6400 5250 50  0000 C CNN
 F 2 "" H 6400 5400 50  0000 C CNN
@@
 $EndComp
 $Comp
-L GND #PWR82
+L GND #PWR078
 U 1 1 5967D6DA
 P 8150 4850
-F 0 "#PWR82" H 8150 4600 50  0001 C CNN
+F 0 "#PWR078" H 8150 4600 50  0001 C CNN
 F 1 "GND" H 8150 4700 50  0000 C CNN
 F 2 "" H 8150 4850 50  0000 C CNN
@@
 	8150 4800 8150 4850
 Wire Wire Line
-	6200 5250 6200 5600
-Wire Wire Line
 	6200 5250 6550 5250
-$Comp
-L TEST_1P W5
-U 1 1 5967D6FB
-P 6000 5500
-F 0 "W5" H 6000 5770 50  0000 C CNN
-F 1 "TEST_1P" H 6000 5700 50  0000 C CNN
-F 2 "SFUSat:Test_Point" H 6200 5500 50  0001 C CNN
-F 3 "" H 6200 5500 50  0000 C CNN
-	1    6000 5500
-	0    -1   -1   0
-$EndComp
-Wire Wire Line
-	6200 5500 6000 5500
-Connection ~ 6200 5500
 Wire Wire Line
 	8050 5350 8050 5450
@@
 $EndComp
 Wire Wire Line
-	7800 5150 9050 5150
-Wire Wire Line
 	8950 5150 8950 5050
 $Comp
-L +3V3 #PWR83
+L +3V3 #PWR079
 U 1 1 5967D717
 P 8950 4700
-F 0 "#PWR83" H 8950 4550 50  0001 C CNN
+F 0 "#PWR079" H 8950 4550 50  0001 C CNN
 F 1 "+3V3" H 8950 4840 50  0000 C CNN
 F 2 "" H 8950 4700 50  0000 C CNN
@@
 Text Notes 8900 4350 0    60   ~ 0
 Note: Only connect one of these at once. \nMASTER_RESET enables simultaneous memory\nand processor reset, with appropriate bits set.
-$Comp
-L TEST_1P W6
-U 1 1 5967D71F
-P 9050 5150
-F 0 "W6" H 9050 5420 50  0000 C CNN
-F 1 "TEST_1P" H 9050 5350 50  0000 C CNN
-F 2 "SFUSat:Test_Point" H 9250 5150 50  0001 C CNN
-F 3 "" H 9250 5150 50  0000 C CNN
-	1    9050 5150
-	0    1    1    0
-$EndComp
-Connection ~ 8950 5150
 Text Notes 7950 2300 0    60   ~ 0
 Triple redundant memory with configurable hold/reset. \nHold will pause comms, reset will reset and can be set \nto be synchronous with processor reset through \nMASTER_RESET\n
@@
 3v3
 $Comp
-L +3V3 #PWR84
+L +3V3 #PWR080
 U 1 1 5967E2DE
 P 10100 950
-F 0 "#PWR84" H 10100 800 50  0001 C CNN
+F 0 "#PWR080" H 10100 800 50  0001 C CNN
 F 1 "+3V3" H 10100 1090 50  0000 C CNN
 F 2 "" H 10100 950 50  0000 C CNN
@@
 	2900 6100 2850 6100
 $Comp
-L +3V3 #PWR?
+L +3V3 #PWR081
 U 1 1 5A54954F
 P 1250 2600
-F 0 "#PWR?" H 1250 2450 50  0001 C CNN
+F 0 "#PWR081" H 1250 2450 50  0001 C CNN
 F 1 "+3V3" H 1250 2740 50  0000 C CNN
 F 2 "" H 1250 2600 50  0000 C CNN
@@
 	1450 2600 1250 2600
 $Comp
-L +3V3 #PWR?
+L +3V3 #PWR082
 U 1 1 5A549794
 P 1150 4900
-F 0 "#PWR?" H 1150 4750 50  0001 C CNN
+F 0 "#PWR082" H 1150 4750 50  0001 C CNN
 F 1 "+3V3" H 1150 5040 50  0000 C CNN
 F 2 "" H 1150 4900 50  0000 C CNN
@@
 	1350 4900 1150 4900
 $Comp
-L +3V3 #PWR?
+L +3V3 #PWR083
 U 1 1 5A5499B9
 P 6050 5900
-F 0 "#PWR?" H 6050 5750 50  0001 C CNN
+F 0 "#PWR083" H 6050 5750 50  0001 C CNN
 F 1 "+3V3" H 6050 6040 50  0000 C CNN
 F 2 "" H 6050 5900 50  0000 C CNN
@@
 	6200 5600 6150 5600
 Wire Wire Line
-	2950 4250 4200 4250
+	2950 4250 4100 4250
+Wire Wire Line
+	4100 4250 4100 4150
+Wire Wire Line
+	6200 5250 6200 5600
+Wire Wire Line
+	8950 5150 7800 5150
+Wire Wire Line
+	4200 1950 3050 1950
+Wire Wire Line
+	1450 2050 1450 2600
 $EndSCHEMATC
