File: OBC_prototypeB_04/bulk_power.sch (KiCad schematic (older format))
At the start: 39 parts, among them P1 3v3_IN_CONNECTOR, P2 INA_INPUT, P3 INA_GND, P4 INA_EN, P5 INA_OUTPUT, Q1 DMN2075U, Q2 DMN2075U, Q3 1v2_GOOD, U1 TMS570LS0714, U2 XC6222B121MR-G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

Commit message: Removed trimpot
Parts:
- removed VR1: Trimpot, SFUSat:Trimpot_Bourns_TC33, symbol Trimpot
Connections:
- wire segments 105 -> 103
Changed lines of the file:
@@
 LIBS:valves
 LIBS:SFUSat
-LIBS:OBC_04-cache
 EELAYER 25 0
 EELAYER END
@@
 	3900 2800 3600 2800
 Wire Wire Line
-	3600 2800 3600 2850
+	3600 2800 3600 3550
 Wire Wire Line
 	3900 3850 3900 3000
@@
 Text Notes 3050 6750 0    60   ~ 0
 C1, C3, C8 were removed at the board level, as multiple pins were connected to one cap.
-$Comp
-L Trimpot VR1
-U 1 1 597E4B2A
-P 3600 3200
-F 0 "VR1" H 3700 3300 60  0000 C CNN
-F 1 "Trimpot" H 3300 3050 60  0000 C CNN
-F 2 "SFUSat:Trimpot_Bourns_TC33" H 3400 3200 60  0001 C CNN
-F 3 "" H 3400 3200 60  0001 C CNN
-	1    3600 3200
-	0    1    1    0
-$EndComp
 Wire Wire Line
 	3600 3850 3900 3850
@@
 	3750 3850 3750 4050
 Connection ~ 3750 3850
-Wire Wire Line
-	3300 3200 3300 3450
-Wire Wire Line
-	3300 3450 3600 3450
-Connection ~ 3600 3450
 $EndSCHEMATC

Commit message: Added load connector, switched RTC to MIBSPI5
RTC on MIBSPI5 because it operates in the same power domain as pretty much everything else. Can now shut off PD3 (though we'd lose I2C access), and the RTC will be fine since it is on PD1.
Parts:
- added P?: LOAD, SFUSat:2x01In_Header_v2, symbol CONN_01X02
Connections:
- wire segments 103 -> 107
Other:
- note added: "For load testing the current limit\n"
Changed lines of the file:
@@
 LIBS:valves
 LIBS:SFUSat
+LIBS:OBC_04-cache
 EELAYER 25 0
 EELAYER END
@@
 	3750 3850 3750 4050
 Connection ~ 3750 3850
+$Comp
+L CONN_01X02 P?
+U 1 1 5A646879
+P 6500 3700
+F 0 "P?" H 6500 3850 50  0000 C CNN
+F 1 "LOAD" V 6600 3700 50  0000 C CNN
+F 2 "SFUSat:2x01In_Header_v2" H 6500 3700 50  0001 C CNN
+F 3 "" H 6500 3700 50  0000 C CNN
+	1    6500 3700
+	-1   0    0    1
+$EndComp
+$Comp
+L +3V3 #PWR?
+U 1 1 5A646F64
+P 6900 3600
+F 0 "#PWR?" H 6900 3450 50  0001 C CNN
+F 1 "+3V3" H 6900 3740 50  0000 C CNN
+F 2 "" H 6900 3600 50  0000 C CNN
+F 3 "" H 6900 3600 50  0000 C CNN
+	1    6900 3600
+	1    0    0    -1
+$EndComp
+$Comp
+L GND #PWR?
+U 1 1 5A6470B7
+P 6900 3850
+F 0 "#PWR?" H 6900 3600 50  0001 C CNN
+F 1 "GND" H 6900 3700 50  0000 C CNN
+F 2 "" H 6900 3850 50  0000 C CNN
+F 3 "" H 6900 3850 50  0000 C CNN
+	1    6900 3850
+	1    0    0    -1
+$EndComp
+Wire Wire Line
+	6700 3650 6900 3650
+Wire Wire Line
+	6900 3650 6900 3600
+Wire Wire Line
+	6700 3750 6900 3750
+Wire Wire Line
+	6900 3750 6900 3850
+Text Notes 6200 4200 0    60   ~ 0
+For load testing the current limit\n
 $EndSCHEMATC

Commit message: Routed xtal
also removed osc fault jumper
Parts:
- gave numbers to parts that had none: 1
Changed lines of the file:
@@
 Connection ~ 3750 3850
 $Comp
-L CONN_01X02 P?
+L CONN_01X02 P12
 U 1 1 5A646879
 P 6500 3700
-F 0 "P?" H 6500 3850 50  0000 C CNN
+F 0 "P12" H 6500 3850 50  0000 C CNN
 F 1 "LOAD" V 6600 3700 50  0000 C CNN
 F 2 "SFUSat:2x01In_Header_v2" H 6500 3700 50  0001 C CNN
@@
 $EndComp
 $Comp
-L +3V3 #PWR?
+L +3V3 #PWR028
 U 1 1 5A646F64
 P 6900 3600
-F 0 "#PWR?" H 6900 3450 50  0001 C CNN
+F 0 "#PWR028" H 6900 3450 50  0001 C CNN
 F 1 "+3V3" H 6900 3740 50  0000 C CNN
 F 2 "" H 6900 3600 50  0000 C CNN
@@
 $EndComp
 $Comp
-L GND #PWR?
+L GND #PWR029
 U 1 1 5A6470B7
 P 6900 3850
-F 0 "#PWR?" H 6900 3600 50  0001 C CNN
+F 0 "#PWR029" H 6900 3600 50  0001 C CNN
 F 1 "GND" H 6900 3700 50  0000 C CNN
 F 2 "" H 6900 3850 50  0000 C CNN
