File: OBC_prototypeB_04/MCU_Support_Reset.sch (KiCad schematic (older format))
At the start: 29 parts, among them P12 JTAG_20PIN, P13 WD_EN, P14 WD_RST_EN, P7 OSC_FUALT_INJECT, SW1 SPST, SW2 SPST, SW4 SPST, U1 TMS570LS0714, U11 STLM75, U9 TPS3110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

Commit message: Board outline, holes
Parts:
- gave numbers to parts that had none: 1
Changed lines of the file:
@@
 $EndComp
 $Comp
-L +3V3 #PWR36
+L +3V3 #PWR3
 U 1 1 5956048B
 P 1200 700
-F 0 "#PWR36" H 1200 550 50  0001 C CNN
+F 0 "#PWR3" H 1200 550 50  0001 C CNN
 F 1 "+3V3" H 1200 840 50  0000 C CNN
 F 2 "" H 1200 700 50  0000 C CNN
@@
 Connection ~ 1550 1700
 $Comp
-L GND #PWR34
+L GND #PWR1
 U 1 1 59682837
 P 800 1550
-F 0 "#PWR34" H 800 1300 50  0001 C CNN
+F 0 "#PWR1" H 800 1300 50  0001 C CNN
 F 1 "GND" H 800 1400 50  0000 C CNN
 F 2 "" H 800 1550 50  0000 C CNN
@@
 	8800 3300 8800 2500
 $Comp
-L GND #PWR52
+L GND #PWR21
 U 1 1 5968A38D
 P 8700 3350
-F 0 "#PWR52" H 8700 3100 50  0001 C CNN
+F 0 "#PWR21" H 8700 3100 50  0001 C CNN
 F 1 "GND" H 8700 3200 50  0000 C CNN
 F 2 "" H 8700 3350 50  0000 C CNN
@@
 $EndComp
 $Comp
-L +3V3 #PWR57
+L +3V3 #PWR24
 U 1 1 5968A3C2
 P 9600 2100
-F 0 "#PWR57" H 9600 1950 50  0001 C CNN
+F 0 "#PWR24" H 9600 1950 50  0001 C CNN
 F 1 "+3V3" H 9600 2240 50  0000 C CNN
 F 2 "" H 9600 2100 50  0000 C CNN
@@
 1v2
 $Comp
-L +1V2 #PWR38
+L +1V2 #PWR5
 U 1 1 5968AD45
 P 1500 700
-F 0 "#PWR38" H 1500 550 50  0001 C CNN
+F 0 "#PWR5" H 1500 550 50  0001 C CNN
 F 1 "+1V2" H 1500 840 50  0000 C CNN
 F 2 "" H 1500 700 50  0000 C CNN
@@
 	7950 1400 9150 1400
 $Comp
-L +3V3 #PWR47
+L +3V3 #PWR14
 U 1 1 597111CE
 P 5500 3450
-F 0 "#PWR47" H 5500 3300 50  0001 C CNN
+F 0 "#PWR14" H 5500 3300 50  0001 C CNN
 F 1 "+3V3" H 5500 3590 50  0000 C CNN
 F 2 "" H 5500 3450 50  0000 C CNN
@@
 $EndComp
 $Comp
-L GND #PWR42
+L GND #PWR9
 U 1 1 59711206
 P 3600 3800
-F 0 "#PWR42" H 3600 3550 50  0001 C CNN
+F 0 "#PWR9" H 3600 3550 50  0001 C CNN
 F 1 "GND" H 3600 3650 50  0000 C CNN
 F 2 "" H 3600 3800 50  0000 C CNN
@@
 $EndComp
 $Comp
-L GND #PWR46
+L GND #PWR13
 U 1 1 59711388
 P 5150 4350
-F 0 "#PWR46" H 5150 4100 50  0001 C CNN
+F 0 "#PWR13" H 5150 4100 50  0001 C CNN
 F 1 "GND" H 5150 4200 50  0000 C CNN
 F 2 "" H 5150 4350 50  0000 C CNN
@@
 	3900 3950 4000 3950
 $Comp
-L GND #PWR43
+L GND #PWR10
 U 1 1 5971283C
 P 3900 5000
-F 0 "#PWR43" H 3900 4750 50  0001 C CNN
+F 0 "#PWR10" H 3900 4750 50  0001 C CNN
 F 1 "GND" H 3900 4850 50  0000 C CNN
 F 2 "" H 3900 5000 50  0000 C CNN
@@
 $EndComp
 $Comp
-L +1V2 #PWR48
+L +1V2 #PWR15
 U 1 1 59712E3B
 P 6100 3400
-F 0 "#PWR48" H 6100 3250 50  0001 C CNN
+F 0 "#PWR15" H 6100 3250 50  0001 C CNN
 F 1 "+1V2" H 6100 3540 50  0000 C CNN
 F 2 "" H 6100 3400 50  0000 C CNN
@@
 	6100 3550 6100 3400
 $Comp
-L GND #PWR49
+L GND #PWR16
 U 1 1 59713064
 P 6100 4500
-F 0 "#PWR49" H 6100 4250 50  0001 C CNN
+F 0 "#PWR16" H 6100 4250 50  0001 C CNN
 F 1 "GND" H 6100 4350 50  0000 C CNN
 F 2 "" H 6100 4500 50  0000 C CNN
@@
 	6100 4400 6100 4500
 $Comp
-L +3V3 #PWR54
+L +3V3 #PWR23
 U 1 1 597134C1
 P 8900 950
-F 0 "#PWR54" H 8900 800 50  0001 C CNN
+F 0 "#PWR23" H 8900 800 50  0001 C CNN
 F 1 "+3V3" H 8900 1090 50  0000 C CNN
 F 2 "" H 8900 950 50  0000 C CNN
@@
 	1300 6300 1300 6500
 $Comp
-L +3V3 #PWR41
+L +3V3 #PWR8
 U 1 1 59719A03
 P 3550 6100
-F 0 "#PWR41" H 3550 5950 50  0001 C CNN
+F 0 "#PWR8" H 3550 5950 50  0001 C CNN
 F 1 "+3V3" H 3550 6240 50  0000 C CNN
 F 2 "" H 3550 6100 50  0000 C CNN
@@
 $EndComp
 $Comp
-L +3V3 #PWR40
+L +3V3 #PWR7
 U 1 1 59719A6D
 P 3250 5800
-F 0 "#PWR40" H 3250 5650 50  0001 C CNN
+F 0 "#PWR7" H 3250 5650 50  0001 C CNN
 F 1 "+3V3" H 3250 5940 50  0000 C CNN
 F 2 "" H 3250 5800 50  0000 C CNN
@@
 $EndComp
 $Comp
-L +3V3 #PWR37
+L +3V3 #PWR4
 U 1 1 59719ABA
 P 1300 5900
-F 0 "#PWR37" H 1300 5750 50  0001 C CNN
+F 0 "#PWR4" H 1300 5750 50  0001 C CNN
 F 1 "+3V3" H 1300 6040 50  0000 C CNN
 F 2 "" H 1300 5900 50  0000 C CNN
@@
 $EndComp
 $Comp
-L +3V3 #PWR35
+L +3V3 #PWR2
 U 1 1 59719B8B
 P 1100 6150
-F 0 "#PWR35" H 1100 6000 50  0001 C CNN
+F 0 "#PWR2" H 1100 6000 50  0001 C CNN
 F 1 "+3V3" H 1100 6290 50  0000 C CNN
 F 2 "" H 1100 6150 50  0000 C CNN
@@
 	1650 6350 1650 5900
 $Comp
-L GND #PWR39
+L GND #PWR6
 U 1 1 59740380
 P 1750 6950
-F 0 "#PWR39" H 1750 6700 50  0001 C CNN
+F 0 "#PWR6" H 1750 6700 50  0001 C CNN
 F 1 "GND" H 1750 6800 50  0000 C CNN
 F 2 "" H 1750 6950 50  0000 C CNN
@@
 	1750 6200 1750 6950
 $Comp
-L +3V3 #PWR45
+L +3V3 #PWR12
 U 1 1 597406F6
 P 4900 6300
-F 0 "#PWR45" H 4900 6150 50  0001 C CNN
+F 0 "#PWR12" H 4900 6150 50  0001 C CNN
 F 1 "+3V3" H 4900 6440 50  0000 C CNN
 F 2 "" H 4900 6300 50  0000 C CNN
@@
 	4900 6400 4900 6300
 $Comp
-L GND #PWR50
+L GND #PWR17
 U 1 1 59740B82
 P 6200 7400
-F 0 "#PWR50" H 6200 7150 50  0001 C CNN
+F 0 "#PWR17" H 6200 7150 50  0001 C CNN
 F 1 "GND" H 6200 7250 50  0000 C CNN
 F 2 "" H 6200 7400 50  0000 C CNN
@@
 $EndComp
 $Comp
-L +5V #PWR44
+L +5V #PWR11
 U 1 1 597411F2
 P 4000 7400
-F 0 "#PWR44" H 4000 7250 50  0001 C CNN
+F 0 "#PWR11" H 4000 7250 50  0001 C CNN
 F 1 "+5V" H 4000 7540 50  0000 C CNN
 F 2 "" H 4000 7400 50  0000 C CNN
@@
 $EndComp
 $Comp
-L GND #PWR56
+L GND #PWR26
 U 1 1 5A52A627
 P 10750 5050
-F 0 "#PWR56" H 10750 4800 50  0001 C CNN
+F 0 "#PWR26" H 10750 4800 50  0001 C CNN
 F 1 "GND" H 10750 4900 50  0000 C CNN
 F 2 "" H 10750 5050 50  0000 C CNN
@@
 $EndComp
 $Comp
-L +3V3 #PWR55
+L +3V3 #PWR25
 U 1 1 5A52A87E
 P 10750 4200
-F 0 "#PWR55" H 10750 4050 50  0001 C CNN
+F 0 "#PWR25" H 10750 4050 50  0001 C CNN
 F 1 "+3V3" H 10750 4340 50  0000 C CNN
 F 2 "" H 10750 4200 50  0000 C CNN
@@
 Connection ~ 8100 1400
 $Comp
-L GND #PWR53
+L GND #PWR22
 U 1 1 5A547DDF
 P 8700 3350
-F 0 "#PWR53" H 8700 3100 50  0001 C CNN
+F 0 "#PWR22" H 8700 3100 50  0001 C CNN
 F 1 "GND" H 8700 3200 50  0000 C CNN
 F 2 "" H 8700 3350 50  0000 C CNN
@@
 $EndComp
 $Comp
-L GND #PWR51
+L GND #PWR19
 U 1 1 5A547F9D
 P 8100 2750
-F 0 "#PWR51" H 8100 2500 50  0001 C CNN
+F 0 "#PWR19" H 8100 2500 50  0001 C CNN
 F 1 "GND" H 8100 2600 50  0000 C CNN
 F 2 "" H 8100 2750 50  0000 C CNN
@@
 Connection ~ 9100 1700
 $Comp
-L conn_1x9 J?
+L conn_1x9 J1
 U 1 1 5A54CD99
 P 7000 6000
-F 0 "J?" H 7100 5850 60  0000 C CNN
+F 0 "J1" H 7100 5850 60  0000 C CNN
 F 1 "conn_1x9" H 7050 5750 60  0000 C CNN
 F 2 "" H 7000 6000 60  0001 C CNN
@@
 Compact JTAG Connector\n
 $Comp
-L +3V3 #PWR?
+L +3V3 #PWR18
 U 1 1 5A54CF50
 P 6600 5700
-F 0 "#PWR?" H 6600 5550 50  0001 C CNN
+F 0 "#PWR18" H 6600 5550 50  0001 C CNN
 F 1 "+3V3" H 6600 5840 50  0000 C CNN
 F 2 "" H 6600 5700 50  0000 C CNN
@@
 MASTER_RESET
 $Comp
-L GND #PWR?
+L GND #PWR20
 U 1 1 5A54D2AE
 P 8100 5800
-F 0 "#PWR?" H 8100 5550 50  0001 C CNN
+F 0 "#PWR20" H 8100 5550 50  0001 C CNN
 F 1 "GND" H 8100 5650 50  0000 C CNN
 F 2 "" H 8100 5800 50  0000 C CNN

Commit message: WIP initial placement
Parts:
- removed J1: conn_1x9, symbol conn_1x9
Connections:
- wire segments 123 -> 114
Other:
- note removed: "Compact JTAG Connector\n"
Changed lines of the file:
@@
 $EndComp
 $Comp
-L +3V3 #PWR3
+L +3V3 #PWR034
 U 1 1 5956048B
 P 1200 700
-F 0 "#PWR3" H 1200 550 50  0001 C CNN
+F 0 "#PWR034" H 1200 550 50  0001 C CNN
 F 1 "+3V3" H 1200 840 50  0000 C CNN
 F 2 "" H 1200 700 50  0000 C CNN
@@
 Connection ~ 1550 1700
 $Comp
-L GND #PWR1
+L GND #PWR035
 U 1 1 59682837
 P 800 1550
-F 0 "#PWR1" H 800 1300 50  0001 C CNN
+F 0 "#PWR035" H 800 1300 50  0001 C CNN
 F 1 "GND" H 800 1400 50  0000 C CNN
 F 2 "" H 800 1550 50  0000 C CNN
@@
 	8800 3300 8800 2500
 $Comp
-L GND #PWR21
+L GND #PWR036
 U 1 1 5968A38D
 P 8700 3350
-F 0 "#PWR21" H 8700 3100 50  0001 C CNN
+F 0 "#PWR036" H 8700 3100 50  0001 C CNN
 F 1 "GND" H 8700 3200 50  0000 C CNN
 F 2 "" H 8700 3350 50  0000 C CNN
@@
 $EndComp
 $Comp
-L +3V3 #PWR24
+L +3V3 #PWR037
 U 1 1 5968A3C2
 P 9600 2100
-F 0 "#PWR24" H 9600 1950 50  0001 C CNN
+F 0 "#PWR037" H 9600 1950 50  0001 C CNN
 F 1 "+3V3" H 9600 2240 50  0000 C CNN
 F 2 "" H 9600 2100 50  0000 C CNN
@@
 1v2
 $Comp
-L +1V2 #PWR5
+L +1V2 #PWR038
 U 1 1 5968AD45
 P 1500 700
-F 0 "#PWR5" H 1500 550 50  0001 C CNN
+F 0 "#PWR038" H 1500 550 50  0001 C CNN
 F 1 "+1V2" H 1500 840 50  0000 C CNN
 F 2 "" H 1500 700 50  0000 C CNN
@@
 	7950 1400 9150 1400
 $Comp
-L +3V3 #PWR14
+L +3V3 #PWR039
 U 1 1 597111CE
 P 5500 3450
-F 0 "#PWR14" H 5500 3300 50  0001 C CNN
+F 0 "#PWR039" H 5500 3300 50  0001 C CNN
 F 1 "+3V3" H 5500 3590 50  0000 C CNN
 F 2 "" H 5500 3450 50  0000 C CNN
@@
 $EndComp
 $Comp
-L GND #PWR9
+L GND #PWR040
 U 1 1 59711206
 P 3600 3800
-F 0 "#PWR9" H 3600 3550 50  0001 C CNN
+F 0 "#PWR040" H 3600 3550 50  0001 C CNN
 F 1 "GND" H 3600 3650 50  0000 C CNN
 F 2 "" H 3600 3800 50  0000 C CNN
@@
 $EndComp
 $Comp
-L GND #PWR13
+L GND #PWR041
 U 1 1 59711388
 P 5150 4350
-F 0 "#PWR13" H 5150 4100 50  0001 C CNN
+F 0 "#PWR041" H 5150 4100 50  0001 C CNN
 F 1 "GND" H 5150 4200 50  0000 C CNN
 F 2 "" H 5150 4350 50  0000 C CNN
@@
 	3900 3950 4000 3950
 $Comp
-L GND #PWR10
+L GND #PWR042
 U 1 1 5971283C
 P 3900 5000
-F 0 "#PWR10" H 3900 4750 50  0001 C CNN
+F 0 "#PWR042" H 3900 4750 50  0001 C CNN
 F 1 "GND" H 3900 4850 50  0000 C CNN
 F 2 "" H 3900 5000 50  0000 C CNN
@@
 $EndComp
 $Comp
-L +1V2 #PWR15
+L +1V2 #PWR043
 U 1 1 59712E3B
 P 6100 3400
-F 0 "#PWR15" H 6100 3250 50  0001 C CNN
+F 0 "#PWR043" H 6100 3250 50  0001 C CNN
 F 1 "+1V2" H 6100 3540 50  0000 C CNN
 F 2 "" H 6100 3400 50  0000 C CNN
@@
 	6100 3550 6100 3400
 $Comp
-L GND #PWR16
+L GND #PWR044
 U 1 1 59713064
 P 6100 4500
-F 0 "#PWR16" H 6100 4250 50  0001 C CNN
+F 0 "#PWR044" H 6100 4250 50  0001 C CNN
 F 1 "GND" H 6100 4350 50  0000 C CNN
 F 2 "" H 6100 4500 50  0000 C CNN
@@
 	6100 4400 6100 4500
 $Comp
-L +3V3 #PWR23
+L +3V3 #PWR045
 U 1 1 597134C1
 P 8900 950
-F 0 "#PWR23" H 8900 800 50  0001 C CNN
+F 0 "#PWR045" H 8900 800 50  0001 C CNN
 F 1 "+3V3" H 8900 1090 50  0000 C CNN
 F 2 "" H 8900 950 50  0000 C CNN
@@
 	1300 6300 1300 6500
 $Comp
-L +3V3 #PWR8
+L +3V3 #PWR046
 U 1 1 59719A03
 P 3550 6100
-F 0 "#PWR8" H 3550 5950 50  0001 C CNN
+F 0 "#PWR046" H 3550 5950 50  0001 C CNN
 F 1 "+3V3" H 3550 6240 50  0000 C CNN
 F 2 "" H 3550 6100 50  0000 C CNN
@@
 $EndComp
 $Comp
-L +3V3 #PWR7
+L +3V3 #PWR047
 U 1 1 59719A6D
 P 3250 5800
-F 0 "#PWR7" H 3250 5650 50  0001 C CNN
+F 0 "#PWR047" H 3250 5650 50  0001 C CNN
 F 1 "+3V3" H 3250 5940 50  0000 C CNN
 F 2 "" H 3250 5800 50  0000 C CNN
@@
 $EndComp
 $Comp
-L +3V3 #PWR4
+L +3V3 #PWR048
 U 1 1 59719ABA
 P 1300 5900
-F 0 "#PWR4" H 1300 5750 50  0001 C CNN
+F 0 "#PWR048" H 1300 5750 50  0001 C CNN
 F 1 "+3V3" H 1300 6040 50  0000 C CNN
 F 2 "" H 1300 5900 50  0000 C CNN
@@
 $EndComp
 $Comp
-L +3V3 #PWR2
+L +3V3 #PWR049
 U 1 1 59719B8B
 P 1100 6150
-F 0 "#PWR2" H 1100 6000 50  0001 C CNN
+F 0 "#PWR049" H 1100 6000 50  0001 C CNN
 F 1 "+3V3" H 1100 6290 50  0000 C CNN
 F 2 "" H 1100 6150 50  0000 C CNN
@@
 	1650 6350 1650 5900
 $Comp
-L GND #PWR6
+L GND #PWR050
 U 1 1 59740380
 P 1750 6950
-F 0 "#PWR6" H 1750 6700 50  0001 C CNN
+F 0 "#PWR050" H 1750 6700 50  0001 C CNN
 F 1 "GND" H 1750 6800 50  0000 C CNN
 F 2 "" H 1750 6950 50  0000 C CNN
@@
 	1750 6200 1750 6950
 $Comp
-L +3V3 #PWR12
+L +3V3 #PWR051
 U 1 1 597406F6
 P 4900 6300
-F 0 "#PWR12" H 4900 6150 50  0001 C CNN
+F 0 "#PWR051" H 4900 6150 50  0001 C CNN
 F 1 "+3V3" H 4900 6440 50  0000 C CNN
 F 2 "" H 4900 6300 50  0000 C CNN
@@
 	4900 6400 4900 6300
 $Comp
-L GND #PWR17
+L GND #PWR052
 U 1 1 59740B82
 P 6200 7400
-F 0 "#PWR17" H 6200 7150 50  0001 C CNN
+F 0 "#PWR052" H 6200 7150 50  0001 C CNN
 F 1 "GND" H 6200 7250 50  0000 C CNN
 F 2 "" H 6200 7400 50  0000 C CNN
@@
 $EndComp
 $Comp
-L +5V #PWR11
+L +5V #PWR053
 U 1 1 597411F2
 P 4000 7400
-F 0 "#PWR11" H 4000 7250 50  0001 C CNN
+F 0 "#PWR053" H 4000 7250 50  0001 C CNN
 F 1 "+5V" H 4000 7540 50  0000 C CNN
 F 2 "" H 4000 7400 50  0000 C CNN
@@
 $EndComp
 $Comp
-L GND #PWR26
+L GND #PWR054
 U 1 1 5A52A627
 P 10750 5050
-F 0 "#PWR26" H 10750 4800 50  0001 C CNN
+F 0 "#PWR054" H 10750 4800 50  0001 C CNN
 F 1 "GND" H 10750 4900 50  0000 C CNN
 F 2 "" H 10750 5050 50  0000 C CNN
@@
 $EndComp
 $Comp
-L +3V3 #PWR25
+L +3V3 #PWR055
 U 1 1 5A52A87E
 P 10750 4200
-F 0 "#PWR25" H 10750 4050 50  0001 C CNN
+F 0 "#PWR055" H 10750 4050 50  0001 C CNN
 F 1 "+3V3" H 10750 4340 50  0000 C CNN
 F 2 "" H 10750 4200 50  0000 C CNN
@@
 Connection ~ 8100 1400
 $Comp
-L GND #PWR22
+L GND #PWR056
 U 1 1 5A547DDF
 P 8700 3350
-F 0 "#PWR22" H 8700 3100 50  0001 C CNN
+F 0 "#PWR056" H 8700 3100 50  0001 C CNN
 F 1 "GND" H 8700 3200 50  0000 C CNN
 F 2 "" H 8700 3350 50  0000 C CNN
@@
 $EndComp
 $Comp
-L GND #PWR19
+L GND #PWR057
 U 1 1 5A547F9D
 P 8100 2750
-F 0 "#PWR19" H 8100 2500 50  0001 C CNN
+F 0 "#PWR057" H 8100 2500 50  0001 C CNN
 F 1 "GND" H 8100 2600 50  0000 C CNN
 F 2 "" H 8100 2750 50  0000 C CNN
@@
 	9200 1850 9200 2000
 Connection ~ 9100 1700
-$Comp
-L conn_1x9 J1
-U 1 1 5A54CD99
-P 7000 6000
-F 0 "J1" H 7100 5850 60  0000 C CNN
-F 1 "conn_1x9" H 7050 5750 60  0000 C CNN
-F 2 "" H 7000 6000 60  0001 C CNN
-F 3 "" H 7000 6000 60  0001 C CNN
-	1    7000 6000
-	1    0    0    -1
-$EndComp
-Text Notes 6850 6450 0    60   ~ 0
-Compact JTAG Connector\n
-$Comp
-L +3V3 #PWR18
-U 1 1 5A54CF50
-P 6600 5700
-F 0 "#PWR18" H 6600 5550 50  0001 C CNN
-F 1 "+3V3" H 6600 5840 50  0000 C CNN
-F 2 "" H 6600 5700 50  0000 C CNN
-F 3 "" H 6600 5700 50  0000 C CNN
-	1    6600 5700
-	1    0    0    -1
-$EndComp
-Text GLabel 6750 5500 1    60   Input ~ 0
-nTRST
-Text GLabel 6900 5500 1    60   Input ~ 0
-TDI
-Text GLabel 7050 5500 1    60   Input ~ 0
-TMS
-Text GLabel 7200 5500 1    60   Input ~ 0
-TCK
-Text GLabel 7350 5500 1    60   Input ~ 0
-RTCK
-Text GLabel 7500 5500 1    60   Input ~ 0
-TDO
-Text GLabel 7650 5500 1    60   Input ~ 0
-MASTER_RESET
-$Comp
-L GND #PWR20
-U 1 1 5A54D2AE
-P 8100 5800
-F 0 "#PWR20" H 8100 5550 50  0001 C CNN
-F 1 "GND" H 8100 5650 50  0000 C CNN
-F 2 "" H 8100 5800 50  0000 C CNN
-F 3 "" H 8100 5800 50  0000 C CNN
-	1    8100 5800
-	1    0    0    -1
-$EndComp
-Wire Wire Line
-	6600 5700 6600 5800
-Wire Wire Line
-	6750 5800 6750 5500
-Wire Wire Line
-	6900 5500 6900 5800
-Wire Wire Line
-	7050 5800 7050 5500
-Wire Wire Line
-	7200 5500 7200 5800
-Wire Wire Line
-	7350 5500 7350 5800
-Wire Wire Line
-	7500 5500 7500 5800
-Wire Wire Line
-	7650 5800 7650 5500
-Wire Wire Line
-	7800 5800 8100 5800
 $EndSCHEMATC

Commit message: Removed JTAG resistors
Parts:
- removed R27, R28, R29, R30: 100k, SFUSat:R_0402, symbol R
Connections:
- wire segments 114 -> 105
Changed lines of the file:
@@
 Connection ~ 3950 3550
-$Comp
-L R R28
-U 1 1 597192CE
-P 1300 6150
-F 0 "R28" V 1380 6150 50  0000 C CNN
-F 1 "100k" V 1300 6150 50  0000 C CNN
-F 2 "SFUSat:R_0402" V 1230 6150 50  0001 C CNN
-F 3 "" H 1300 6150 50  0000 C CNN
-	1    1300 6150
-	1    0    0    -1
-$EndComp
-$Comp
-L R R27
-U 1 1 59719326
-P 1100 6400
-F 0 "R27" V 1180 6400 50  0000 C CNN
-F 1 "100k" V 1100 6400 50  0000 C CNN
-F 2 "SFUSat:R_0402" V 1030 6400 50  0001 C CNN
-F 3 "" H 1100 6400 50  0000 C CNN
-	1    1100 6400
-	1    0    0    -1
-$EndComp
-$Comp
-L R R29
-U 1 1 59719386
-P 3250 6050
-F 0 "R29" V 3330 6050 50  0000 C CNN
-F 1 "100k" V 3250 6050 50  0000 C CNN
-F 2 "SFUSat:R_0402" V 3180 6050 50  0001 C CNN
-F 3 "" H 3250 6050 50  0000 C CNN
-	1    3250 6050
-	1    0    0    -1
-$EndComp
-$Comp
-L R R30
-U 1 1 597193EC
-P 3550 6350
-F 0 "R30" V 3630 6350 50  0000 C CNN
-F 1 "100k" V 3550 6350 50  0000 C CNN
-F 2 "SFUSat:R_0402" V 3480 6350 50  0001 C CNN
-F 3 "" H 3550 6350 50  0000 C CNN
-	1    3550 6350
-	1    0    0    -1
-$EndComp
-Wire Wire Line
-	3050 6250 3250 6250
-Wire Wire Line
-	3250 6250 3250 6200
-Wire Wire Line
-	3050 6550 3550 6550
-Wire Wire Line
-	3550 6550 3550 6500
-Wire Wire Line
-	1100 6650 1950 6650
-Wire Wire Line
-	1100 6650 1100 6550
-Wire Wire Line
-	1300 6500 1950 6500
-Wire Wire Line
-	1300 6300 1300 6500
-$Comp
-L +3V3 #PWR046
-U 1 1 59719A03
-P 3550 6100
-F 0 "#PWR046" H 3550 5950 50  0001 C CNN
-F 1 "+3V3" H 3550 6240 50  0000 C CNN
-F 2 "" H 3550 6100 50  0000 C CNN
-F 3 "" H 3550 6100 50  0000 C CNN
-	1    3550 6100
-	1    0    0    -1
-$EndComp
-$Comp
-L +3V3 #PWR047
-U 1 1 59719A6D
-P 3250 5800
-F 0 "#PWR047" H 3250 5650 50  0001 C CNN
-F 1 "+3V3" H 3250 5940 50  0000 C CNN
-F 2 "" H 3250 5800 50  0000 C CNN
-F 3 "" H 3250 5800 50  0000 C CNN
-	1    3250 5800
-	1    0    0    -1
-$EndComp
-$Comp
-L +3V3 #PWR048
-U 1 1 59719ABA
-P 1300 5900
-F 0 "#PWR048" H 1300 5750 50  0001 C CNN
-F 1 "+3V3" H 1300 6040 50  0000 C CNN
-F 2 "" H 1300 5900 50  0000 C CNN
-F 3 "" H 1300 5900 50  0000 C CNN
-	1    1300 5900
-	1    0    0    -1
-$EndComp
-$Comp
-L +3V3 #PWR049
-U 1 1 59719B8B
-P 1100 6150
-F 0 "#PWR049" H 1100 6000 50  0001 C CNN
-F 1 "+3V3" H 1100 6290 50  0000 C CNN
-F 2 "" H 1100 6150 50  0000 C CNN
-F 3 "" H 1100 6150 50  0000 C CNN
-	1    1100 6150
-	1    0    0    -1
-$EndComp
-Wire Wire Line
-	3250 5800 3250 5900
-Wire Wire Line
-	3550 6100 3550 6200
-Wire Wire Line
-	1300 5900 1300 6000
-Wire Wire Line
-	1100 6150 1100 6250
 $Comp
 L JTAG_20PIN P12
@@
 Wire Wire Line
 	3350 6600 3350 6550
-Connection ~ 3350 6550
 Wire Wire Line
 	4800 6700 4950 6700
@@
 Wire Wire Line
 	3100 6150 3100 6250
-Connection ~ 3100 6250
 Text GLabel 4800 6850 0    60   Input ~ 0
 TCK
@@
 Wire Wire Line
 	1400 6750 1400 6650
-Connection ~ 1400 6650
 Wire Wire Line
 	4800 6850 4800 6800
@@
 RTCK
 Wire Wire Line
-	1300 6350 1500 6350
-Wire Wire Line
-	1500 6350 1500 5900
-Connection ~ 1300 6350
+	1500 5900 1500 6500
 Text GLabel 4800 7000 0    60   Input ~ 0
 RTCK
@@
 	9200 1850 9200 2000
 Connection ~ 9100 1700
+Wire Wire Line
+	3350 6550 3050 6550
+Wire Wire Line
+	3100 6250 3050 6250
+Wire Wire Line
+	1500 6500 1950 6500
+Wire Wire Line
+	1400 6650 1950 6650
 $EndSCHEMATC

Commit message: Added note about R25, changed value of R24
Parts:
- R24: value 100k -> 2.2k
Other:
- note added: "R25 is not populated in 0.3"
Changed lines of the file:
@@
 P 8900 1200
 F 0 "R24" V 8980 1200 50  0000 C CNN
-F 1 "100k" V 8900 1200 50  0000 C CNN
+F 1 "2.2k" V 8900 1200 50  0000 C CNN
 F 2 "SFUSat:R_0402" V 8830 1200 50  0001 C CNN
 F 3 "" H 8900 1200 50  0000 C CNN
@@
 U 1 1 59741105
 P 4750 7600
-F 0 "JTAG5V_IN1" V 4850 7600 50  0000 C CNN
+F 0 "JTAG5V_IN1" V 4750 7950 50  0000 C CNN
 F 1 "JTAG5V_IN" V 4850 7600 50  0000 C CNN
 F 2 "SFUSat:2x01In_Header_v2" H 4750 7600 50  0001 C CNN
@@
 Wire Wire Line
 	1400 6650 1950 6650
+Text Notes 9250 2450 0    60   ~ 0
+R25 is not populated in 0.3
 $EndSCHEMATC
