File: OBC_prototypeB_04/MCU_Support_Reset.sch (KiCad schematic (older format))
At the start: 24 parts, among them P12 JTAG_20PIN, P13 WD_EN, P14 WD_RST_EN, P7 OSC_FUALT_INJECT, SW1 SPST, SW2 SPST, SW4 SPST, U1 TMS570LS0714, U11 STLM75, U9 TPS3110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

Commit message: Updated to 10 pin JTAG
Parts:
- removed JTAG5V_IN1: JTAG5V_IN, SFUSat:2x01In_Header_v2, symbol CONN_01X02
- removed P12: JTAG_20PIN, SFUSat:JTAG_20pin, symbol JTAG_20PIN
- added P?: JTAG_10PIN, symbol JTAG_10PIN
Connections:
- net labels removed: +5V
- wire segments 105 -> 86
Changed lines of the file:
@@
 	3950 3400 3950 3550
 Connection ~ 3950 3550
-$Comp
-L JTAG_20PIN P12
-U 1 1 5973ED32
-P 5550 6950
-F 0 "P12" V 5550 7400 60  0000 C CNN
-F 1 "JTAG_20PIN" V 5550 6950 60  0000 C CNN
-F 2 "SFUSat:JTAG_20pin" H 5550 6950 60  0001 C CNN
-F 3 "" H 5550 6950 60  0001 C CNN
-	1    5550 6950
-	1    0    0    -1
-$EndComp
-Text GLabel 4800 6700 0    60   Input ~ 0
+Text GLabel 5700 5100 0    60   Input ~ 0
 TMS
 Text GLabel 3350 6600 3    60   Input ~ 0
 TMS
-Text GLabel 4800 7150 0    60   Input ~ 0
+Text GLabel 5200 5450 0    60   Input ~ 0
 TDO
 Text GLabel 3150 6400 2    60   Input ~ 0
@@
 Wire Wire Line
 	3350 6600 3350 6550
-Wire Wire Line
-	4800 6700 4950 6700
-Text GLabel 4750 6550 0    60   Input ~ 0
+Text GLabel 5700 5700 0    60   Input ~ 0
 TDI
 Text GLabel 3100 6150 1    60   Input ~ 0
 TDI
 Wire Wire Line
-	4750 6550 4950 6550
-Wire Wire Line
-	4950 6550 4950 6600
-Wire Wire Line
 	3100 6150 3100 6250
-Text GLabel 4800 6850 0    60   Input ~ 0
+Text GLabel 5700 5300 0    60   Input ~ 0
 TCK
 Text GLabel 1400 6750 3    60   Input ~ 0
@@
 Wire Wire Line
 	1400 6750 1400 6650
-Wire Wire Line
-	4800 6850 4800 6800
-Wire Wire Line
-	4800 6800 4950 6800
 Text GLabel 1500 5900 1    60   Input ~ 0
 RTCK
 Wire Wire Line
 	1500 5900 1500 6500
-Text GLabel 4800 7000 0    60   Input ~ 0
-RTCK
-Wire Wire Line
-	4800 7000 4800 6900
-Wire Wire Line
-	4800 6900 4950 6900
-Wire Wire Line
-	4800 7150 4800 7050
-Wire Wire Line
-	4800 7050 4850 7050
-Wire Wire Line
-	4850 7050 4850 7000
-Wire Wire Line
-	4850 7000 4950 7000
 Text GLabel 1650 5900 1    60   Input ~ 0
 nTRST
-Text GLabel 4750 6400 0    60   Input ~ 0
+Text GLabel 5700 5550 0    60   Input ~ 0
 nTRST
-Wire Wire Line
-	4750 6400 4800 6400
-Wire Wire Line
-	4800 6400 4800 6500
-Wire Wire Line
-	4800 6500 4950 6500
 Wire Wire Line
 	1950 6350 1650 6350
@@
 L +3V3 #PWR051
 U 1 1 597406F6
-P 4900 6300
-F 0 "#PWR051" H 4900 6150 50  0001 C CNN
-F 1 "+3V3" H 4900 6440 50  0000 C CNN
-F 2 "" H 4900 6300 50  0000 C CNN
-F 3 "" H 4900 6300 50  0000 C CNN
-	1    4900 6300
-	1    0    0    -1
-$EndComp
-Wire Wire Line
-	4950 6400 4900 6400
-Wire Wire Line
-	4900 6400 4900 6300
+P 5450 4950
+F 0 "#PWR051" H 5450 4800 50  0001 C CNN
+F 1 "+3V3" H 5450 5090 50  0000 C CNN
+F 2 "" H 5450 4950 50  0000 C CNN
+F 3 "" H 5450 4950 50  0000 C CNN
+	1    5450 4950
+	1    0    0    -1
+$EndComp
 $Comp
 L GND #PWR052
 U 1 1 59740B82
-P 6200 7400
-F 0 "#PWR052" H 6200 7150 50  0001 C CNN
-F 1 "GND" H 6200 7250 50  0000 C CNN
-F 2 "" H 6200 7400 50  0000 C CNN
-F 3 "" H 6200 7400 50  0000 C CNN
-	1    6200 7400
-	1    0    0    -1
-$EndComp
-Wire Wire Line
-	6100 6500 6200 6500
-Wire Wire Line
-	6200 6500 6200 7400
-Wire Wire Line
-	6100 6600 6200 6600
-Connection ~ 6200 6600
-Wire Wire Line
-	6100 6700 6200 6700
-Connection ~ 6200 6700
-Wire Wire Line
-	6100 6800 6200 6800
-Connection ~ 6200 6800
-Wire Wire Line
-	6100 6900 6200 6900
-Connection ~ 6200 6900
-Wire Wire Line
-	6100 7000 6200 7000
-Connection ~ 6200 7000
-Wire Wire Line
-	6100 7100 6200 7100
-Connection ~ 6200 7100
-Wire Wire Line
-	6100 7200 6200 7200
-Connection ~ 6200 7200
-Wire Wire Line
-	6100 7300 6200 7300
-Connection ~ 6200 7300
-$Comp
-L CONN_01X02 JTAG5V_IN1
-U 1 1 59741105
-P 4750 7600
-F 0 "JTAG5V_IN1" V 4750 7950 50  0000 C CNN
-F 1 "JTAG5V_IN" V 4850 7600 50  0000 C CNN
-F 2 "SFUSat:2x01In_Header_v2" H 4750 7600 50  0001 C CNN
-F 3 "" H 4750 7600 50  0000 C CNN
-	1    4750 7600
-	0    1    1    0
-$EndComp
-$Comp
-L +5V #PWR053
-U 1 1 597411F2
-P 4000 7400
-F 0 "#PWR053" H 4000 7250 50  0001 C CNN
-F 1 "+5V" H 4000 7540 50  0000 C CNN
-F 2 "" H 4000 7400 50  0000 C CNN
-F 3 "" H 4000 7400 50  0000 C CNN
-	1    4000 7400
-	1    0    0    -1
-$EndComp
-Wire Wire Line
-	4000 7400 4700 7400
-Wire Wire Line
-	4800 7400 4800 7300
-Wire Wire Line
-	4800 7300 4950 7300
+P 4750 5200
+F 0 "#PWR052" H 4750 4950 50  0001 C CNN
+F 1 "GND" H 4750 5050 50  0000 C CNN
+F 2 "" H 4750 5200 50  0000 C CNN
+F 3 "" H 4750 5200 50  0000 C CNN
+	1    4750 5200
+	1    0    0    -1
+$EndComp
 $Comp
 L CONN_01X02 P13
@@
 Wire Wire Line
 	4050 2150 3850 2150
-Text GLabel 4250 7050 0    60   Input ~ 0
+Text GLabel 5700 5900 0    60   Input ~ 0
 MASTER_RESET
-Wire Wire Line
-	4250 7050 4350 7050
-Wire Wire Line
-	4350 7050 4350 7250
-Wire Wire Line
-	4350 7250 4850 7250
-Wire Wire Line
-	4850 7250 4850 7100
-Wire Wire Line
-	4850 7100 4950 7100
 $Comp
 L SPST SW4
@@
 Text Notes 9250 2450 0    60   ~ 0
 R25 is not populated in 0.3
+$Comp
+L JTAG_10PIN P?
+U 1 1 5A66B705
+P 6650 5550
+F 0 "P?" V 6650 6000 60  0000 C CNN
+F 1 "JTAG_10PIN" V 6650 5550 60  0000 C CNN
+F 2 "" H 6650 5550 60  0001 C CNN
+F 3 "" H 6650 5550 60  0001 C CNN
+	1    6650 5550
+	1    0    0    -1
+$EndComp
+Wire Wire Line
+	6050 5900 5700 5900
+Wire Wire Line
+	5700 5700 6050 5700
+Wire Wire Line
+	5700 5550 5800 5550
+Wire Wire Line
+	5800 5550 5800 5600
+Wire Wire Line
+	5800 5600 6050 5600
+Wire Wire Line
+	6050 5500 5800 5500
+Wire Wire Line
+	5700 5300 6050 5300
+Wire Wire Line
+	5700 5100 6050 5100
+Wire Wire Line
+	5800 5500 5800 5450
+Wire Wire Line
+	5800 5450 5200 5450
+Wire Wire Line
+	6050 5200 4750 5200
+Wire Wire Line
+	5450 4950 6050 4950
+Wire Wire Line
+	6050 4950 6050 5000
+Wire Wire Line
+	6050 5400 5900 5400
+Wire Wire Line
+	5900 5400 5900 5200
+Connection ~ 5900 5200
 $EndSCHEMATC

Commit message: Routed xtal
also removed osc fault jumper
Parts:
- removed P7: OSC_FUALT_INJECT, SFUSat:2x01In_Header_v2, symbol CONN_01X02
- removed R38: 1k, SFUSat:R_0402, symbol R
- P16: renamed from P?; footprint (none) -> SFUSat:JTAG_10pin_1.27mm
Connections:
- wire segments 86 -> 82
Changed lines of the file:
@@
 $EndComp
 $Comp
-L +3V3 #PWR034
+L +3V3 #PWR036
 U 1 1 5956048B
 P 1200 700
-F 0 "#PWR034" H 1200 550 50  0001 C CNN
+F 0 "#PWR036" H 1200 550 50  0001 C CNN
 F 1 "+3V3" H 1200 840 50  0000 C CNN
 F 2 "" H 1200 700 50  0000 C CNN
@@
 Wire Wire Line
 	1300 2250 2250 2250
-$Comp
-L CONN_01X02 P7
-U 1 1 596827B1
-P 850 1300
-F 0 "P7" H 850 1450 50  0000 C CNN
-F 1 "OSC_FUALT_INJECT" V 950 1300 50  0000 C CNN
-F 2 "SFUSat:2x01In_Header_v2" H 850 1300 50  0001 C CNN
-F 3 "" H 850 1300 50  0000 C CNN
-	1    850  1300
-	0    -1   -1   0
-$EndComp
-Wire Wire Line
-	1550 1500 1550 1700
-Connection ~ 1550 1700
-$Comp
-L GND #PWR035
-U 1 1 59682837
-P 800 1550
-F 0 "#PWR035" H 800 1300 50  0001 C CNN
-F 1 "GND" H 800 1400 50  0000 C CNN
-F 2 "" H 800 1550 50  0000 C CNN
-F 3 "" H 800 1550 50  0000 C CNN
-	1    800  1550
-	1    0    0    -1
-$EndComp
-Wire Wire Line
-	800  1500 800  1550
 Text GLabel 3150 3550 0    60   Input ~ 0
 MASTER_RESET
@@
 	8800 3300 8800 2500
 $Comp
-L GND #PWR036
+L GND #PWR038
 U 1 1 5968A38D
 P 8700 3350
-F 0 "#PWR036" H 8700 3100 50  0001 C CNN
+F 0 "#PWR038" H 8700 3100 50  0001 C CNN
 F 1 "GND" H 8700 3200 50  0000 C CNN
 F 2 "" H 8700 3350 50  0000 C CNN
@@
 $EndComp
 $Comp
-L +3V3 #PWR037
+L +3V3 #PWR039
 U 1 1 5968A3C2
 P 9600 2100
-F 0 "#PWR037" H 9600 1950 50  0001 C CNN
+F 0 "#PWR039" H 9600 1950 50  0001 C CNN
 F 1 "+3V3" H 9600 2240 50  0000 C CNN
 F 2 "" H 9600 2100 50  0000 C CNN
@@
 1v2
 $Comp
-L +1V2 #PWR038
+L +1V2 #PWR040
 U 1 1 5968AD45
 P 1500 700
-F 0 "#PWR038" H 1500 550 50  0001 C CNN
+F 0 "#PWR040" H 1500 550 50  0001 C CNN
 F 1 "+1V2" H 1500 840 50  0000 C CNN
 F 2 "" H 1500 700 50  0000 C CNN
@@
 	7950 1400 9150 1400
 $Comp
-L +3V3 #PWR039
+L +3V3 #PWR041
 U 1 1 597111CE
 P 5500 3450
-F 0 "#PWR039" H 5500 3300 50  0001 C CNN
+F 0 "#PWR041" H 5500 3300 50  0001 C CNN
 F 1 "+3V3" H 5500 3590 50  0000 C CNN
 F 2 "" H 5500 3450 50  0000 C CNN
@@
 $EndComp
 $Comp
-L GND #PWR040
+L GND #PWR042
 U 1 1 59711206
 P 3600 3800
-F 0 "#PWR040" H 3600 3550 50  0001 C CNN
+F 0 "#PWR042" H 3600 3550 50  0001 C CNN
 F 1 "GND" H 3600 3650 50  0000 C CNN
 F 2 "" H 3600 3800 50  0000 C CNN
@@
 $EndComp
 $Comp
-L GND #PWR041
+L GND #PWR043
 U 1 1 59711388
 P 5150 4350
-F 0 "#PWR041" H 5150 4100 50  0001 C CNN
+F 0 "#PWR043" H 5150 4100 50  0001 C CNN
 F 1 "GND" H 5150 4200 50  0000 C CNN
 F 2 "" H 5150 4350 50  0000 C CNN
@@
 	3900 3950 4000 3950
 $Comp
-L GND #PWR042
+L GND #PWR044
 U 1 1 5971283C
 P 3900 5000
-F 0 "#PWR042" H 3900 4750 50  0001 C CNN
+F 0 "#PWR044" H 3900 4750 50  0001 C CNN
 F 1 "GND" H 3900 4850 50  0000 C CNN
 F 2 "" H 3900 5000 50  0000 C CNN
@@
 $EndComp
 $Comp
-L +1V2 #PWR043
+L +1V2 #PWR045
 U 1 1 59712E3B
 P 6100 3400
-F 0 "#PWR043" H 6100 3250 50  0001 C CNN
+F 0 "#PWR045" H 6100 3250 50  0001 C CNN
 F 1 "+1V2" H 6100 3540 50  0000 C CNN
 F 2 "" H 6100 3400 50  0000 C CNN
@@
 	6100 3550 6100 3400
 $Comp
-L GND #PWR044
+L GND #PWR046
 U 1 1 59713064
 P 6100 4500
-F 0 "#PWR044" H 6100 4250 50  0001 C CNN
+F 0 "#PWR046" H 6100 4250 50  0001 C CNN
 F 1 "GND" H 6100 4350 50  0000 C CNN
 F 2 "" H 6100 4500 50  0000 C CNN
@@
 	6100 4400 6100 4500
 $Comp
-L +3V3 #PWR045
+L +3V3 #PWR047
 U 1 1 597134C1
 P 8900 950
-F 0 "#PWR045" H 8900 800 50  0001 C CNN
+F 0 "#PWR047" H 8900 800 50  0001 C CNN
 F 1 "+3V3" H 8900 1090 50  0000 C CNN
 F 2 "" H 8900 950 50  0000 C CNN
@@
 	1650 6350 1650 5900
 $Comp
-L GND #PWR050
+L GND #PWR048
 U 1 1 59740380
 P 1750 6950
-F 0 "#PWR050" H 1750 6700 50  0001 C CNN
+F 0 "#PWR048" H 1750 6700 50  0001 C CNN
 F 1 "GND" H 1750 6800 50  0000 C CNN
 F 2 "" H 1750 6950 50  0000 C CNN
@@
 	1750 6200 1750 6950
 $Comp
-L +3V3 #PWR051
+L +3V3 #PWR049
 U 1 1 597406F6
 P 5450 4950
-F 0 "#PWR051" H 5450 4800 50  0001 C CNN
+F 0 "#PWR049" H 5450 4800 50  0001 C CNN
 F 1 "+3V3" H 5450 5090 50  0000 C CNN
 F 2 "" H 5450 4950 50  0000 C CNN
@@
 $EndComp
 $Comp
-L GND #PWR052
+L GND #PWR050
 U 1 1 59740B82
 P 4750 5200
-F 0 "#PWR052" H 4750 4950 50  0001 C CNN
+F 0 "#PWR050" H 4750 4950 50  0001 C CNN
 F 1 "GND" H 4750 5050 50  0000 C CNN
 F 2 "" H 4750 5200 50  0000 C CNN
@@
 	2250 1700 2250 1850
 Connection ~ 1800 1700
-$Comp
-L R R38
-U 1 1 597F6613
-P 1200 1500
-F 0 "R38" V 1280 1500 50  0000 C CNN
-F 1 "1k" V 1200 1500 50  0000 C CNN
-F 2 "SFUSat:R_0402" V 1130 1500 50  0001 C CNN
-F 3 "" H 1200 1500 50  0000 C CNN
-	1    1200 1500
-	0    1    1    0
-$EndComp
-Wire Wire Line
-	1350 1500 1550 1500
-Wire Wire Line
-	1050 1500 900  1500
 Text Label 1950 1700 0    60   ~ 0
 OSC_P
@@
 $EndComp
 $Comp
-L GND #PWR054
+L GND #PWR051
 U 1 1 5A52A627
 P 10750 5050
-F 0 "#PWR054" H 10750 4800 50  0001 C CNN
+F 0 "#PWR051" H 10750 4800 50  0001 C CNN
 F 1 "GND" H 10750 4900 50  0000 C CNN
 F 2 "" H 10750 5050 50  0000 C CNN
@@
 $EndComp
 $Comp
-L +3V3 #PWR055
+L +3V3 #PWR052
 U 1 1 5A52A87E
 P 10750 4200
-F 0 "#PWR055" H 10750 4050 50  0001 C CNN
+F 0 "#PWR052" H 10750 4050 50  0001 C CNN
 F 1 "+3V3" H 10750 4340 50  0000 C CNN
 F 2 "" H 10750 4200 50  0000 C CNN
@@
 Connection ~ 8100 1400
 $Comp
-L GND #PWR056
+L GND #PWR053
 U 1 1 5A547DDF
 P 8700 3350
-F 0 "#PWR056" H 8700 3100 50  0001 C CNN
+F 0 "#PWR053" H 8700 3100 50  0001 C CNN
 F 1 "GND" H 8700 3200 50  0000 C CNN
 F 2 "" H 8700 3350 50  0000 C CNN
@@
 $EndComp
 $Comp
-L GND #PWR057
+L GND #PWR054
 U 1 1 5A547F9D
 P 8100 2750
-F 0 "#PWR057" H 8100 2500 50  0001 C CNN
+F 0 "#PWR054" H 8100 2500 50  0001 C CNN
 F 1 "GND" H 8100 2600 50  0000 C CNN
 F 2 "" H 8100 2750 50  0000 C CNN
@@
 R25 is not populated in 0.3
 $Comp
-L JTAG_10PIN P?
+L JTAG_10PIN P16
 U 1 1 5A66B705
 P 6650 5550
-F 0 "P?" V 6650 6000 60  0000 C CNN
+F 0 "P16" V 6650 6000 60  0000 C CNN
 F 1 "JTAG_10PIN" V 6650 5550 60  0000 C CNN
-F 2 "" H 6650 5550 60  0001 C CNN
+F 2 "SFUSat:JTAG_10pin_1.27mm" H 6650 5550 60  0001 C CNN
 F 3 "" H 6650 5550 60  0001 C CNN
 	1    6650 5550
