File: v0.5/PC104_Connector.sch (KiCad schematic (older format))
At the start: 19 parts, among them J1 PC104-8BIT, P11 USB_5V, P15 3pin-DC-power, P6 USB_PORT, Q4 DMN2075U, U10 FT230XQ-R

Commit message: Updated 1.2v regulator, removed DC jack
Parts:
- removed P15: 3pin-DC-power, SFUSat:PJ-028-SMT-TR-3pin-DC-jack PJ-028-SMT-TR, symbol 3pin-DC-power
- J1: symbol PC104-8BIT -> PC104-8BIT-RESCUE-OBC_05
Connections:
- wire segments 206 -> 194
Changed lines of the file:
@@
 EESchema Schematic File Version 2
+LIBS:OBC_05-rescue
 LIBS:power
 LIBS:device
@@
 LIBS:valves
 LIBS:SFUSat
-LIBS:OBC_04-cache
+LIBS:OBC_05-cache
 EELAYER 25 0
 EELAYER END
@@
 $EndDescr
 $Comp
-L PC104-8BIT J1
+L PC104-8BIT-RESCUE-OBC_05 J1
 U 1 1 5955D07C
 P 7900 2850
@@
 Text Notes 10550 4200 0    60   ~ 0
 Sun Sensors
-$Comp
-L 3pin-DC-power P15
-U 1 1 5A5EF47C
-P 6350 4750
-F 0 "P15" H 5700 4850 60  0000 C CNN
-F 1 "3pin-DC-power" H 6000 5000 60  0000 C CNN
-F 2 "SFUSat:PJ-028-SMT-TR-3pin-DC-jackPJ-028-SMT-TR" H 6350 4750 60  0001 C CNN
-F 3 "" H 6350 4750 60  0001 C CNN
-	1    6350 4750
-	0    -1   -1   0
-$EndComp
 Wire Wire Line
 	5400 1550 7350 1550
@@
 Wire Wire Line
 	8750 4150 10100 4150
-Wire Wire Line
-	7350 4250 6450 4250
-Wire Wire Line
-	6450 4250 6450 4950
-Wire Wire Line
-	7350 4150 6900 4150
-Wire Wire Line
-	6900 4150 6900 4250
-Connection ~ 6900 4250
-Wire Wire Line
-	6350 4950 6350 4850
-Wire Wire Line
-	6350 4850 6450 4850
-Connection ~ 6450 4850
-Wire Wire Line
-	6250 4950 6250 4600
-Wire Wire Line
-	6250 4600 6400 4600
-Wire Wire Line
-	6400 4600 6400 4050
-Wire Wire Line
-	6400 4050 7350 4050
-Wire Wire Line
-	7100 4050 7100 3950
-Wire Wire Line
-	7100 3950 7350 3950
-Connection ~ 7100 4050
 $EndSCHEMATC

Commit message: Removed extraneous 104 connections
Parts:
- added 0Ω (x4): R_Small, symbol R_Small
Connections:
- net labels added: LIN_RX, LIN_TX, RF_CS2, xGPIO0, xGPIO1, xGPIO2, xGPIO3, xGPIO4, xGPIO5
- net labels removed: AD1_10, AD1_3, AD1_4, AD1_5, AD1_6, AD1_7, AD1_8, AD1_9, ANTENNA_DEPLOY, NHET1_22, NHET1_26, NHET1_4, NHET1_7, RF_ADC1, RF_ADC2, RF_GAIN_CS, RF_PWM1, RF_PWM2, SPI4_CLK, SPI4_CS0, SPI4_MISO, SPI4_MOSI
- wire segments 194 -> 179
Other:
- note removed: "ANTENNA_ADC"
- note removed: "GIOA7"
- note removed: "HEAT_ADC"
- note removed: "RF.ADC3"
- note removed: "RF.ADC4\n"
- note removed: "RF.ADC5\n"
- note removed: "SENS_ADC"

Commit message: Added required xGPIO, removed 5V from 104 connector
Connections:
- net labels added: 104_3v3, xGPIO6, xGPIO7, xGPIO8
- wire segments 179 -> 167
Other:
- note added: "EPS_CHRG_OK"
- note added: "EPS_PROCHP"
- note added: "GPS_RST\n"
- note added: "RF_Deploy0"
- note added: "RF_Deploy1\n\n"
- note added: "RF_IRQ2"
- note removed: "RF_Deploy"
- note removed: "RF_Deploy\n"
- note removed: "RTC_INT\n"

Commit message: Removed traces, gen netlist, fixed button footprints
Parts:
- 0Ω1, 0Ω2, 0Ω3, 0Ω4: renamed from 0Ω; footprint (none) -> SFUSat:R_0402
Changed lines of the file:
@@
 RF_CS2
 $Comp
-L +5V #PWR032
+L +5V #PWR32
 U 1 1 59569513
 P 10100 750
-F 0 "#PWR032" H 10100 600 50  0001 C CNN
+F 0 "#PWR32" H 10100 600 50  0001 C CNN
 F 1 "+5V" H 10100 890 50  0000 C CNN
 F 2 "" H 10100 750 50  0000 C CNN
@@
 $EndComp
 $Comp
-L +5V #PWR033
+L +5V #PWR30
 U 1 1 595F60FC
 P 950 2150
-F 0 "#PWR033" H 950 2000 50  0001 C CNN
+F 0 "#PWR30" H 950 2000 50  0001 C CNN
 F 1 "+5V" H 950 2290 50  0000 C CNN
 F 2 "" H 950 2150 50  0000 C CNN
@@
 $EndComp
 $Comp
-L +5V #PWR034
+L +5V #PWR33
 U 1 1 595F65FA
 P 10900 700
-F 0 "#PWR034" H 10900 550 50  0001 C CNN
+F 0 "#PWR33" H 10900 550 50  0001 C CNN
 F 1 "+5V" H 10900 840 50  0000 C CNN
 F 2 "" H 10900 700 50  0000 C CNN
@@
 GIOB3
 $Comp
-L +5V #PWR035
+L +5V #PWR31
 U 1 1 5974EE2F
 P 7450 5550
-F 0 "#PWR035" H 7450 5400 50  0001 C CNN
+F 0 "#PWR31" H 7450 5400 50  0001 C CNN
 F 1 "+5V" H 7450 5690 50  0000 C CNN
 F 2 "" H 7450 5550 50  0000 C CNN
@@
 xGPIO5
 $Comp
-L R_Small 0Ω
+L R_Small 0Ω4
 U 1 1 5AADBCDE
 P 10350 3350
-F 0 "0Ω" H 10380 3370 50  0000 L CNN
+F 0 "0Ω4" H 10380 3370 50  0000 L CNN
 F 1 "R_Small" H 10380 3310 50  0000 L CNN
-F 2 "" H 10350 3350 50  0000 C CNN
+F 2 "SFUSat:R_0402" H 10350 3350 50  0001 C CNN
 F 3 "" H 10350 3350 50  0000 C CNN
 	1    10350 3350
@@
 $EndComp
 $Comp
-L R_Small 0Ω
+L R_Small 0Ω3
 U 1 1 5AADBD42
 P 10350 3200
-F 0 "0Ω" H 10380 3220 50  0000 L CNN
+F 0 "0Ω3" H 10380 3220 50  0000 L CNN
 F 1 "R_Small" H 10380 3160 50  0000 L CNN
-F 2 "" H 10350 3200 50  0000 C CNN
+F 2 "SFUSat:R_0402" H 10350 3200 50  0001 C CNN
 F 3 "" H 10350 3200 50  0000 C CNN
 	1    10350 3200
@@
 $EndComp
 $Comp
-L R_Small 0Ω
+L R_Small 0Ω2
 U 1 1 5AADBD96
 P 10350 3050
-F 0 "0Ω" H 10380 3070 50  0000 L CNN
+F 0 "0Ω2" H 10380 3070 50  0000 L CNN
 F 1 "R_Small" H 10380 3010 50  0000 L CNN
-F 2 "" H 10350 3050 50  0000 C CNN
+F 2 "SFUSat:R_0402" H 10350 3050 50  0001 C CNN
 F 3 "" H 10350 3050 50  0000 C CNN
 	1    10350 3050
@@
 $EndComp
 $Comp
-L R_Small 0Ω
+L R_Small 0Ω1
 U 1 1 5AADBDEC
 P 10350 2900
-F 0 "0Ω" H 10380 2920 50  0000 L CNN
+F 0 "0Ω1" H 10380 2920 50  0000 L CNN
 F 1 "R_Small" H 10380 2860 50  0000 L CNN
-F 2 "" H 10350 2900 50  0000 C CNN
+F 2 "SFUSat:R_0402" H 10350 2900 50  0001 C CNN
 F 3 "" H 10350 2900 50  0000 C CNN
 	1    10350 2900
@@
 	1900 4800 2800 4800
 Wire Wire Line
-	2800 5500 2800 4800
-Wire Wire Line
-	2650 5500 2800 5500
+	2800 4800 2800 5500
+Wire Wire Line
+	2800 5500 2650 5500
 Wire Wire Line
 	2700 5400 2700 5500

Commit message: Cleaned out old stuff
Fixed library references
Parts:
- J1: symbol PC104-8BIT-RESCUE-OBC_05 -> PC104-8BIT
Changed lines of the file:
@@
 EESchema Schematic File Version 2
-LIBS:OBC_05-rescue
 LIBS:power
 LIBS:device
@@
 LIBS:valves
 LIBS:SFUSat
-LIBS:OBC_05-cache
 EELAYER 25 0
 EELAYER END
@@
 $EndDescr
 $Comp
-L PC104-8BIT-RESCUE-OBC_05 J1
+L PC104-8BIT J1
 U 1 1 5955D07C
 P 7900 2850

Commit message: Added 4 more xGPIO
From CAN peripheral. Currently unused
Connections:
- net labels added: xGPIO10, xGPIO11, xGPIO12, xGPIO9
- wire segments 167 -> 177

Commit message: Made 4 layer PCB, WIP: decoupling caps
Parts:
- R38: renamed from 0Ω4; value R_Small -> 0
- R39: renamed from 0Ω3; value R_Small -> 0
- R40: renamed from 0Ω2; value R_Small -> 0
- R41: renamed from 0Ω1; value R_Small -> 0
Connections:
- net labels added: xNHET0, xNHET1
- wire segments 177 -> 183
Changed lines of the file:
@@
 RF_CS2
 $Comp
-L +5V #PWR32
+L +5V #PWR030
 U 1 1 59569513
 P 10100 750
-F 0 "#PWR32" H 10100 600 50  0001 C CNN
+F 0 "#PWR030" H 10100 600 50  0001 C CNN
 F 1 "+5V" H 10100 890 50  0000 C CNN
 F 2 "" H 10100 750 50  0000 C CNN
@@
 $EndComp
 $Comp
-L +5V #PWR30
+L +5V #PWR031
 U 1 1 595F60FC
 P 950 2150
-F 0 "#PWR30" H 950 2000 50  0001 C CNN
+F 0 "#PWR031" H 950 2000 50  0001 C CNN
 F 1 "+5V" H 950 2290 50  0000 C CNN
 F 2 "" H 950 2150 50  0000 C CNN
@@
 $EndComp
 $Comp
-L +5V #PWR33
+L +5V #PWR032
 U 1 1 595F65FA
 P 10900 700
-F 0 "#PWR33" H 10900 550 50  0001 C CNN
+F 0 "#PWR032" H 10900 550 50  0001 C CNN
 F 1 "+5V" H 10900 840 50  0000 C CNN
 F 2 "" H 10900 700 50  0000 C CNN
@@
 GIOB3
 $Comp
-L +5V #PWR31
+L +5V #PWR033
 U 1 1 5974EE2F
 P 7450 5550
-F 0 "#PWR31" H 7450 5400 50  0001 C CNN
+F 0 "#PWR033" H 7450 5400 50  0001 C CNN
 F 1 "+5V" H 7450 5690 50  0000 C CNN
 F 2 "" H 7450 5550 50  0000 C CNN
@@
 xGPIO5
 $Comp
-L R_Small 0Ω4
+L R_Small R38
 U 1 1 5AADBCDE
 P 10350 3350
-F 0 "0Ω4" H 10380 3370 50  0000 L CNN
-F 1 "R_Small" H 10380 3310 50  0000 L CNN
+F 0 "R38" H 10380 3370 50  0000 L CNN
+F 1 "0" H 10380 3310 50  0000 L CNN
 F 2 "SFUSat:R_0402" H 10350 3350 50  0001 C CNN
 F 3 "" H 10350 3350 50  0000 C CNN
@@
 $EndComp
 $Comp
-L R_Small 0Ω3
+L R_Small R39
 U 1 1 5AADBD42
 P 10350 3200
-F 0 "0Ω3" H 10380 3220 50  0000 L CNN
-F 1 "R_Small" H 10380 3160 50  0000 L CNN
+F 0 "R39" H 10380 3220 50  0000 L CNN
+F 1 "0" H 10380 3160 50  0000 L CNN
 F 2 "SFUSat:R_0402" H 10350 3200 50  0001 C CNN
 F 3 "" H 10350 3200 50  0000 C CNN
@@
 $EndComp
 $Comp
-L R_Small 0Ω2
+L R_Small R40
 U 1 1 5AADBD96
 P 10350 3050
-F 0 "0Ω2" H 10380 3070 50  0000 L CNN
-F 1 "R_Small" H 10380 3010 50  0000 L CNN
+F 0 "R40" H 10380 3070 50  0000 L CNN
+F 1 "0" H 10380 3010 50  0000 L CNN
 F 2 "SFUSat:R_0402" H 10350 3050 50  0001 C CNN
 F 3 "" H 10350 3050 50  0000 C CNN
@@
 $EndComp
 $Comp
-L R_Small 0Ω1
+L R_Small R41
 U 1 1 5AADBDEC
 P 10350 2900
-F 0 "0Ω1" H 10380 2920 50  0000 L CNN
-F 1 "R_Small" H 10380 2860 50  0000 L CNN
+F 0 "R41" H 10380 2920 50  0000 L CNN
+F 1 "0" H 10380 2860 50  0000 L CNN
 F 2 "SFUSat:R_0402" H 10350 2900 50  0001 C CNN
 F 3 "" H 10350 2900 50  0000 C CNN
@@
 Wire Wire Line
 	5450 2150 7350 2150
+Text GLabel 6150 2650 0    60   Input ~ 0
+xNHET0
+Text GLabel 6150 2800 0    60   Input ~ 0
+xNHET1
+Wire Wire Line
+	6150 2650 6200 2650
+Wire Wire Line
+	6200 2650 6200 2550
+Wire Wire Line
+	6200 2550 7350 2550
+Wire Wire Line
+	7350 2650 6250 2650
+Wire Wire Line
+	6250 2650 6250 2800
+Wire Wire Line
+	6250 2800 6150 2800
 $EndSCHEMATC

Commit message: Updated power setup
We now either go over USB_5V or through the 104 connector. For flexibility, our own 3V3 header is included, but this is identical to the 104 connector one.
Parts:
- removed D2: PESD5Zx, SFUSat:PESD57zx, symbol PESD5Zx
- removed Q4: DMN2075U, SFUSat:SOT23_DMN2075U, symbol DMN2075U
Connections:
- net labels removed: 104_GND
- wire segments 183 -> 176
Other:
- note added: "USB 5V jumper:\n- if shorted, we use 5V from USB and regulate to 3.3 onboard\n- otherwise: we use 3.3 from the 104 connector"
- note removed: "5v reverse polarity FET"
Changed lines of the file:
@@
 L +5V #PWR030
 U 1 1 59569513
-P 10100 750
-F 0 "#PWR030" H 10100 600 50  0001 C CNN
-F 1 "+5V" H 10100 890 50  0000 C CNN
-F 2 "" H 10100 750 50  0000 C CNN
-F 3 "" H 10100 750 50  0000 C CNN
-	1    10100 750
-	1    0    0    -1
-$EndComp
-Text GLabel 10100 900  3    60   Input ~ 0
+P 9800 950
+F 0 "#PWR030" H 9800 800 50  0001 C CNN
+F 1 "+5V" H 9800 1090 50  0000 C CNN
+F 2 "" H 9800 950 50  0000 C CNN
+F 3 "" H 9800 950 50  0000 C CNN
+	1    9800 950
+	1    0    0    -1
+$EndComp
+Text GLabel 9800 1100 3    60   Input ~ 0
 5v0
 Text Notes 7400 700  0    60   ~ 0
@@
 Text Notes 650  1200 0    60   ~ 0
 Grounding: 104_GND is connected \neither to "GND" net directly, or to GND \nnet through the FET, allowing the load \nto be switched by the SEL mitigation \ncircuit. This is selected by a jumper \non the power page.\n
-Text GLabel 1450 2700 3    60   Input ~ 0
-104_GND
 Text GLabel 9600 1650 2    60   Input ~ 0
 UART_RX
 Text GLabel 9600 1800 2    60   Input ~ 0
 UART_TX
-$Comp
-L DMN2075U Q4
-U 1 1 595F60D8
-P 1450 2250
-F 0 "Q4" V 1150 2150 60  0000 C CNN
-F 1 "DMN2075U" H 1750 2400 60  0000 C CNN
-F 2 "SFUSat:SOT23_DMN2075U" V 1150 2150 60  0001 C CNN
-F 3 "" V 1150 2150 60  0001 C CNN
-	1    1450 2250
-	1    0    0    -1
-$EndComp
-$Comp
-L +5V #PWR031
-U 1 1 595F60FC
-P 950 2150
-F 0 "#PWR031" H 950 2000 50  0001 C CNN
-F 1 "+5V" H 950 2290 50  0000 C CNN
-F 2 "" H 950 2150 50  0000 C CNN
-F 3 "" H 950 2150 50  0000 C CNN
-	1    950  2150
-	1    0    0    -1
-$EndComp
 Text GLabel 8850 4350 2    60   Input ~ 0
 104_In_GND
@@
 Text GLabel 8700 1000 2    60   Input ~ 0
 104_In_GND
-Text GLabel 1550 1700 2    60   Input ~ 0
-104_In_GND
-$Comp
-L PESD5Zx D2
-U 1 1 595F65D3
-P 10900 1050
-F 0 "D2" H 11000 850 60  0000 C CNN
-F 1 "PESD5Zx" H 10650 1150 60  0000 C CNN
-F 2 "SFUSat:PESD57zx" H 10900 1050 60  0001 C CNN
-F 3 "" H 10900 1050 60  0001 C CNN
-	1    10900 1050
-	1    0    0    -1
-$EndComp
-$Comp
-L +5V #PWR032
-U 1 1 595F65FA
-P 10900 700
-F 0 "#PWR032" H 10900 550 50  0001 C CNN
-F 1 "+5V" H 10900 840 50  0000 C CNN
-F 2 "" H 10900 700 50  0000 C CNN
-F 3 "" H 10900 700 50  0000 C CNN
-	1    10900 700
-	1    0    0    -1
-$EndComp
-Text GLabel 10750 1350 0    60   Input ~ 0
-104_In_GND
 Text GLabel 9550 2850 2    60   Input ~ 0
 I2C_SDA
 Text GLabel 9550 3000 2    60   Input ~ 0
 I2C_SCL
-Text Notes 900  3350 0    60   ~ 0
-5v reverse polarity FET
 Text GLabel 9600 1950 2    60   Input ~ 0
 GIOA0
@@
 	8700 1250 8450 1250
 Wire Wire Line
-	10100 750  10100 900
+	9800 950  9800 1100
 Wire Wire Line
 	8700 1000 8700 1250
@@
 Wire Wire Line
 	9150 1800 9600 1800
-Wire Wire Line
-	1450 2550 1450 2700
-Wire Wire Line
-	1050 2250 950  2250
-Wire Wire Line
-	950  2250 950  2150
-Wire Wire Line
-	1550 1700 1450 1700
-Wire Wire Line
-	1450 1700 1450 1950
-Wire Wire Line
-	10900 1350 10750 1350
-Wire Wire Line
-	10900 750  10900 700
 Wire Wire Line
 	8450 2850 9550 2850
@@
 Wire Wire Line
 	6250 2800 6150 2800
+Text Notes 6650 6450 0    60   ~ 0
+USB 5V jumper:\n- if shorted, we use 5V from USB and regulate to 3.3 onboard\n- otherwise: we use 3.3 from the 104 connector
 $EndSCHEMATC
