File: v0.5/PC104_Connector.sch (KiCad schematic (older format))
At the start: 20 parts, among them J1 PC104-8BIT, P11 USB_5V, P6 USB_PORT, U10 FT230XQ-R

Commit message: Routed the nasty stuff
Needs cleanup but the 104 connector is almost done
Other:
- note added: "Connect 0Ω on 41 and 39 \nor 38 and 40.\n\nDefault (expected) config is 0Ω on even labels"
Changed lines of the file:
@@
 RF_CS2
 $Comp
-L +5V #PWR030
+L +5V #PWR028
 U 1 1 59569513
 P 9800 950
-F 0 "#PWR030" H 9800 800 50  0001 C CNN
+F 0 "#PWR028" H 9800 800 50  0001 C CNN
 F 1 "+5V" H 9800 1090 50  0000 C CNN
 F 2 "" H 9800 950 50  0000 C CNN
@@
 GIOB3
 $Comp
-L +5V #PWR033
+L +5V #PWR029
 U 1 1 5974EE2F
 P 7450 5550
-F 0 "#PWR033" H 7450 5400 50  0001 C CNN
+F 0 "#PWR029" H 7450 5400 50  0001 C CNN
 F 1 "+5V" H 7450 5690 50  0000 C CNN
 F 2 "" H 7450 5550 50  0000 C CNN
@@
 Text Notes 6650 6450 0    60   ~ 0
 USB 5V jumper:\n- if shorted, we use 5V from USB and regulate to 3.3 onboard\n- otherwise: we use 3.3 from the 104 connector
+Text Notes 11100 3200 0    60   ~ 0
+Connect 0Ω on 41 and 39 \nor 38 and 40.\n\nDefault (expected) config is 0Ω on even labels
 $EndSCHEMATC

Commit message: FTDI changes
added test point
Parts:
- added W?: TEST_1P, symbol TEST_1P
- J1: symbol PC104-8BIT -> PC104-8BIT-RESCUE-OBC_05
Connections:
- wire segments 176 -> 178
Changed lines of the file:
@@
 EESchema Schematic File Version 2
+LIBS:OBC_05-rescue
 LIBS:power
 LIBS:device
@@
 $EndDescr
 $Comp
-L PC104-8BIT J1
+L PC104-8BIT-RESCUE-OBC_05 J1
 U 1 1 5955D07C
 P 7900 2850
+AR Path="/5955D07C" Ref="J1"  Part="1"
+AR Path="/5955CFBC/5955D07C" Ref="J1"  Part="1"
 F 0 "J1" H 8150 1200 60  0000 C CNN
 F 1 "PC104-8BIT" H 7850 4600 60  0000 C CNN
@@
 Text Notes 11100 3200 0    60   ~ 0
 Connect 0Ω on 41 and 39 \nor 38 and 40.\n\nDefault (expected) config is 0Ω on even labels
+$Comp
+L TEST_1P W?
+U 1 1 5AB36319
+P 9300 6200
+F 0 "W?" H 9300 6470 50  0000 C CNN
+F 1 "TEST_1P" H 9300 6400 50  0000 C CNN
+F 2 "" H 9500 6200 50  0000 C CNN
+F 3 "" H 9500 6200 50  0000 C CNN
+	1    9300 6200
+	1    0    0    -1
+$EndComp
+Wire Wire Line
+	8800 6250 9300 6250
+Wire Wire Line
+	9300 6250 9300 6200
+Connection ~ 8800 6250
 $EndSCHEMATC

Commit message: not finished layout routing
Parts:
- removed U10: FT230XQ-R, SFUSat:QFN-16_650P, symbol FT230XQ-R
- added U10: FTDI_SSOP, SFUSat:16-SSOP, symbol FTDI_SSOP
- P11: symbol CONN_01X02 -> Conn_01x02
- W1: renamed from W?; footprint (none) -> SFUSat:Test_Point
Connections:
- wire segments 178 -> 175

Commit message: fixed 104 and connections in schematic
Parts:
- J1: symbol PC104-8BIT-RESCUE-OBC_05 -> PC104-8BIT
- P11: symbol Conn_01x02 -> CONN_01X02
Connections:
- wire segments 175 -> 177
Changed lines of the file:
@@
 $EndDescr
 $Comp
-L PC104-8BIT-RESCUE-OBC_05 J1
+L PC104-8BIT J1
 U 1 1 5955D07C
 P 7900 2850
@@
 NoConn ~ 8050 5900
 $Comp
-L Conn_01x02 P11
+L CONN_01X02 P11
 U 1 1 597E6761
 P 7800 5400
@@
 L R R36
 U 1 1 5AB488BF
-P 4850 2750
-F 0 "R36" V 4930 2750 50  0000 C CNN
-F 1 "270" V 4850 2750 50  0000 C CNN
-F 2 "SFUSat:R_0402" V 4780 2750 50  0001 C CNN
-F 3 "" H 4850 2750 50  0000 C CNN
-	1    4850 2750
+P 4850 2850
+F 0 "R36" V 4930 2850 50  0000 C CNN
+F 1 "270" V 4850 2850 50  0000 C CNN
+F 2 "SFUSat:R_0402" V 4780 2850 50  0001 C CNN
+F 3 "" H 4850 2850 50  0000 C CNN
+	1    4850 2850
 	1    0    0    -1
 $EndComp
@@
 L LED D4
 U 1 1 5AB489CE
-P 4850 3550
-F 0 "D4" H 4850 3650 50  0000 C CNN
-F 1 "TX" H 4850 3450 50  0000 C CNN
-F 2 "SFUSat:LED_0603" H 4850 3550 50  0001 C CNN
-F 3 "" H 4850 3550 50  0000 C CNN
-	1    4850 3550
+P 4850 3300
+F 0 "D4" H 4850 3400 50  0000 C CNN
+F 1 "TX" H 4850 3200 50  0000 C CNN
+F 2 "SFUSat:LED_0603" H 4850 3300 50  0001 C CNN
+F 3 "" H 4850 3300 50  0000 C CNN
+	1    4850 3300
 	0    -1   -1   0
 $EndComp
@@
 L LED D5
 U 1 1 5AB48A6F
-P 5100 3450
-F 0 "D5" H 5100 3550 50  0000 C CNN
-F 1 "RX" H 5100 3350 50  0000 C CNN
-F 2 "SFUSat:LED_0603" H 5100 3450 50  0001 C CNN
-F 3 "" H 5100 3450 50  0000 C CNN
-	1    5100 3450
+P 5100 3300
+F 0 "D5" H 5100 3400 50  0000 C CNN
+F 1 "RX" H 5100 3200 50  0000 C CNN
+F 2 "SFUSat:LED_0603" H 5100 3300 50  0001 C CNN
+F 3 "" H 5100 3300 50  0000 C CNN
+	1    5100 3300
 	0    -1   -1   0
 $EndComp
@@
 	850  3700 200  3700
 Wire Wire Line
-	5100 2900 5100 3300
-Wire Wire Line
 	3000 3700 4850 3700
 Wire Wire Line
-	5100 3600 5100 3850
+	5100 3500 5100 3850
 Wire Wire Line
 	5100 3850 3000 3850
-Wire Wire Line
-	4850 2900 4850 3400
 Wire Wire Line
 	1350 3800 1150 3800
@@
 Text Label 600  3700 0    60   ~ 0
 RUSB_P
+Wire Wire Line
+	5100 2900 5100 3100
+Wire Wire Line
+	4850 3700 4850 3500
+Wire Wire Line
+	4850 3000 4850 3100
+Wire Wire Line
+	4850 2700 4850 2600
+Connection ~ 4850 2600
 $EndSCHEMATC

Commit message: Routed differential pair
Parts:
- added C37, C38: 47pF, SFUSat:C_0402, symbol C_Small
Connections:
- wire segments 177 -> 181
Changed lines of the file:
@@
 	4850 2700 4850 2600
 Connection ~ 4850 2600
+$Comp
+L C_Small C37
+U 1 1 5ABC920F
+P 2150 5700
+F 0 "C37" H 2160 5770 50  0000 L CNN
+F 1 "47pF" H 2160 5620 50  0000 L CNN
+F 2 "SFUSat:C_0402" H 2150 5700 50  0001 C CNN
+F 3 "" H 2150 5700 50  0000 C CNN
+	1    2150 5700
+	1    0    0    -1
+$EndComp
+$Comp
+L C_Small C38
+U 1 1 5ABC927F
+P 2600 5700
+F 0 "C38" H 2610 5770 50  0000 L CNN
+F 1 "47pF" H 2610 5620 50  0000 L CNN
+F 2 "SFUSat:C_0402" H 2600 5700 50  0001 C CNN
+F 3 "" H 2600 5700 50  0000 C CNN
+	1    2600 5700
+	1    0    0    -1
+$EndComp
+Text GLabel 2150 5400 1    60   Input ~ 0
+USB_N
+Text GLabel 2600 5400 1    60   Input ~ 0
+USB_P
+Text GLabel 2400 6150 3    60   Input ~ 0
+104_In_GND
+Wire Wire Line
+	2150 5800 2600 5800
+Wire Wire Line
+	2400 5800 2400 6150
+Connection ~ 2400 5800
+Wire Wire Line
+	2150 5600 2150 5400
+Wire Wire Line
+	2600 5400 2600 5600
 $EndSCHEMATC

Commit message: FTDI is 3V3 powered now
Before, FTDI was exclusively 5v powered. Since the main supply is now 3.3, we can't do that. Moved to 3.3V
Connections:
- net labels added: +3V3, 3v3
- net labels removed: FTDI_VCCIO
Changed lines of the file:
@@
 L +5V #PWR028
 U 1 1 59569513
-P 9800 950
-F 0 "#PWR028" H 9800 800 50  0001 C CNN
-F 1 "+5V" H 9800 1090 50  0000 C CNN
-F 2 "" H 9800 950 50  0000 C CNN
-F 3 "" H 9800 950 50  0000 C CNN
-	1    9800 950
-	1    0    0    -1
-$EndComp
-Text GLabel 9800 1100 3    60   Input ~ 0
+P 10400 950
+F 0 "#PWR028" H 10400 800 50  0001 C CNN
+F 1 "+5V" H 10400 1090 50  0000 C CNN
+F 2 "" H 10400 950 50  0000 C CNN
+F 3 "" H 10400 950 50  0000 C CNN
+	1    10400 950
+	1    0    0    -1
+$EndComp
+Text GLabel 10400 1100 3    60   Input ~ 0
 5v0
-Text Notes 7400 700  0    60   ~ 0
+Text Notes 7900 700  0    60   ~ 0
 Global Power\nNeeded to connect power on the different sheets\n
 Text Notes 650  1200 0    60   ~ 0
@@
 	8700 1250 8450 1250
 Wire Wire Line
-	9800 950  9800 1100
+	10400 950  10400 1100
 Wire Wire Line
 	8700 1000 8700 1250
@@
 Wire Wire Line
 	3000 2750 4200 2750
-Text GLabel 2300 2250 1    60   Input ~ 0
-FTDI_VCCIO
-Text GLabel 2050 2250 1    60   Input ~ 0
-USB_5V
 $Comp
 L R R36
@@
 Text GLabel 1250 4650 3    60   Input ~ 0
 104_In_GND
-Text GLabel 850  4300 3    60   Input ~ 0
-FTDI_VCCIO
 $Comp
 L C_Small C8
@@
 	2050 2250 2050 2450
 Wire Wire Line
-	2300 2250 2300 2450
-Wire Wire Line
-	1350 2950 1350 1600
-Wire Wire Line
-	1350 1600 2500 1600
-Wire Wire Line
-	2500 1600 2500 2350
-Wire Wire Line
-	2500 2350 2300 2350
-Connection ~ 2300 2350
-Wire Wire Line
-	2500 2250 4550 2250
+	1300 2250 4550 2250
 Wire Wire Line
 	4550 2250 4550 2600
 Wire Wire Line
 	4550 2600 5100 2600
-Connection ~ 2500 2250
 Wire Wire Line
 	3150 2250 3150 2350
@@
 	1350 3800 1150 3800
 Wire Wire Line
-	1150 3800 1150 4150
-Wire Wire Line
-	1150 4150 850  4150
-Wire Wire Line
-	850  4150 850  4300
-Wire Wire Line
-	1100 4200 1100 4150
-Connection ~ 1100 4150
+	1150 4150 1150 3800
+Wire Wire Line
+	800  4150 1150 4150
+Wire Wire Line
+	1100 4150 1100 4200
 Wire Wire Line
 	1100 4400 1100 4450
@@
 Wire Wire Line
 	2600 5400 2600 5600
+$Comp
+L +3V3 #PWR?
+U 1 1 5AD41AA7
+P 2200 2150
+F 0 "#PWR?" H 2200 2000 50  0001 C CNN
+F 1 "+3V3" H 2200 2290 50  0000 C CNN
+F 2 "" H 2200 2150 50  0000 C CNN
+F 3 "" H 2200 2150 50  0000 C CNN
+	1    2200 2150
+	1    0    0    -1
+$EndComp
+Wire Wire Line
+	2200 2250 2200 2150
+Wire Wire Line
+	2300 2250 2300 2450
+Connection ~ 2200 2250
+Connection ~ 2300 2250
+Wire Wire Line
+	1300 2250 1300 2950
+Wire Wire Line
+	1300 2950 1350 2950
+Connection ~ 2050 2250
+$Comp
+L +3V3 #PWR?
+U 1 1 5AD425DA
+P 10750 950
+F 0 "#PWR?" H 10750 800 50  0001 C CNN
+F 1 "+3V3" H 10750 1090 50  0000 C CNN
+F 2 "" H 10750 950 50  0000 C CNN
+F 3 "" H 10750 950 50  0000 C CNN
+	1    10750 950
+	1    0    0    -1
+$EndComp
+Text GLabel 10750 1100 3    60   Input ~ 0
+3v3
+Wire Wire Line
+	10750 950  10750 1100
+$Comp
+L +3V3 #PWR?
+U 1 1 5AD44256
+P 800 4100
+F 0 "#PWR?" H 800 3950 50  0001 C CNN
+F 1 "+3V3" H 800 4240 50  0000 C CNN
+F 2 "" H 800 4100 50  0000 C CNN
+F 3 "" H 800 4100 50  0000 C CNN
+	1    800  4100
+	1    0    0    -1
+$EndComp
+Wire Wire Line
+	800  4150 800  4100
+Connection ~ 1100 4150
 $EndSCHEMATC

Commit message: Added logo, I2c pullup
- i2c now has pullup resistor pads. 
- added big logo on the bottom side
Changed lines of the file:
@@
 RF_CS2
 $Comp
-L +5V #PWR028
+L +5V #PWR31
 U 1 1 59569513
 P 10400 950
-F 0 "#PWR028" H 10400 800 50  0001 C CNN
+F 0 "#PWR31" H 10400 800 50  0001 C CNN
 F 1 "+5V" H 10400 1090 50  0000 C CNN
 F 2 "" H 10400 950 50  0000 C CNN
@@
 GIOB3
 $Comp
-L +5V #PWR029
+L +5V #PWR30
 U 1 1 5974EE2F
 P 7450 5550
-F 0 "#PWR029" H 7450 5400 50  0001 C CNN
+F 0 "#PWR30" H 7450 5400 50  0001 C CNN
 F 1 "+5V" H 7450 5690 50  0000 C CNN
 F 2 "" H 7450 5550 50  0000 C CNN
@@
 	1350 3800 1150 3800
 Wire Wire Line
-	1150 4150 1150 3800
-Wire Wire Line
-	800  4150 1150 4150
+	1150 3800 1150 4150
+Wire Wire Line
+	1150 4150 800  4150
 Wire Wire Line
 	1100 4150 1100 4200
@@
 	2600 5400 2600 5600
 $Comp
-L +3V3 #PWR?
+L +3V3 #PWR29
 U 1 1 5AD41AA7
 P 2200 2150
-F 0 "#PWR?" H 2200 2000 50  0001 C CNN
+F 0 "#PWR29" H 2200 2000 50  0001 C CNN
 F 1 "+3V3" H 2200 2290 50  0000 C CNN
 F 2 "" H 2200 2150 50  0000 C CNN
@@
 Connection ~ 2050 2250
 $Comp
-L +3V3 #PWR?
+L +3V3 #PWR32
 U 1 1 5AD425DA
 P 10750 950
-F 0 "#PWR?" H 10750 800 50  0001 C CNN
+F 0 "#PWR32" H 10750 800 50  0001 C CNN
 F 1 "+3V3" H 10750 1090 50  0000 C CNN
 F 2 "" H 10750 950 50  0000 C CNN
@@
 	10750 950  10750 1100
 $Comp
-L +3V3 #PWR?
+L +3V3 #PWR28
 U 1 1 5AD44256
 P 800 4100
-F 0 "#PWR?" H 800 3950 50  0001 C CNN
+F 0 "#PWR28" H 800 3950 50  0001 C CNN
 F 1 "+3V3" H 800 4240 50  0000 C CNN
 F 2 "" H 800 4100 50  0000 C CNN
