File: v0.5/GPIO.sch (KiCad schematic (older format))
At the start: 6 parts, among them Q5 DMN2075U, U1 TMS570LS0714

Commit message: Removed extraneous 104 connections
Connections:
- net labels removed: ANTENNA_DEPLOY
- wire segments 19 -> 20
Changed lines of the file:
@@
 $Descr A4 11693 8268
 encoding utf-8
-Sheet 9 12
+Sheet 9 13
 Title ""
 Date ""
@@
 WATCHDOG
 Wire Wire Line
-	4250 2600 5750 2600
+	4250 2600 4400 2600
+Wire Wire Line
+	4400 2600 4700 2600
+Wire Wire Line
+	4700 2600 5750 2600
 $Comp
 L R R26
@@
 Wire Wire Line
 	5600 2150 5750 2150
-Text GLabel 5600 2450 0    60   Input ~ 0
-ANTENNA_DEPLOY
-Wire Wire Line
-	5600 2450 5750 2450
 Text GLabel 5550 2750 0    60   Input ~ 0
 GIOB1

Commit message: Added required xGPIO, removed 5V from 104 connector
Connections:
- net labels added: xGPIO7
- wire segments 20 -> 19
Changed lines of the file:
@@
 WATCHDOG
 Wire Wire Line
-	4250 2600 4400 2600
-Wire Wire Line
-	4400 2600 4700 2600
-Wire Wire Line
-	4700 2600 5750 2600
+	4250 2600 5750 2600
 $Comp
 L R R26
@@
 Wire Wire Line
 	2400 3250 2600 3250
+Text GLabel 5600 2450 0    60   Input ~ 0
+xGPIO7
+Wire Wire Line
+	5750 2450 5600 2450
 $EndSCHEMATC
