File: v0.5/bulk_power.sch (KiCad schematic (older format))
At the start: 39 parts, among them P1 3v3_IN_CONNECTOR, P12 LOAD, P2 INA_INPUT, P3 INA_GND, P4 INA_EN, P5 INA_OUTPUT, Q1 DMN2075U, Q2 DMN2075U, Q3 1v2_GOOD, U1 TMS570LS0714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

Commit message: Updated 1.2v regulator, removed DC jack
Parts:
- removed U2: XC6222B121MR-G, SFUSat:SOT25, symbol AP7331
- added U2: MCP1825S, SFUSat:SOT-223, symbol MCP1825S
- C2: value 10µF -> 1µF
- C21: value 1µF -> 4.7µF
Connections:
- wire segments 107 -> 101
- no-connect marks 1 -> 0
Changed lines of the file:
@@
 EESchema Schematic File Version 2
+LIBS:OBC_05-rescue
 LIBS:power
 LIBS:device
@@
 LIBS:valves
 LIBS:SFUSat
-LIBS:OBC_04-cache
+LIBS:OBC_05-cache
 EELAYER 25 0
 EELAYER END
@@
 $EndDescr
 $Comp
-L AP7331 U2
-U 1 1 594C86F3
-P 7700 1200
-F 0 "U2" H 7700 1100 60  0000 C CNN
-F 1 "XC6222B121MR-G" H 7700 1450 60  0000 C CNN
-F 2 "SFUSat:SOT25" H 7700 1100 60  0001 C CNN
-F 3 "" H 7700 1100 60  0001 C CNN
-	1    7700 1200
-	1    0    0    -1
-$EndComp
-$Comp
 L CONN_01X02 P1
 U 1 1 594C872A
@@
 L C C2
 U 1 1 594C879F
-P 8500 1350
-F 0 "C2" H 8525 1450 50  0000 L CNN
-F 1 "10µF" H 8525 1250 50  0000 L CNN
-F 2 "SFUSat:C_0402" H 8538 1200 50  0001 C CNN
-F 3 "" H 8500 1350 50  0000 C CNN
-	1    8500 1350
-	1    0    0    -1
-$EndComp
-Text GLabel 8500 800  1    60   Input ~ 0
+P 7950 2050
+F 0 "C2" H 7975 2150 50  0000 L CNN
+F 1 "1µF" H 7975 1950 50  0000 L CNN
+F 2 "SFUSat:C_0402" H 7988 1900 50  0001 C CNN
+F 3 "" H 7950 2050 50  0000 C CNN
+	1    7950 2050
+	1    0    0    -1
+$EndComp
+Text GLabel 8050 1750 2    60   Input ~ 0
 1v2
-Wire Wire Line
-	8500 1050 8150 1050
-Wire Wire Line
-	8500 800  8500 1200
-Connection ~ 8500 1050
-Wire Wire Line
-	8500 1500 8500 1750
-Wire Wire Line
-	6850 1050 7250 1050
 Text GLabel 1000 900  3    60   Input ~ 0
 3v3
 Wire Wire Line
 	1050 2100 950  2100
-Wire Wire Line
-	7100 800  7100 1050
-Connection ~ 7100 1050
-Wire Wire Line
-	6850 1350 6850 1500
-Wire Wire Line
-	7250 1200 7100 1200
-Wire Wire Line
-	7100 1200 7100 1400
-Wire Wire Line
-	7100 1400 6850 1400
-Connection ~ 6850 1400
-Wire Wire Line
-	7250 1350 7200 1350
-Wire Wire Line
-	7200 1350 7200 1050
-Connection ~ 7200 1050
 $Comp
 L C C21
 U 1 1 594C8CAA
-P 6850 1200
-F 0 "C21" H 6875 1300 50  0000 L CNN
-F 1 "1µF" H 6875 1100 50  0000 L CNN
-F 2 "SFUSat:C_0402" H 6888 1050 50  0001 C CNN
-F 3 "" H 6850 1200 50  0000 C CNN
-	1    6850 1200
-	1    0    0    -1
-$EndComp
-NoConn ~ 8250 1200
-Wire Wire Line
-	8150 1200 8250 1200
+P 7200 1100
+F 0 "C21" H 7225 1200 50  0000 L CNN
+F 1 "4.7µF" H 7225 1000 50  0000 L CNN
+F 2 "SFUSat:C_0402" H 7238 950 50  0001 C CNN
+F 3 "" H 7200 1100 50  0000 C CNN
+	1    7200 1100
+	1    0    0    -1
+$EndComp
 $Comp
 L TMS570LS0714 U?
@@
 Wire Wire Line
 	6750 5250 7050 5250
-Text Notes 7450 800  0    60   ~ 0
+Text Notes 7550 750  0    60   ~ 0
 1.2v regulator\n
 Wire Wire Line
@@
 L +1V2 #PWR05
 U 1 1 595698EB
-P 8750 750
-F 0 "#PWR05" H 8750 600 50  0001 C CNN
-F 1 "+1V2" H 8750 890 50  0000 C CNN
-F 2 "" H 8750 750 50  0000 C CNN
-F 3 "" H 8750 750 50  0000 C CNN
-	1    8750 750
+P 7700 1750
+F 0 "#PWR05" H 7700 1600 50  0001 C CNN
+F 1 "+1V2" H 7700 1890 50  0000 C CNN
+F 2 "" H 7700 1750 50  0000 C CNN
+F 3 "" H 7700 1750 50  0000 C CNN
+	1    7700 1750
 	1    0    0    -1
 $EndComp
@@
 L GND #PWR06
 U 1 1 595699CF
-P 6850 1500
-F 0 "#PWR06" H 6850 1250 50  0001 C CNN
-F 1 "GND" H 6850 1350 50  0000 C CNN
-F 2 "" H 6850 1500 50  0000 C CNN
-F 3 "" H 6850 1500 50  0000 C CNN
-	1    6850 1500
-	1    0    0    -1
-$EndComp
-Wire Wire Line
-	8750 850  8750 750
-Wire Wire Line
-	8750 850  8500 850
-Connection ~ 8500 850
+P 7200 1350
+F 0 "#PWR06" H 7200 1100 50  0001 C CNN
+F 1 "GND" H 7200 1200 50  0000 C CNN
+F 2 "" H 7200 1350 50  0000 C CNN
+F 3 "" H 7200 1350 50  0000 C CNN
+	1    7200 1350
+	1    0    0    -1
+$EndComp
 $Comp
 L +3V3 #PWR07
 U 1 1 59569C16
-P 7100 800
-F 0 "#PWR07" H 7100 650 50  0001 C CNN
-F 1 "+3V3" H 7100 940 50  0000 C CNN
-F 2 "" H 7100 800 50  0000 C CNN
-F 3 "" H 7100 800 50  0000 C CNN
-	1    7100 800
+P 7750 950
+F 0 "#PWR07" H 7750 800 50  0001 C CNN
+F 1 "+3V3" H 7750 1090 50  0000 C CNN
+F 2 "" H 7750 950 50  0000 C CNN
+F 3 "" H 7750 950 50  0000 C CNN
+	1    7750 950
 	1    0    0    -1
 $EndComp
@@
 L GND #PWR019
 U 1 1 5956AAB6
-P 8500 1750
-F 0 "#PWR019" H 8500 1500 50  0001 C CNN
-F 1 "GND" H 8500 1600 50  0000 C CNN
-F 2 "" H 8500 1750 50  0000 C CNN
-F 3 "" H 8500 1750 50  0000 C CNN
-	1    8500 1750
+P 7950 2350
+F 0 "#PWR019" H 7950 2100 50  0001 C CNN
+F 1 "GND" H 7950 2200 50  0000 C CNN
+F 2 "" H 7950 2350 50  0000 C CNN
+F 3 "" H 7950 2350 50  0000 C CNN
+	1    7950 2350
 	1    0    0    -1
 $EndComp
@@
 Wire Wire Line
 	3850 2150 4650 2150
-Text Notes 5050 2050 0    60   ~ 0
-INA_POWER_ENABLE\nShort this connector if using INA\nPrevents INA from being powered \nwhen it is supposed to be disconnected
 Wire Wire Line
 	1000 3850 1150 3850
@@
 Text Notes 6200 4200 0    60   ~ 0
 For load testing the current limit\n
+$Comp
+L MCP1825S U2
+U 1 1 5AAD94D2
+P 8550 1250
+F 0 "U2" H 8700 1150 60  0000 C CNN
+F 1 "MCP1825S" H 8600 1500 60  0000 C CNN
+F 2 "SFUSat:SOT-223" H 8350 1650 60  0001 C CNN
+F 3 "" H 8350 1650 60  0001 C CNN
+	1    8550 1250
+	1    0    0    -1
+$EndComp
+Wire Wire Line
+	7200 950  7950 950
+Wire Wire Line
+	7950 950  7950 1000
+Connection ~ 7750 950
+Wire Wire Line
+	7200 1250 7200 1350
+Wire Wire Line
+	7950 1300 7950 1150
+Wire Wire Line
+	7950 1250 7200 1250
+Connection ~ 7950 1250
+Wire Wire Line
+	7950 1450 7950 1900
+Wire Wire Line
+	7700 1750 8050 1750
+Connection ~ 7950 1750
+Wire Wire Line
+	7950 2200 7950 2350
+Text Notes 5050 2050 0    60   ~ 0
+INA_POWER_ENABLE\nShort this connector if using INA\nPrevents INA from being powered \nwhen it is supposed to be disconnected
 $EndSCHEMATC

Commit message: Added 4 more xGPIO
From CAN peripheral. Currently unused
Other:
- note added: "Add connection to \nthe 104 3.3v here"
Changed lines of the file:
@@
 LIBS:valves
 LIBS:SFUSat
+LIBS:OBC_05-cache
 EELAYER 25 0
 EELAYER END
@@
 Text Notes 5050 2050 0    60   ~ 0
 INA_POWER_ENABLE\nShort this connector if using INA\nPrevents INA from being powered \nwhen it is supposed to be disconnected
+Text Notes 250  2650 0    60   ~ 0
+Add connection to \nthe 104 3.3v here
 $EndSCHEMATC

Commit message: Made 4 layer PCB, WIP: decoupling caps
Parts:
- added C3: 0.1µF, SFUSat:C_0402, symbol C_Small
Other:
- note added: "C8 were removed at the board level, as multiple pins were connected to one cap."
- note removed: "C1, C3, C8 were removed at the board level, as multiple pins were connected to one cap."
Changed lines of the file:
@@
 	7800 4900 7800 5100
 $Comp
-L GND #PWR24
+L GND #PWR01
 U 1 1 595695D8
 P 7800 5450
-F 0 "#PWR24" H 7800 5200 50  0001 C CNN
+F 0 "#PWR01" H 7800 5200 50  0001 C CNN
 F 1 "GND" H 7800 5300 50  0000 C CNN
 F 2 "" H 7800 5450 50  0000 C CNN
@@
 $EndComp
 $Comp
-L +3V3 #PWR4
+L +3V3 #PWR02
 U 1 1 59569610
 P 1000 800
-F 0 "#PWR4" H 1000 650 50  0001 C CNN
+F 0 "#PWR02" H 1000 650 50  0001 C CNN
 F 1 "+3V3" H 1000 940 50  0000 C CNN
 F 2 "" H 1000 800 50  0000 C CNN
@@
 	1000 800  1000 900
 $Comp
-L +3V3 #PWR3
+L +3V3 #PWR03
 U 1 1 595697BF
 P 800 2250
-F 0 "#PWR3" H 800 2100 50  0001 C CNN
+F 0 "#PWR03" H 800 2100 50  0001 C CNN
 F 1 "+3V3" H 800 2390 50  0000 C CNN
 F 2 "" H 800 2250 50  0000 C CNN
@@
 $EndComp
 $Comp
-L GND #PWR6
+L GND #PWR04
 U 1 1 59569803
 P 1450 2800
-F 0 "#PWR6" H 1450 2550 50  0001 C CNN
+F 0 "#PWR04" H 1450 2550 50  0001 C CNN
 F 1 "GND" H 1450 2650 50  0000 C CNN
 F 2 "" H 1450 2800 50  0000 C CNN
@@
 	950  2250 800  2250
 $Comp
-L +1V2 #PWR21
+L +1V2 #PWR05
 U 1 1 595698EB
 P 7700 1750
-F 0 "#PWR21" H 7700 1600 50  0001 C CNN
+F 0 "#PWR05" H 7700 1600 50  0001 C CNN
 F 1 "+1V2" H 7700 1890 50  0000 C CNN
 F 2 "" H 7700 1750 50  0000 C CNN
@@
 $EndComp
 $Comp
-L GND #PWR18
+L GND #PWR06
 U 1 1 595699CF
 P 7200 1350
-F 0 "#PWR18" H 7200 1100 50  0001 C CNN
+F 0 "#PWR06" H 7200 1100 50  0001 C CNN
 F 1 "GND" H 7200 1200 50  0000 C CNN
 F 2 "" H 7200 1350 50  0000 C CNN
@@
 $EndComp
 $Comp
-L +3V3 #PWR22
+L +3V3 #PWR07
 U 1 1 59569C16
 P 7750 950
-F 0 "#PWR22" H 7750 800 50  0001 C CNN
+F 0 "#PWR07" H 7750 800 50  0001 C CNN
 F 1 "+3V3" H 7750 1090 50  0000 C CNN
 F 2 "" H 7750 950 50  0000 C CNN
@@
 $EndComp
 $Comp
-L GND #PWR2
+L GND #PWR08
 U 1 1 59569D86
 P 750 6650
-F 0 "#PWR2" H 750 6400 50  0001 C CNN
+F 0 "#PWR08" H 750 6400 50  0001 C CNN
 F 1 "GND" H 750 6500 50  0000 C CNN
 F 2 "" H 750 6650 50  0000 C CNN
@@
 $EndComp
 $Comp
-L GND #PWR7
+L GND #PWR09
 U 1 1 59569E21
 P 1950 6650
-F 0 "#PWR7" H 1950 6400 50  0001 C CNN
+F 0 "#PWR09" H 1950 6400 50  0001 C CNN
 F 1 "GND" H 1950 6500 50  0000 C CNN
 F 2 "" H 1950 6650 50  0000 C CNN
@@
 $EndComp
 $Comp
-L +1V2 #PWR11
+L +1V2 #PWR010
 U 1 1 59569E8C
 P 3250 6050
-F 0 "#PWR11" H 3250 5900 50  0001 C CNN
+F 0 "#PWR010" H 3250 5900 50  0001 C CNN
 F 1 "+1V2" H 3250 6190 50  0000 C CNN
 F 2 "" H 3250 6050 50  0000 C CNN
@@
 	3450 6050 3250 6050
 $Comp
-L +1V2 #PWR12
+L +1V2 #PWR011
 U 1 1 59569FC3
 P 4750 6050
-F 0 "#PWR12" H 4750 5900 50  0001 C CNN
+F 0 "#PWR011" H 4750 5900 50  0001 C CNN
 F 1 "+1V2" H 4750 6190 50  0000 C CNN
 F 2 "" H 4750 6050 50  0000 C CNN
@@
 	4600 6050 4750 6050
 $Comp
-L +3V3 #PWR13
+L +3V3 #PWR012
 U 1 1 5956A06D
 P 5300 5250
-F 0 "#PWR13" H 5300 5100 50  0001 C CNN
+F 0 "#PWR012" H 5300 5100 50  0001 C CNN
 F 1 "+3V3" H 5300 5390 50  0000 C CNN
 F 2 "" H 5300 5250 50  0000 C CNN
@@
 $EndComp
 $Comp
-L +3V3 #PWR17
+L +3V3 #PWR013
 U 1 1 5956A12A
 P 7050 5250
-F 0 "#PWR17" H 7050 5100 50  0001 C CNN
+F 0 "#PWR013" H 7050 5100 50  0001 C CNN
 F 1 "+3V3" H 7050 5390 50  0000 C CNN
 F 2 "" H 7050 5250 50  0000 C CNN
@@
 $EndComp
 $Comp
-L +3V3 #PWR23
+L +3V3 #PWR014
 U 1 1 5956A1DB
 P 7800 4900
-F 0 "#PWR23" H 7800 4750 50  0001 C CNN
+F 0 "#PWR014" H 7800 4750 50  0001 C CNN
 F 1 "+3V3" H 7800 5040 50  0000 C CNN
 F 2 "" H 7800 4900 50  0000 C CNN
@@
 $EndComp
 Wire Wire Line
-	7150 6000 7750 6000
+	6850 6000 7750 6000
 Connection ~ 7350 6000
 Wire Wire Line
 	7350 6000 7350 6150
 Wire Wire Line
-	7150 5800 7750 5800
+	6850 5800 7750 5800
 Connection ~ 7350 5800
 Wire Wire Line
 	7350 5600 7350 5800
 $Comp
-L GND #PWR20
+L GND #PWR015
 U 1 1 5956A394
 P 7350 6150
-F 0 "#PWR20" H 7350 5900 50  0001 C CNN
+F 0 "#PWR015" H 7350 5900 50  0001 C CNN
 F 1 "GND" H 7350 6000 50  0000 C CNN
 F 2 "" H 7350 6150 50  0000 C CNN
@@
 $EndComp
 $Comp
-L +3V3 #PWR19
+L +3V3 #PWR016
 U 1 1 5956A39A
 P 7350 5600
-F 0 "#PWR19" H 7350 5450 50  0001 C CNN
+F 0 "#PWR016" H 7350 5450 50  0001 C CNN
 F 1 "+3V3" H 7350 5740 50  0000 C CNN
 F 2 "" H 7350 5600 50  0000 C CNN
@@
 	2750 6150 2750 6350
 $Comp
-L GND #PWR10
+L GND #PWR017
 U 1 1 5956A940
 P 2750 6700
-F 0 "#PWR10" H 2750 6450 50  0001 C CNN
+F 0 "#PWR017" H 2750 6450 50  0001 C CNN
 F 1 "GND" H 2750 6550 50  0000 C CNN
 F 2 "" H 2750 6700 50  0000 C CNN
@@
 5v0
 $Comp
-L +5V #PWR1
+L +5V #PWR018
 U 1 1 595699C9
 P 750 800
-F 0 "#PWR1" H 750 650 50  0001 C CNN
+F 0 "#PWR018" H 750 650 50  0001 C CNN
 F 1 "+5V" H 750 940 50  0000 C CNN
 F 2 "" H 750 800 50  0000 C CNN
@@
 $EndComp
 $Comp
-L GND #PWR25
+L GND #PWR019
 U 1 1 5956AAB6
 P 7950 2350
-F 0 "#PWR25" H 7950 2100 50  0001 C CNN
+F 0 "#PWR019" H 7950 2100 50  0001 C CNN
 F 1 "GND" H 7950 2200 50  0000 C CNN
 F 2 "" H 7950 2350 50  0000 C CNN
@@
 $EndComp
 $Comp
-L +5V #PWR8
+L +5V #PWR020
 U 1 1 5956AE0D
 P 2450 750
-F 0 "#PWR8" H 2450 600 50  0001 C CNN
+F 0 "#PWR020" H 2450 600 50  0001 C CNN
 F 1 "+5V" H 2450 890 50  0000 C CNN
 F 2 "" H 2450 750 50  0000 C CNN
@@
 	5300 2650 5750 2650
 $Comp
-L +3V3 #PWR14
+L +3V3 #PWR021
 U 1 1 595A8DFE
 P 5750 2650
-F 0 "#PWR14" H 5750 2500 50  0001 C CNN
+F 0 "#PWR021" H 5750 2500 50  0001 C CNN
 F 1 "+3V3" H 5750 2790 50  0000 C CNN
 F 2 "" H 5750 2650 50  0000 C CNN
@@
 3v3_OUTPUT
 $Comp
-L +3V3 #PWR5
+L +3V3 #PWR022
 U 1 1 595A95DC
 P 1150 3850
-F 0 "#PWR5" H 1150 3700 50  0001 C CNN
+F 0 "#PWR022" H 1150 3700 50  0001 C CNN
 F 1 "+3V3" H 1150 3990 50  0000 C CNN
 F 2 "" H 1150 3850 50  0000 C CNN
@@
 104_GND
 $Comp
-L GND #PWR27
+L GND #PWR023
 U 1 1 595B0A44
 P 10000 4050
-F 0 "#PWR27" H 10000 3800 50  0001 C CNN
+F 0 "#PWR023" H 10000 3800 50  0001 C CNN
 F 1 "GND" H 10000 3900 50  0000 C CNN
 F 2 "" H 10000 4050 50  0000 C CNN
@@
 	10450 1700 10450 1800
 $Comp
-L +1V2 #PWR26
+L +1V2 #PWR024
 U 1 1 5965C95D
 P 9900 2550
-F 0 "#PWR26" H 9900 2400 50  0001 C CNN
+F 0 "#PWR024" H 9900 2400 50  0001 C CNN
 F 1 "+1V2" H 9900 2690 50  0000 C CNN
 F 2 "" H 9900 2550 50  0000 C CNN
@@
 $EndComp
 $Comp
-L GND #PWR28
+L GND #PWR025
 U 1 1 5965C9F5
 P 10250 3100
-F 0 "#PWR28" H 10250 2850 50  0001 C CNN
+F 0 "#PWR025" H 10250 2850 50  0001 C CNN
 F 1 "GND" H 10250 2950 50  0000 C CNN
 F 2 "" H 10250 3100 50  0000 C CNN
@@
 $EndComp
 $Comp
-L +3V3 #PWR29
+L +3V3 #PWR026
 U 1 1 5965CA8D
 P 10450 1250
-F 0 "#PWR29" H 10450 1100 50  0001 C CNN
+F 0 "#PWR026" H 10450 1100 50  0001 C CNN
 F 1 "+3V3" H 10450 1390 50  0000 C CNN
 F 2 "" H 10450 1250 50  0000 C CNN
@@
 Connection ~ 9900 2600
 $Comp
-L +1V2 #PWR9
+L +1V2 #PWR027
 U 1 1 59725D84
 P 2750 6150
-F 0 "#PWR9" H 2750 6000 50  0001 C CNN
+F 0 "#PWR027" H 2750 6000 50  0001 C CNN
 F 1 "+1V2" H 2750 6290 50  0000 C CNN
 F 2 "" H 2750 6150 50  0000 C CNN
@@
 	2750 6550 4750 6550
 Text Notes 3050 6750 0    60   ~ 0
-C1, C3, C8 were removed at the board level, as multiple pins were connected to one cap.
+C8 were removed at the board level, as multiple pins were connected to one cap.
 Wire Wire Line
 	3600 3850 3900 3850
@@
 $EndComp
 $Comp
-L +3V3 #PWR15
+L +3V3 #PWR028
 U 1 1 5A646F64
 P 6900 3600
-F 0 "#PWR15" H 6900 3450 50  0001 C CNN
+F 0 "#PWR028" H 6900 3450 50  0001 C CNN
 F 1 "+3V3" H 6900 3740 50  0000 C CNN
 F 2 "" H 6900 3600 50  0000 C CNN
@@
 $EndComp
 $Comp
-L GND #PWR16
+L GND #PWR029
 U 1 1 5A6470B7
 P 6900 3850
-F 0 "#PWR16" H 6900 3600 50  0001 C CNN
+F 0 "#PWR029" H 6900 3600 50  0001 C CNN
 F 1 "GND" H 6900 3700 50  0000 C CNN
 F 2 "" H 6900 3850 50  0000 C CNN
@@
 Text Notes 250  2650 0    60   ~ 0
 Add connection to \nthe 104 3.3v here
+$Comp
+L C_Small C3
+U 1 1 5AAEB815
+P 6850 5900
+F 0 "C3" H 6860 5970 50  0000 L CNN
+F 1 "0.1µF" H 6860 5820 50  0000 L CNN
+F 2 "SFUSat:C_0402" H 6850 5900 50  0001 C CNN
+F 3 "" H 6850 5900 50  0000 C CNN
+	1    6850 5900
+	1    0    0    -1
+$EndComp
+Connection ~ 7150 5800
+Connection ~ 7150 6000
 $EndSCHEMATC

Commit message: Updated power setup
We now either go over USB_5V or through the 104 connector. For flexibility, our own 3V3 header is included, but this is identical to the 104 connector one.
Connections:
- net labels added: 104_3v3
- wire segments 101 -> 105
Other:
- note added: "Either use 3V3 from 104 (or our power header, they're identical),\nor short USB_5V and don't have any 3V3 on the 104 connector or \nour power header."
- note added: "Normal mode: connect pins 3 and 1\nINA off: remove the resistor"
- note added: "OBC power header for\nflexibility if 104 is blocked"
- note removed: "Add connection to \nthe 104 3.3v here"
Changed lines of the file:
@@
 L CONN_01X02 P1
 U 1 1 594C872A
-P 1100 1900
+P 1050 1500
 AR Path="/594C7FEF/594C872A" Ref="P1"  Part="1"
 AR Path="/5955FC9A/594C872A" Ref="P1"  Part="1"
-F 0 "P1" H 1100 2050 50  0000 C CNN
-F 1 "3v3_IN_CONNECTOR" V 1200 1900 50  0000 C CNN
-F 2 "SFUSat:2x01In_Header_v2" H 1100 1900 50  0001 C CNN
-F 3 "" H 1100 1900 50  0000 C CNN
-	1    1100 1900
+F 0 "P1" H 1050 1650 50  0000 C CNN
+F 1 "3v3_IN_CONNECTOR" V 1150 1500 50  0000 C CNN
+F 2 "SFUSat:2x01In_Header_v2" H 1050 1500 50  0001 C CNN
+F 3 "" H 1050 1500 50  0000 C CNN
+	1    1050 1500
 	0    -1   -1   0
 $EndComp
@@
 Text GLabel 1000 900  3    60   Input ~ 0
 3v3
-Wire Wire Line
-	1050 2100 950  2100
 $Comp
 L C C21
@@
 Text GLabel 1150 3950 2    60   Input ~ 0
 3v3_OUTPUT
-Text GLabel 2200 1100 1    60   Input ~ 0
-3v3_OUTPUT
 $Comp
 L +3V3 #PWR022
@@
 $EndComp
 Wire Wire Line
-	1150 2100 1450 2100
+	1100 2100 1450 2100
 Wire Wire Line
 	950  2400 1050 2400
@@
 Text Notes 5050 2050 0    60   ~ 0
 INA_POWER_ENABLE\nShort this connector if using INA\nPrevents INA from being powered \nwhen it is supposed to be disconnected
-Text Notes 250  2650 0    60   ~ 0
-Add connection to \nthe 104 3.3v here
 $Comp
 L C_Small C3
@@
 Connection ~ 7150 5800
 Connection ~ 7150 6000
+Text Notes 550  4350 0    60   ~ 0
+Normal mode: connect pins 3 and 1\nINA off: remove the resistor
+Text GLabel 1200 1850 2    60   Input ~ 0
+104_GND
+Text GLabel 950  1900 0    60   Input ~ 0
+104_3v3
+Wire Wire Line
+	1000 1700 1000 2100
+Wire Wire Line
+	1000 1900 950  1900
+Connection ~ 1000 1900
+Wire Wire Line
+	1000 2100 950  2100
+Wire Wire Line
+	1100 1700 1100 2100
+Wire Wire Line
+	1200 1850 1100 1850
+Connection ~ 1100 1850
+Text Notes -400 1750 0    60   ~ 0
+OBC power header for\nflexibility if 104 is blocked
+$Comp
+L +3V3 #PWR?
+U 1 1 5AAF4886
+P 2200 1100
+F 0 "#PWR?" H 2200 950 50  0001 C CNN
+F 1 "+3V3" H 2200 1240 50  0000 C CNN
+F 2 "" H 2200 1100 50  0000 C CNN
+F 3 "" H 2200 1100 50  0000 C CNN
+	1    2200 1100
+	1    0    0    -1
+$EndComp
+Text Notes 3750 850  0    60   ~ 0
+Either use 3V3 from 104 (or our power header, they're identical),\nor short USB_5V and don't have any 3V3 on the 104 connector or \nour power header.
 $EndSCHEMATC

Commit message: Routed the nasty stuff
Needs cleanup but the 104 connector is almost done
Parts:
- added C34, C35, C36: 0.1µF, SFUSat:C_0402, symbol C_Small
Connections:
- net labels added: 104_In_GND, 3v3_before_shunt
- net labels removed: 3v3_OUTPUT
Other:
- note added: "Either connect 3v3 before shunt to \nthe top end of the shunt, or we bypass \nthe shunt and connect right to 3V3 net.\n\n"
- note removed: "Normal mode: connect pins 3 and 1\nINA off: remove the resistor"
