File: v0.5/bulk_power.sch (KiCad schematic (older format))
At the start: 43 parts, among them P1 3v3_IN_CONNECTOR, P12 LOAD, P2 INA_INPUT, P3 INA_GND, P4 INA_EN, P5 INA_OUTPUT, Q1 DMN2075U, Q2 DMN2075U, Q3 1v2_GOOD, U1 TMS570LS0714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

Commit message: not finished layout routing
Parts:
- P1, P12, P4, P5: symbol CONN_01X02 -> Conn_01x02
- P2, P3: symbol CONN_01X03 -> Conn_01x03
Changed lines of the file:
@@
 $EndDescr
 $Comp
-L CONN_01X02 P1
+L Conn_01x02 P1
 U 1 1 594C872A
 P 1050 1500
 AR Path="/594C7FEF/594C872A" Ref="P1"  Part="1"
 AR Path="/5955FC9A/594C872A" Ref="P1"  Part="1"
+AR Path="/594C872A" Ref="P1"  Part="1"
 F 0 "P1" H 1050 1650 50  0000 C CNN
 F 1 "3v3_IN_CONNECTOR" V 1150 1500 50  0000 C CNN
@@
 $EndComp
 $Comp
-L CONN_01X03 P2
+L Conn_01x03 P2
 U 1 1 595A8F65
 P 800 3950
@@
 $EndComp
 $Comp
-L CONN_01X03 P3
+L Conn_01x03 P3
 U 1 1 595A901D
 P 9350 4050
@@
 INA_OUT
 $Comp
-L CONN_01X02 P5
+L Conn_01x02 P5
 U 1 1 595B2CF2
 P 850 3250
+AR Path="/595B2CF2" Ref="P5"  Part="1"
+AR Path="/594C7FEF/595B2CF2" Ref="P5"  Part="1"
 F 0 "P5" H 850 3400 50  0000 C CNN
 F 1 "INA_OUTPUT" V 950 3250 50  0000 C CNN
@@
 C8 were removed at the board level, as multiple pins were connected to one cap.
 $Comp
-L CONN_01X02 P12
+L Conn_01x02 P12
 U 1 1 5A646879
 P 6500 3700
+AR Path="/5A646879" Ref="P12"  Part="1"
+AR Path="/594C7FEF/5A646879" Ref="P12"  Part="1"
 F 0 "P12" H 6500 3850 50  0000 C CNN
 F 1 "LOAD" V 6600 3700 50  0000 C CNN
@@
 Either connect 3v3 before shunt to \nthe top end of the shunt, or we bypass \nthe shunt and connect right to 3V3 net.\n\n
 $Comp
-L CONN_01X02 P4
+L Conn_01x02 P4
 U 1 1 5AAFC0C3
 P 4400 1900
+AR Path="/5AAFC0C3" Ref="P4"  Part="1"
+AR Path="/594C7FEF/5AAFC0C3" Ref="P4"  Part="1"
 F 0 "P4" H 4400 2050 50  0000 C CNN
 F 1 "INA_EN" V 4500 1900 50  0000 C CNN

Commit message: fixed 104 and connections in schematic
Parts:
- P1, P12, P4, P5: symbol Conn_01x02 -> CONN_01X02
- P2, P3: symbol Conn_01x03 -> CONN_01X03
Changed lines of the file:
@@
 $EndDescr
 $Comp
-L Conn_01x02 P1
+L CONN_01X02 P1
 U 1 1 594C872A
 P 1050 1500
@@
 $EndComp
 $Comp
-L Conn_01x03 P2
+L CONN_01X03 P2
 U 1 1 595A8F65
 P 800 3950
@@
 $EndComp
 $Comp
-L Conn_01x03 P3
+L CONN_01X03 P3
 U 1 1 595A901D
 P 9350 4050
@@
 INA_OUT
 $Comp
-L Conn_01x02 P5
+L CONN_01X02 P5
 U 1 1 595B2CF2
 P 850 3250
@@
 C8 were removed at the board level, as multiple pins were connected to one cap.
 $Comp
-L Conn_01x02 P12
+L CONN_01X02 P12
 U 1 1 5A646879
 P 6500 3700
@@
 Either connect 3v3 before shunt to \nthe top end of the shunt, or we bypass \nthe shunt and connect right to 3V3 net.\n\n
 $Comp
-L Conn_01x02 P4
+L CONN_01X02 P4
 U 1 1 5AAFC0C3
 P 4400 1900

Commit message: Added slot-accessible 3v3 input
Parts:
- added J2: Conn_01x02, SFUSat:2x01In_Header_v2, symbol Conn_01x02
Connections:
- wire segments 105 -> 108
Other:
- note added: "Extra 3V3 input located \nin satellite access hole"
Changed lines of the file:
@@
 	1    0    0    -1
 $EndComp
-Text Notes 1350 2050 0    60   ~ 0
+Text Notes 150  2500 0    60   ~ 0
 reverse polarity fet\n
 Text Notes 9900 4650 0    60   ~ 0
@@
 Connection ~ 5050 6350
 Connection ~ 5050 6550
+$Comp
+L Conn_01x02 J2
+U 1 1 5AD2E52A
+P 2850 2100
+F 0 "J2" H 2850 2200 50  0000 C CNN
+F 1 "Conn_01x02" H 2850 1900 50  0000 C CNN
+F 2 "SFUSat:2x01In_Header_v2" H 2850 2100 50  0001 C CNN
+F 3 "" H 2850 2100 50  0001 C CNN
+	1    2850 2100
+	1    0    0    -1
+$EndComp
+Text GLabel 2500 2100 0    60   Input ~ 0
+104_3v3
+Text GLabel 2500 2350 3    60   Input ~ 0
+104_In_GND
+Wire Wire Line
+	2650 2100 2500 2100
+Wire Wire Line
+	2500 2350 2500 2200
+Wire Wire Line
+	2500 2200 2650 2200
+Text Notes 2350 2000 0    60   ~ 0
+Extra 3V3 input located \nin satellite access hole
 $EndSCHEMATC
