File: v0.5/ADC.sch (KiCad schematic (older format))
At the start: 4 parts, among them U1 TMS570LS0714

Commit message: Removed extraneous 104 connections
Connections:
- net labels removed: AD1_10, AD1_3, AD1_4, AD1_5, AD1_6, AD1_7, AD1_8, AD1_9, RF_ADC1, RF_ADC2
- wire segments 78 -> 54
Changed lines of the file:
@@
 $Descr A4 11693 8268
 encoding utf-8
-Sheet 6 12
+Sheet 6 13
 Title ""
 Date ""
@@
 	1    0    0    -1
 $EndComp
-Text GLabel 3200 2450 0    60   Input ~ 0
-RF_ADC1
-Text GLabel 3200 2600 0    60   Input ~ 0
-RF_ADC2
-Wire Wire Line
-	3450 2500 3300 2500
-Wire Wire Line
-	3300 2500 3300 2450
-Wire Wire Line
-	3300 2450 3200 2450
-Wire Wire Line
-	3200 2600 3450 2600
 $Comp
 L R R7
@@
 INA_OUT
 Wire Wire Line
-	1000 2700 3450 2700
+	1000 2700 1200 2700
+Wire Wire Line
+	1200 2700 3450 2700
 Wire Wire Line
 	1200 2700 1200 2750
@@
 $EndComp
 Wire Wire Line
-	2900 2000 3450 2000
+	2900 2000 3300 2000
+Wire Wire Line
+	3300 2000 3450 2000
 Wire Wire Line
 	3450 1900 3300 1900
@@
 Wire Wire Line
 	2350 2300 3450 2300
-Text GLabel 2050 2800 0    60   Input ~ 0
-AD1_3
-Wire Wire Line
-	2050 2800 3450 2800
-Text GLabel 2050 2950 0    60   Input ~ 0
-AD1_4
-Text GLabel 2050 3100 0    60   Input ~ 0
-AD1_5
-Text GLabel 2050 3250 0    60   Input ~ 0
-AD1_6
-Text GLabel 2050 3400 0    60   Input ~ 0
-AD1_7
-Text GLabel 2050 3550 0    60   Input ~ 0
-AD1_8
-Text GLabel 2050 3700 0    60   Input ~ 0
-AD1_9
-Text GLabel 2050 3850 0    60   Input ~ 0
-AD1_10
-Wire Wire Line
-	2050 2950 2100 2950
-Wire Wire Line
-	2100 2950 2100 2900
-Wire Wire Line
-	2100 2900 3450 2900
-Wire Wire Line
-	2100 3000 3450 3000
-Wire Wire Line
-	2100 3000 2100 3100
-Wire Wire Line
-	2100 3100 2050 3100
-Wire Wire Line
-	2050 3250 2150 3250
-Wire Wire Line
-	2150 3250 2150 3100
-Wire Wire Line
-	2150 3100 3450 3100
-Wire Wire Line
-	2050 3400 2200 3400
-Wire Wire Line
-	2200 3400 2200 3200
-Wire Wire Line
-	2200 3200 3450 3200
-Wire Wire Line
-	2050 3550 2250 3550
-Wire Wire Line
-	2250 3550 2250 3300
-Wire Wire Line
-	2250 3300 3450 3300
-Wire Wire Line
-	2050 3700 2300 3700
-Wire Wire Line
-	2300 3700 2300 3400
-Wire Wire Line
-	2300 3400 3450 3400
-Wire Wire Line
-	2050 3850 2350 3850
-Wire Wire Line
-	2350 3850 2350 3500
-Wire Wire Line
-	2350 3500 3450 3500
 Text GLabel 2050 4000 0    60   Input ~ 0
 AD1_11

Commit message: Removed traces, gen netlist, fixed button footprints
Connections:
- wire segments 54 -> 52
Changed lines of the file:
@@
 INA_OUT
 Wire Wire Line
-	1000 2700 1200 2700
-Wire Wire Line
-	1200 2700 3450 2700
+	1000 2700 3450 2700
 Wire Wire Line
 	1200 2700 1200 2750
@@
 3v3
 $Comp
-L +3V3 #PWR054
+L +3V3 #PWR55
 U 1 1 59681373
 P 4650 1050
-F 0 "#PWR054" H 4650 900 50  0001 C CNN
+F 0 "#PWR55" H 4650 900 50  0001 C CNN
 F 1 "+3V3" H 4650 1190 50  0000 C CNN
 F 2 "" H 4650 1050 50  0000 C CNN
@@
 	4500 1050 4650 1050
 $Comp
-L +3V3 #PWR055
+L +3V3 #PWR54
 U 1 1 596815A0
 P 3300 1750
-F 0 "#PWR055" H 3300 1600 50  0001 C CNN
+F 0 "#PWR54" H 3300 1600 50  0001 C CNN
 F 1 "+3V3" H 3300 1890 50  0000 C CNN
 F 2 "" H 3300 1750 50  0000 C CNN
@@
 $EndComp
 $Comp
-L +3V3 #PWR056
+L +3V3 #PWR52
 U 1 1 596815BA
 P 2550 2100
-F 0 "#PWR056" H 2550 1950 50  0001 C CNN
+F 0 "#PWR52" H 2550 1950 50  0001 C CNN
 F 1 "+3V3" H 2550 2240 50  0000 C CNN
 F 2 "" H 2550 2100 50  0000 C CNN
@@
 $EndComp
 $Comp
-L GND #PWR057
+L GND #PWR53
 U 1 1 596815EE
 P 2900 2000
-F 0 "#PWR057" H 2900 1750 50  0001 C CNN
+F 0 "#PWR53" H 2900 1750 50  0001 C CNN
 F 1 "GND" H 2900 2100 50  0000 C CNN
 F 2 "" H 2900 2000 50  0000 C CNN
@@
 $EndComp
 Wire Wire Line
-	2900 2000 3300 2000
-Wire Wire Line
-	3300 2000 3450 2000
+	2900 2000 3450 2000
 Wire Wire Line
 	3450 1900 3300 1900
