File: v0.5/Extra.sch (KiCad schematic (older format))
At the start: 1 part, among them U1 TMS570LS0714

Commit message: Removed extraneous 104 connections
Parts:
- removed U1: TMS570LS0714, Housings_QFP:LQFP-144_20x20mm_Pitch0.5mm, symbol TMS570LS0714
- added U?: TMS570LS0714, symbol TMS570LS0714
Connections:
- net labels added: LIN_RX, LIN_TX
- net labels removed: I2C_SCL, I2C_SDA
Changed lines of the file:
@@
 $Descr A4 11693 8268
 encoding utf-8
-Sheet 12 13
+Sheet 13 13
 Title ""
 Date ""
@@
 $EndDescr
 $Comp
-L TMS570LS0714 U1
-U 8 1 597160C7
-P 7400 2150
-F 0 "U1" H 7800 2700 60  0000 C CNN
-F 1 "TMS570LS0714" H 7350 2700 60  0000 C CNN
-F 2 "Housings_QFP:LQFP-144_20x20mm_Pitch0.5mm" H 5000 900 60  0001 C CNN
-F 3 "" H 5000 900 60  0001 C CNN
-	8    7400 2150
+L TMS570LS0714 U?
+U 11 1 5AADD749
+P 5500 2800
+F 0 "U?" H 5900 3350 60  0000 C CNN
+F 1 "TMS570LS0714" H 5450 3350 60  0000 C CNN
+F 2 "" H 3100 1550 60  0001 C CNN
+F 3 "" H 3100 1550 60  0001 C CNN
+	11   5500 2800
 	1    0    0    -1
 $EndComp
-Text GLabel 6700 2100 0    60   Input ~ 0
-I2C_SDA
-Text GLabel 6700 2300 0    60   Input ~ 0
-I2C_SCL
+Text GLabel 5050 2450 0    60   Input ~ 0
+LIN_RX
+Text GLabel 5050 2600 0    60   Input ~ 0
+LIN_TX
 Wire Wire Line
-	6700 2100 6850 2100
+	5050 2450 5250 2450
 Wire Wire Line
-	6850 2300 6700 2300
+	5250 2600 5050 2600
 $EndSCHEMATC

Commit message: Removed traces, gen netlist, fixed button footprints
Parts:
- U1: renamed from U?; footprint (none) -> Housings_QFP:LQFP-144_20x20mm_Pitch0.5mm
Changed lines of the file:
@@
 $EndDescr
 $Comp
-L TMS570LS0714 U?
+L TMS570LS0714 U1
 U 11 1 5AADD749
 P 5500 2800
-F 0 "U?" H 5900 3350 60  0000 C CNN
+F 0 "U1" H 5900 3350 60  0000 C CNN
 F 1 "TMS570LS0714" H 5450 3350 60  0000 C CNN
-F 2 "" H 3100 1550 60  0001 C CNN
+F 2 "Housings_QFP:LQFP-144_20x20mm_Pitch0.5mm" H 3100 1550 60  0001 C CNN
 F 3 "" H 3100 1550 60  0001 C CNN
 	11   5500 2800

Commit message: Added 4 more xGPIO
From CAN peripheral. Currently unused
Connections:
- net labels added: xGPIO10, xGPIO11, xGPIO12, xGPIO9
- wire segments 2 -> 6
Changed lines of the file:
@@
 LIBS:valves
 LIBS:SFUSat
+LIBS:OBC_05-cache
 EELAYER 25 0
 EELAYER END
@@
 Wire Wire Line
 	5250 2600 5050 2600
+Text GLabel 5050 3150 0    60   Input ~ 0
+xGPIO9
+Text GLabel 5050 3300 0    60   Input ~ 0
+xGPIO10
+Text GLabel 5050 3450 0    60   Input ~ 0
+xGPIO11
+Text GLabel 5050 3600 0    60   Input ~ 0
+xGPIO12
+Wire Wire Line
+	5050 3150 5250 3150
+Wire Wire Line
+	5250 3300 5050 3300
+Wire Wire Line
+	5050 3450 5250 3450
+Wire Wire Line
+	5050 3600 5250 3600
 $EndSCHEMATC
