File: v0.5/NHET.sch (KiCad schematic (older format))
At the start: 1 part, among them U1 TMS570LS0714

Commit message: Removed extraneous 104 connections
Connections:
- net labels removed: NHET1_22, NHET1_26, NHET1_4, NHET1_7, RF_PWM1, RF_PWM2
- wire segments 6 -> 0
Changed lines of the file:
@@
 $Descr A4 11693 8268
 encoding utf-8
-Sheet 7 12
+Sheet 7 13
 Title ""
 Date ""
@@
 	1    0    0    -1
 $EndComp
-Text GLabel 6150 2800 0    60   Input ~ 0
-RF_PWM1
-Text GLabel 6150 2950 0    60   Input ~ 0
-RF_PWM2
-Wire Wire Line
-	6350 2800 6150 2800
-Wire Wire Line
-	6150 2950 6350 2950
-Text GLabel 6100 2050 0    60   Input ~ 0
-NHET1_4
-Text GLabel 6100 3700 0    60   Input ~ 0
-NHET1_7
-Text GLabel 6150 3100 0    60   Input ~ 0
-NHET1_22
-Text GLabel 6150 3250 0    60   Input ~ 0
-NHET1_26
-Wire Wire Line
-	6100 2050 6350 2050
-Wire Wire Line
-	6150 3100 6350 3100
-Wire Wire Line
-	6150 3250 6350 3250
-Wire Wire Line
-	6100 3700 6350 3700
 $EndSCHEMATC

Commit message: Made 4 layer PCB, WIP: decoupling caps
Connections:
- net labels added: xNHET0, xNHET1
- wire segments 0 -> 2
Other:
- note added: "Spare NHET in case we \nneed to turn them into a \nUART or i2c or something\n"
Changed lines of the file:
@@
 	1    0    0    -1
 $EndComp
+Text GLabel 6150 3100 0    60   Input ~ 0
+xNHET0
+Text GLabel 6150 3250 0    60   Input ~ 0
+xNHET1
+Wire Wire Line
+	6150 3100 6350 3100
+Wire Wire Line
+	6350 3250 6150 3250
+Text Notes 4450 3300 0    60   ~ 0
+Spare NHET in case we \nneed to turn them into a \nUART or i2c or something\n
 $EndSCHEMATC
