File: v0.5/RTC.sch (KiCad schematic (older format))
At the start: 7 parts, among them P8 RTC_SPI, U8 AB-RTCMC-EOA9-S3

Commit message: Updated 1.2v regulator, removed DC jack
Parts:
- C30: footprint SFUSat:Supercap_v2 -> SFUSat:Supercap_dual
Changed lines of the file:
@@
 EESchema Schematic File Version 2
+LIBS:OBC_05-rescue
 LIBS:power
 LIBS:device
@@
 LIBS:valves
 LIBS:SFUSat
-LIBS:OBC_04-cache
+LIBS:OBC_05-cache
 EELAYER 25 0
 EELAYER END
@@
 F 0 "C30" H 5275 2300 50  0000 L CNN
 F 1 "470µF" H 5275 2100 50  0000 L CNN
-F 2 "SFUSat:Supercap_v2" H 5250 2200 50  0001 C CNN
+F 2 "SFUSat:Supercap_dual" H 5250 2200 50  0001 C CNN
 F 3 "" H 5250 2200 50  0000 C CNN
 	1    5250 2200
