File: v0.5/SPI.sch (KiCad schematic (older format))
At the start: 1 part, among them U1 TMS570LS0714

Commit message: Removed extraneous 104 connections
Connections:
- net labels added: RF_CS2
- net labels removed: RF_GAIN_CS, SPI4_CLK, SPI4_CS0, SPI4_MISO, SPI4_MOSI
- wire segments 22 -> 15
Changed lines of the file:
@@
 $Descr A4 11693 8268
 encoding utf-8
-Sheet 4 12
+Sheet 4 13
 Title ""
 Date ""
@@
 	6000 5200 6250 5200
 Text GLabel 6000 5050 0    60   Input ~ 0
-RF_GAIN_CS
+RF_CS2
 Wire Wire Line
 	6250 5050 6000 5050
@@
 Text GLabel 5900 4450 0    60   Input ~ 0
 RTC_CLK
-Wire Wire Line
-	6050 1200 6200 1200
-Wire Wire Line
-	5850 1350 6200 1350
-Wire Wire Line
-	5850 1650 6200 1650
-Wire Wire Line
-	5850 1800 6200 1800
 Text GLabel 6200 2350 0    60   Input ~ 0
 FLASH_MOSI
@@
 Wire Wire Line
 	6400 3100 6200 3100
-Text GLabel 5850 1800 0    60   Input ~ 0
-SPI4_MISO
 Wire Wire Line
 	5900 4150 6250 4150
-Text GLabel 5850 1600 0    60   Input ~ 0
-SPI4_MOSI
 Wire Wire Line
 	5900 4300 6250 4300
-Text GLabel 5850 1150 0    60   Input ~ 0
-SPI4_CLK
 Wire Wire Line
 	5900 4450 6250 4450
-Text GLabel 5850 1350 0    60   Input ~ 0
-SPI4_CS0
 Wire Wire Line
 	5900 4600 6250 4600
-Wire Wire Line
-	5850 1650 5850 1600
-Wire Wire Line
-	6050 1200 6050 1150
-Wire Wire Line
-	6050 1150 5850 1150
 $EndSCHEMATC

Commit message: Added required xGPIO, removed 5V from 104 connector
Connections:
- net labels added: xGPIO0, xGPIO1, xGPIO2, xGPIO3, xGPIO4, xGPIO5, xGPIO6, xGPIO8
- wire segments 15 -> 23
Changed lines of the file:
@@
 Wire Wire Line
 	5900 4600 6250 4600
+Text GLabel 6200 2200 0    60   Input ~ 0
+xGPIO8
+Wire Wire Line
+	6200 2200 6400 2200
+Text GLabel 6200 3250 0    60   Input ~ 0
+xGPIO6
+Text GLabel 6200 3400 0    60   Input ~ 0
+xGPIO5
+Text GLabel 6200 3550 0    60   Input ~ 0
+xGPIO4
+Wire Wire Line
+	6200 3250 6400 3250
+Wire Wire Line
+	6200 3400 6400 3400
+Wire Wire Line
+	6200 3550 6400 3550
+Text GLabel 5900 4000 0    60   Input ~ 0
+xGPIO3
+Wire Wire Line
+	6250 4000 5900 4000
+Text GLabel 5950 1800 0    60   Input ~ 0
+xGPIO2
+Wire Wire Line
+	6200 1800 5950 1800
+Text GLabel 5950 1650 0    60   Input ~ 0
+xGPIO1
+Text GLabel 5950 1500 0    60   Input ~ 0
+xGPIO0
+Wire Wire Line
+	6200 1500 5950 1500
+Wire Wire Line
+	5950 1650 6200 1650
 $EndSCHEMATC
