File: v0.5/OBC_05.kicad_pcb (KiCad board)
At the start: 4 copper layers, 95.9 x 90.2 mm, 116 parts, among them J1 PC104-8BIT, P1 3v3_IN_CONNECTOR, P10 FLASH_CS, P11 USB_5V, P12 LOAD, P13 WD_EN, P14 WD_RST_EN, P16 JTAG_10PIN, P2 INA_INPUT, P3 INA_GND, P4 INA_EN, P5 INA_OUTPUT, P6 USB_PORT, P8 RTC_SPI, P9 FLASH_SPI, Q1 DMN2075U, Q2 DMN2075U, Q3 1v2_GOOD, Q5 DMN2075U, SW1 SPST, SW2 SPST, SW4 SPST, U1 TMS570LS0714, U10 FTDI_SSOP, U11 STLM75, U2 MCP1825S, U3 AP7361_3.3v, U4 INA301, U5 FLASH_IS25LP016D, U6 FLASH_IS25LP016D, U7 FLASH_IS25LP016D, U8 AB-RTCMC-EOA9-S3, U9 TPS3110, Y1 XTAL

Commit message: Added logo, finished routing
Parts:
- added G***: LOGO, SFUSat:SFUSat_15mm_2, F.Cu at (170.5, 81.0)
- moved W1 16.7 mm to (159.0, 100.2)
- moved P11 1.72 mm to (104.5, 91.7), turned to 180 degrees
- moved W11 1.13 mm to (130.6, 44.9)
- moved Q3 0.99 mm to (117.0, 91.8)
- moved C1 0.78 mm to (171.5, 56.1)
- moved R36 0.26 mm to (119.5, 87.0), turned to 90 degrees
Routing:
- net INA_INPUT: track 0.00 -> 53.8 mm, vias 0 -> 1
- net 5v0: track 15.6 -> 67.9 mm
- net INA_OUT: track 85.3 -> 129.2 mm, vias 4 -> 2
- net 104_In_GND: track 150.3 -> 189.5 mm, vias 7 -> 9
- net Net-(P4-Pad2): track 9.18 -> 26.4 mm
- net Net-(D3-Pad1): track 0.00 -> 12.1 mm
- net 104_GND: track 65.5 -> 54.9 mm
- net Net-(J1-Pad19B): track 4.13 -> 12.1 mm
- net USB_5V: track 28.4 -> 36.0 mm
- net (no net): track 17.1 -> 10.7 mm
- net INA_ALERT: track 11.6 -> 18.0 mm
- net Net-(J1-Pad20B): track 4.08 -> 8.68 mm
- net Net-(D1-Pad2): track 0.00 -> 4.38 mm, vias 0 -> 2
- net GND: track 161.2 -> 165.4 mm, vias 45 -> 46
- net FTDI_VCCIO: track 38.2 -> 42.2 mm
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Other:
- board text removed: "SDA"

Commit message: Tweaked silkscreen, power section
Parts:
- added G***: LOGO, SFUSat:long-logo, B.Cu at (191.0, 65.0)
Routing:
- net INA_INPUT: track 53.8 -> 91.9 mm, vias 1 -> 0
- net INA_OUT: track 129.2 -> 117.8 mm
Other:
- board text removed: "4 CLK"
- board text removed: "4 CS0"
- board text removed: "4 MISO"
- board text removed: "4 MOSI"

Commit message: relocated USB power enable header
It will now be accessible from the slot in the side of the satellite
Parts:
- moved P11 20.4 mm to (105.6, 71.3)
Routing:
- net USB_5V: track 36.0 -> 68.0 mm, vias 0 -> 2
- net 5v0: track 67.9 -> 94.8 mm

Commit message: Added slot-accessible 3v3 input
Parts:
- added J2: Conn_01x02, SFUSat:2x01In_Header_v2, F.Cu at (105.5, 48.9)
- moved P13 9.02 mm to (108.5, 41.2)
Routing:
- net 104_3v3: track 144.7 -> 243.8 mm
- net 104_In_GND: track 189.5 -> 218.2 mm, vias 9 -> 11
- net Net-(C31-Pad1): track 22.6 -> 31.5 mm
- net 3v3: track 97.4 -> 98.4 mm, vias 22 -> 23
Other:
- board text added: "- +"
- board text added: "3v3"
- board text added: "3v3 In"
- board text added: "USB_5V"
- board text removed: "USB_5V_EN"

Commit message: various cleanup
Routing:
- net xGPIO3: track 44.9 -> 46.7 mm
- net xGPIO4: track 45.3 -> 46.8 mm
- net 1v2: track 239.3 -> 240.6 mm
- net RTC_MISO: track 46.5 -> 47.7 mm
- net RTC_MOSI: track 42.4 -> 43.1 mm
- net xGPIO10: track 60.7 -> 60.1 mm
- net xNHET0: track 85.8 -> 85.3 mm
Other:
- board text added: "3V3 In"
- board text removed: "3v3"
- board text removed: "3v3 In"

Commit message: Redo watchdog disable
We now have two modes: program and space

- in program mode, watchdog is disabled
- in space mode, watchdog is enabled

- uses a MOSFET with gate pulled up normally (to connect watchdog reset and master reset), gate shorted to ground to disconnect master and watchdog resets.
Parts:
- removed G***: LOGO, SFUSat:SFUSat_15mm_2
- removed G***: LOGO, SFUSat:long-logo
- added Q4: DMN2075U, SFUSat:SOT23_DMN2075U, F.Cu at (108.5, 34.5)
- added R8: 10k, SFUSat:R_0402, F.Cu at (104.5, 36.0)
- added W2: MASTER_RST, SFUSat:Test_Point, F.Cu at (111.8, 45.5)
- P14: value WD_RST_EN -> WD_RST_DIS
- moved P14 20.7 mm to (105.5, 47.0), turned to 180 degrees
- moved J2 2.10 mm to (105.5, 51.0)
Connections:
- P14 pad 1: MASTER_RESET -> GND
- U9 pad 1: Net-(P14-Pad2) -> Net-(Q4-Pad3)
- W14 pad 1: Net-(P14-Pad2) -> Net-(Q4-Pad3)
Routing:
- net Net-(Q4-Pad3): track 0.00 -> 21.7 mm
- net Net-(P14-Pad2): track 10.6 -> 15.0 mm
- net 104_3v3: track 243.5 -> 246.7 mm
- net MASTER_RESET: track 94.7 -> 97.1 mm
- net 104_In_GND: track 218.2 -> 216.6 mm
- net 3v3: track 98.4 -> 99.2 mm, vias 23 -> 24
Other:
- board text added: "M RST"
- board text added: "WD_RST DISABLE"
- board text removed: "WD_RST_EN"

Commit message: FTDI is 3V3 powered now
Before, FTDI was exclusively 5v powered. Since the main supply is now 3.3, we can't do that. Moved to 3.3V
Parts:
- moved C33 11.5 mm to (110.2, 75.6), turned to 270 degrees
Connections:
- C8 pad 1: FTDI_VCCIO -> 3v3
- R32 pad 1: FTDI_VCCIO -> 3v3
- R33 pad 1: FTDI_VCCIO -> 3v3
- R34 pad 1: FTDI_VCCIO -> 3v3
- R35 pad 1: FTDI_VCCIO -> 3v3
- R36 pad 1: FTDI_VCCIO -> 3v3
- R37 pad 1: FTDI_VCCIO -> 3v3
- U10 pad 10: FTDI_VCCIO -> 3v3
- U10 pad 11: FTDI_VCCIO -> 3v3
- U10 pad 12: USB_5V -> 3v3
- U10 pad 3: FTDI_VCCIO -> 3v3
Routing:
- net USB_5V: track 68.0 -> 16.7 mm, vias 2 -> 0
- net FTDI_VCCIO: track 42.2 -> 0.00 mm, vias 2 -> 0
- net 3v3: track 99.2 -> 139.9 mm, vias 24 -> 28
- net 104_In_GND: track 216.6 -> 220.0 mm

Commit message: Added logos
Parts:
- added G***: LOGO, SFUSat:SFUSat_15mm_2, F.Cu at (169.3, 79.7)
- added G***: LOGO, SFUSat:long2, B.Cu at (191.3, 65.4)
