File: v0.5/Flash.sch (KiCad schematic (older format))
At the start: 11 parts, among them P10 FLASH_CS, P9 FLASH_SPI, U5 FLASH_IS25LP016D, U6 FLASH_IS25LP016D, U7 FLASH_IS25LP016D

Commit message: not finished layout routing
Parts:
- P10, P9: symbol CONN_01X03 -> Conn_01x03
Changed lines of the file:
@@
 	9700 950  10100 950
 $Comp
-L CONN_01X03 P10
+L Conn_01x03 P10
 U 1 1 5968894C
 P 2750 6300
@@
 FLASH_CLK
 $Comp
-L CONN_01X03 P9
+L Conn_01x03 P9
 U 1 1 59688A9E
 P 2000 6300

Commit message: fixed 104 and connections in schematic
Parts:
- P10, P9: symbol Conn_01x03 -> CONN_01X03
Changed lines of the file:
@@
 	9700 950  10100 950
 $Comp
-L Conn_01x03 P10
+L CONN_01X03 P10
 U 1 1 5968894C
 P 2750 6300
@@
 FLASH_CLK
 $Comp
-L Conn_01x03 P9
+L CONN_01X03 P9
 U 1 1 59688A9E
 P 2000 6300
