File: v0.5/i2c.sch (KiCad schematic (older format))
At the start: 1 part, among them U1 TMS570LS0714

Commit message: Added logo, I2c pullup
- i2c now has pullup resistor pads. 
- added big logo on the bottom side
Parts:
- added R10, R11: 10k, SFUSat:R_0402, symbol R
Connections:
- net labels added: +3V3, 3v3
- wire segments 2 -> 7
Other:
- note added: "I2C pullup resistor values are hotly contested. \nTemp sensor datasheet says 10k, this has been tested\nand works with 0.4. May need to adjust once more devices\nare on the bus."
Changed lines of the file:
@@
 	1    0    0    -1
 $EndComp
-Text GLabel 6700 2100 0    60   Input ~ 0
+Text GLabel 6150 2100 0    60   Input ~ 0
 I2C_SDA
-Text GLabel 6700 2300 0    60   Input ~ 0
+Text GLabel 6150 2300 0    60   Input ~ 0
 I2C_SCL
 Wire Wire Line
-	6700 2100 6850 2100
+	6150 2100 6850 2100
 Wire Wire Line
-	6850 2300 6700 2300
+	6150 2300 6850 2300
+$Comp
+L R R10
+U 1 1 5AD996EA
+P 6350 1650
+F 0 "R10" V 6430 1650 50  0000 C CNN
+F 1 "10k" V 6350 1650 50  0000 C CNN
+F 2 "SFUSat:R_0402" V 6280 1650 50  0001 C CNN
+F 3 "" H 6350 1650 50  0000 C CNN
+	1    6350 1650
+	1    0    0    -1
+$EndComp
+Text GLabel 8850 1350 3    60   Input ~ 0
+3v3
+$Comp
+L +3V3 #PWR84
+U 1 1 5AD99743
+P 8850 1200
+F 0 "#PWR84" H 8850 1050 50  0001 C CNN
+F 1 "+3V3" H 8850 1340 50  0000 C CNN
+F 2 "" H 8850 1200 50  0000 C CNN
+F 3 "" H 8850 1200 50  0000 C CNN
+	1    8850 1200
+	1    0    0    -1
+$EndComp
+$Comp
+L +3V3 #PWR83
+U 1 1 5AD99760
+P 6650 1300
+F 0 "#PWR83" H 6650 1150 50  0001 C CNN
+F 1 "+3V3" H 6650 1440 50  0000 C CNN
+F 2 "" H 6650 1300 50  0000 C CNN
+F 3 "" H 6650 1300 50  0000 C CNN
+	1    6650 1300
+	1    0    0    -1
+$EndComp
+$Comp
+L +3V3 #PWR82
+U 1 1 5AD9977D
+P 6350 1300
+F 0 "#PWR82" H 6350 1150 50  0001 C CNN
+F 1 "+3V3" H 6350 1440 50  0000 C CNN
+F 2 "" H 6350 1300 50  0000 C CNN
+F 3 "" H 6350 1300 50  0000 C CNN
+	1    6350 1300
+	1    0    0    -1
+$EndComp
+Wire Wire Line
+	6350 1300 6350 1500
+Wire Wire Line
+	6650 1500 6650 1300
+Wire Wire Line
+	6350 1800 6350 2100
+Connection ~ 6350 2100
+Wire Wire Line
+	6650 1800 6650 2300
+Connection ~ 6650 2300
+Wire Wire Line
+	8850 1200 8850 1350
+Text Notes 5700 2900 0    60   ~ 0
+I2C pullup resistor values are hotly contested. \nTemp sensor datasheet says 10k, this has been tested\nand works with 0.4. May need to adjust once more devices\nare on the bus.
+$Comp
+L R R11
+U 1 1 5AD99C5E
+P 6650 1650
+F 0 "R11" V 6730 1650 50  0000 C CNN
+F 1 "10k" V 6650 1650 50  0000 C CNN
+F 2 "SFUSat:R_0402" V 6580 1650 50  0001 C CNN
+F 3 "" H 6650 1650 50  0000 C CNN
+	1    6650 1650
+	1    0    0    -1
+$EndComp
 $EndSCHEMATC
